Commit message: [1] Solving Gazebo issues

File: urdf/lynxmotion_al5d.gazebo.xacro (robot description, xacro)
@@ -3,20 +3,6 @@
     <xacro:include filename="$(find lynxmotion_al5d_description)/urdf/lynxmotion_al5d_properties.urdf.xacro" />
     <!-- Base link comprising the board behind the robot and the cylinder at its bottom -->
-    <!-- <link name="world">
-        <visual>
-            <geometry>
-                <box size="0.001 0.001 0.001" />
-            </geometry>
-            <origin rpy="0 0 0" xyz="0 0 0" />
-        </visual>
-        <collision>
-            <geometry>
-                <box size="0.001 0.001 0.001" />
-            </geometry>
-            <origin rpy="0 0 0" xyz="0 0 0" />
-        </collision>
-        <xacro:inertial_matrix_bis mass="1" />
-    </link>
-    <gazebo reference="world" /> -->
+    <link name="world" />
+    <gazebo reference="world" />
     <link name="robot_support">
         <visual>
@@ -189,9 +175,9 @@
     </sensor>
     <!-- Adding joints -->
-    <!-- <joint name="world_to_robot" type="fixed">
+    <joint name="world_to_robot" type="fixed">
         <parent link="world" />
         <child link="robot_support" />
         <dynamics damping="0" friction="0" />
-    </joint> -->
+    </joint>
     <joint name="camera_joint" type="fixed">
         <parent link="robot_support" />

Commit message: Fixing bugs

File: urdf/lynxmotion_al5d.gazebo.xacro (robot description, xacro)
@@ -1,5 +1,8 @@
 <?xml version="1.0" ?>
 <robot name="lynxmotion_al5d" xmlns:xacro="http://www.ros.org/wiki/xacro" xmlns:sensor="http://playerstage.sourceforge.net/gazebo/xmlschema/#sensor" xmlns:controller="http://playerstage.sourceforge.net/gazebo/xmlschema/#controller" xmlns:interface="http://playerstage.sourceforge.net/gazebo/xmlschema/#interface">
+<!-- This file has been created specifically to run with Gazebo since this requires a specific link named world for the robot to stick to the map -->
     <xacro:include filename="$(find lynxmotion_al5d_description)/urdf/lynxmotion_al5d_properties.urdf.xacro" />
+    <!-- Base link comprising the board behind the robot and the cylinder at its bottom -->
+    <link name="world" />
     <link name="robot_support">
         <visual>
@@ -172,13 +175,18 @@
     </sensor>
     <!-- Adding joints -->
-    <!-- <joint name="world_to_robot" type="fixed">
+    <joint name="world_to_robot" type="fixed">
         <parent link="world" />
         <child link="robot_support" />
         <dynamics damping="0" friction="0" />
-    </joint> -->
+    </joint>
     <joint name="camera_joint" type="fixed">
         <parent link="robot_support" />
         <child link="camera_link" />
         <origin xyz="0 -0.35 0" />
+        <dynamics damping="10" friction="0.7" />
+    </joint>
+    <joint name="robot_base_fixed" type="fixed">
+        <parent link="robot_base_cylinder" />
+        <child link="robot_base_top_box" />
         <dynamics damping="10" friction="0.7" />
     </joint>
@@ -192,9 +200,4 @@
         <dynamics damping="10" friction="0.7" />
     </joint>
-    <joint name="base_to_cylinder" type="fixed">
-        <parent link="robot_base_cylinder" />
-        <child link="robot_base_top_box" />
-        <dynamics damping="10" friction="0.7" />
-    </joint>
     <joint name="Joint2" type="revolute">
         <parent link="robot_base_top_box" />
@@ -240,5 +243,5 @@
         <child link="right_finger" />
         <origin xyz="0 -0.01 0" />
-        <limit effort="10" velocity="0.001" lower="0" upper="${gripper_base_width/2}" />
+        <limit effort="10" velocity="0.005" lower="0" upper="${gripper_base_width/2}" />
         <mimic joint="Gripper" multiplier="-1" />
         <dynamics damping="10" friction="0.7" />

Commit message: Fixed issues identified at the previous step

File: urdf/lynxmotion_al5d.gazebo.xacro (robot description, xacro)
@@ -4,5 +4,5 @@
     <xacro:include filename="$(find lynxmotion_al5d_description)/urdf/lynxmotion_al5d_properties.urdf.xacro" />
     <!-- Base link comprising the board behind the robot and the cylinder at its bottom -->
-    <link name="world" />
+    <!-- <link name="world" /> -->
     <link name="robot_support">
         <visual>
@@ -175,18 +175,13 @@
     </sensor>
     <!-- Adding joints -->
-    <joint name="world_to_robot" type="fixed">
+    <!-- <joint name="world_to_robot" type="fixed">
         <parent link="world" />
         <child link="robot_support" />
         <dynamics damping="0" friction="0" />
-    </joint>
+    </joint> -->
     <joint name="camera_joint" type="fixed">
         <parent link="robot_support" />
         <child link="camera_link" />
         <origin xyz="0 -0.35 0" />
-        <dynamics damping="10" friction="0.7" />
-    </joint>
-    <joint name="robot_base_fixed" type="fixed">
-        <parent link="robot_base_cylinder" />
-        <child link="robot_base_top_box" />
         <dynamics damping="10" friction="0.7" />
     </joint>
@@ -198,4 +193,9 @@
         <limit effort="10" velocity="1" lower="${-PI}" upper="${PI}" />
         <dynamics damping="0" friction="0" />
+        <dynamics damping="10" friction="0.7" />
+    </joint>
+    <joint name="robot_base_fixed" type="fixed">
+        <parent link="robot_base_cylinder" />
+        <child link="robot_base_top_box" />
         <dynamics damping="10" friction="0.7" />
     </joint>

File: urdf/lynxmotion_al5d.xacro (robot description, xacro)
@@ -1,9 +1,10 @@
 <?xml version="1.0" ?>
 <robot name="lynxmotion_al5d" xmlns:xacro="http://www.ros.org/wiki/xacro" xmlns:sensor="http://playerstage.sourceforge.net/gazebo/xmlschema/#sensor" xmlns:controller="http://playerstage.sourceforge.net/gazebo/xmlschema/#controller" xmlns:interface="http://playerstage.sourceforge.net/gazebo/xmlschema/#interface">
-    <xacro:include filename="$(find lynxmotion_al5d_description)/urdf/lynxmotion_al5d_properties.urdf.xacro" />
-    <link name="robot_support">
-        <visual>
-            <geometry>
-                <mesh filename="package://lynxmotion_al5d_description/meshes/robot_parts/support.dae" />
+    <xacro:include filename="$(find al5d_description)/urdf/lynxmotion_al5d_properties.urdf.xacro" />
+    <!-- Base link comprising the board behind the robot and the cylinder at its bottom -->
+    <!-- <link name="world">
+        <visual>
+            <geometry>
+                <box size="0.001 0.001 0.001" />
             </geometry>
             <origin rpy="0 0 0" xyz="0 0 0" />
@@ -11,15 +12,31 @@
         <collision>
             <geometry>
-                <mesh filename="package://lynxmotion_al5d_description/meshes/robot_parts/support.dae" />
+                <box size="0.001 0.001 0.001" />
             </geometry>
             <origin rpy="0 0 0" xyz="0 0 0" />
         </collision>
+        <xacro:inertial_matrix_bis mass="1" />
+    </link>
+    <gazebo reference="world" /> -->
+    <link name="base_link">
+        <visual>
+            <geometry>
+                <mesh filename="package://al5d_description/meshes/robot_parts/support.dae" />
+            </geometry>
+            <origin rpy="0 0 0" xyz="0 0 0" />
+        </visual>
+        <collision>
+            <geometry>
+                <mesh filename="package://al5d_description/meshes/robot_parts/support.dae" />
+            </geometry>
+            <origin rpy="0 0 0" xyz="0 0 0" />
+        </collision>
         <xacro:inertial_matrix mass="0.133" ixx="3.6565e-7" ixy="-3.72e-9" ixz="1e-6" iyy="9.404e-8" iyz="4.375e-8" izz="4.1776e-7" xyz="0.000585 0.0602746 0.0170628" />
     </link>
-    <gazebo reference="robot_support" />
+    <gazebo reference="base_link" />
     <link name="robot_base_cylinder">
         <visual>
             <geometry>
-                <mesh filename="package://lynxmotion_al5d_description/meshes/robot_parts/rotation_cylinder.dae" />
+                <mesh filename="package://al5d_description/meshes/robot_parts/rotation_cylinder.dae" />
             </geometry>
             <origin rpy="0 0 0" xyz="0 -0.021165 0" />
@@ -27,5 +44,5 @@
         <collision>
             <geometry>
-                <mesh filename="package://lynxmotion_al5d_description/meshes/robot_parts/rotation_cylinder.dae" />
+                <mesh filename="package://al5d_description/meshes/robot_parts/rotation_cylinder.dae" />
             </geometry>
             <origin rpy="0 0 0" xyz="0 -0.021165 0" />
@@ -37,5 +54,5 @@
         <visual>
             <geometry>
-                <mesh filename="package://lynxmotion_al5d_description/meshes/robot_parts/top_box.dae" />
+                <mesh filename="package://al5d_description/meshes/robot_parts/top_box.dae" />
             </geometry>
             <origin xyz="0.007 -0.024 0" rpy="0 0 0" />
@@ -43,5 +60,5 @@
         <collision>
             <geometry>
-                <mesh filename="package://lynxmotion_al5d_description/meshes/robot_parts/top_box.dae" />
+                <mesh filename="package://al5d_description/meshes/robot_parts/top_box.dae" />
             </geometry>
             <origin xyz="0.007 -0.024 0" rpy="0 0 0" />
@@ -53,5 +70,5 @@
         <visual>
             <geometry>
-                <mesh filename="package://lynxmotion_al5d_description/meshes/robot_parts/shoulder.dae" />
+                <mesh filename="package://al5d_description/meshes/robot_parts/shoulder.dae" />
             </geometry>
             <origin rpy="${-5*PI/8} 0 0" xyz="0 -0.0625 0.036" />
@@ -59,5 +76,5 @@
         <collision>
             <geometry>
-                <mesh filename="package://lynxmotion_al5d_description/meshes/robot_parts/shoulder.dae" />
+                <mesh filename="package://al5d_description/meshes/robot_parts/shoulder.dae" />
             </geometry>
             <origin rpy="${-5*PI/8} 0 0" xyz="0 -0.0625 0.036" />
@@ -69,5 +86,5 @@
         <visual>
             <geometry>
-                <mesh filename="package://lynxmotion_al5d_description/meshes/robot_parts/arm.dae" />
+                <mesh filename="package://al5d_description/meshes/robot_parts/arm.dae" />
             </geometry>
             <origin rpy="-0.895 0 0" xyz="0 ${-tube_length + 2*hs_755eb_depth/5} ${-shoulder_to_elbow - 0.02}" />
@@ -75,5 +92,5 @@
         <collision>
             <geometry>
-                <mesh filename="package://lynxmotion_al5d_description/meshes/robot_parts/arm.dae" />
+                <mesh filename="package://al5d_description/meshes/robot_parts/arm.dae" />
             </geometry>
             <origin rpy="-0.895 0 0" xyz="0 ${-tube_length + 2*hs_755eb_depth/5} ${-shoulder_to_elbow - 0.02}" />
@@ -85,5 +102,5 @@
         <visual>
             <geometry>
-                <mesh filename="package://lynxmotion_al5d_description/meshes/robot_parts/wrist.dae" />
+                <mesh filename="package://al5d_description/meshes/robot_parts/wrist.dae" />
             </geometry>
             <origin rpy="${PI} 0 0" xyz="0.005 -0.165 0.067" />
@@ -91,5 +108,5 @@
         <collision>
             <geometry>
-                <mesh filename="package://lynxmotion_al5d_description/meshes/robot_parts/wrist.dae" />
+                <mesh filename="package://al5d_description/meshes/robot_parts/wrist.dae" />
             </geometry>
             <origin rpy="${PI} 0 0" xyz="0.005 -0.165 0.067" />
@@ -101,5 +118,5 @@
         <visual>
             <geometry>
-                <mesh filename="package://lynxmotion_al5d_description/meshes/robot_parts/gripper.dae" />
+                <mesh filename="package://al5d_description/meshes/robot_parts/gripper.dae" />
             </geometry>
             <origin rpy="${PI/2} 0 ${-PI/2}" xyz="0 -0.021 -0.005" />
@@ -107,5 +124,5 @@
         <collision>
             <geometry>
-                <mesh filename="package://lynxmotion_al5d_description/meshes/robot_parts/gripper.dae" />
+                <mesh filename="package://al5d_description/meshes/robot_parts/gripper.dae" />
             </geometry>
             <origin rpy="${PI/2} 0 ${-PI/2}" xyz="0 -0.021 -0.005" />
@@ -117,5 +134,5 @@
         <visual>
             <geometry>
-                <mesh filename="package://lynxmotion_al5d_description/meshes/robot_parts/finger_left.dae" />
+                <mesh filename="package://al5d_description/meshes/robot_parts/finger_left.dae" />
             </geometry>
             <origin rpy="${PI/2} 0 ${-PI/2}" xyz="0.003 -0.012 0" />
@@ -123,5 +140,5 @@
         <collision>
             <geometry>
-                <mesh filename="package://lynxmotion_al5d_description/meshes/robot_parts/finger_left.dae" />
+                <mesh filename="package://al5d_description/meshes/robot_parts/finger_left.dae" />
             </geometry>
             <origin rpy="${PI/2} 0 ${-PI/2}" xyz="0.003 -0.012 0" />
@@ -133,5 +150,5 @@
         <visual>
             <geometry>
-                <mesh filename="package://lynxmotion_al5d_description/meshes/robot_parts/finger_right.dae" />
+                <mesh filename="package://al5d_description/meshes/robot_parts/finger_right.dae" />
             </geometry>
             <origin rpy="${PI/2} 0 ${-PI/2}" xyz="-0.003 -0.012 0" />
@@ -139,5 +156,5 @@
         <collision>
             <geometry>
-                <mesh filename="package://lynxmotion_al5d_description/meshes/robot_parts/finger_right.dae" />
+                <mesh filename="package://al5d_description/meshes/robot_parts/finger_right.dae" />
             </geometry>
             <origin rpy="${PI/2} 0 ${-PI/2}" xyz="-0.003 -0.012 0" />
@@ -174,9 +191,9 @@
     <!-- <joint name="world_to_robot" type="fixed">
         <parent link="world" />
-        <child link="robot_support" />
+        <child link="base_link" />
         <dynamics damping="0" friction="0" />
     </joint> -->
     <joint name="camera_joint" type="fixed">
-        <parent link="robot_support" />
+        <parent link="base_link" />
         <child link="camera_link" />
         <origin xyz="0 -0.35 0" />
@@ -184,5 +201,5 @@
     </joint>
     <joint name="Joint1" type="revolute">
-        <parent link="robot_support" />
+        <parent link="base_link" />
         <child link="robot_base_cylinder" />
         <axis xyz="0 0 1" />

Commit message: Fixed issues identified at the previous step

File: urdf/lynxmotion_al5d.gazebo.xacro (robot description, xacro)
@@ -4,5 +4,5 @@
     <xacro:include filename="$(find lynxmotion_al5d_description)/urdf/lynxmotion_al5d_properties.urdf.xacro" />
     <!-- Base link comprising the board behind the robot and the cylinder at its bottom -->
-    <!-- <link name="world" /> -->
+    <link name="world" />
     <link name="robot_support">
         <visual>
@@ -175,9 +175,9 @@
     </sensor>
     <!-- Adding joints -->
-    <!-- <joint name="world_to_robot" type="fixed">
+    <joint name="world_to_robot" type="fixed">
         <parent link="world" />
         <child link="robot_support" />
         <dynamics damping="0" friction="0" />
-    </joint> -->
+    </joint>
     <joint name="camera_joint" type="fixed">
         <parent link="robot_support" />
@@ -281,5 +281,5 @@
                 <alwaysOn>true</alwaysOn>
                 <updateRate>1.0</updateRate>
-                <cameraName>al5d_external_vision</cameraName>
+                <cameraName>camera</cameraName>
                 <imageTopicName>image_raw</imageTopicName>
                 <cameraInfoTopicName>camera_info</cameraInfoTopicName>

File: urdf/lynxmotion_al5d.xacro (robot description, xacro)
@@ -3,20 +3,4 @@
     <xacro:include filename="$(find al5d_description)/urdf/lynxmotion_al5d_properties.urdf.xacro" />
     <!-- Base link comprising the board behind the robot and the cylinder at its bottom -->
-    <!-- <link name="world">
-        <visual>
-            <geometry>
-                <box size="0.001 0.001 0.001" />
-            </geometry>
-            <origin rpy="0 0 0" xyz="0 0 0" />
-        </visual>
-        <collision>
-            <geometry>
-                <box size="0.001 0.001 0.001" />
-            </geometry>
-            <origin rpy="0 0 0" xyz="0 0 0" />
-        </collision>
-        <xacro:inertial_matrix_bis mass="1" />
-    </link>
-    <gazebo reference="world" /> -->
     <link name="base_link">
         <visual>
@@ -189,9 +173,4 @@
     </sensor>
     <!-- Adding joints -->
-    <!-- <joint name="world_to_robot" type="fixed">
-        <parent link="world" />
-        <child link="base_link" />
-        <dynamics damping="0" friction="0" />
-    </joint> -->
     <joint name="camera_joint" type="fixed">
         <parent link="base_link" />
@@ -295,5 +274,5 @@
                 <alwaysOn>true</alwaysOn>
                 <updateRate>1.0</updateRate>
-                <cameraName>al5d_external_vision</cameraName>
+                <cameraName>camera</cameraName>
                 <imageTopicName>image_raw</imageTopicName>
                 <cameraInfoTopicName>camera_info</cameraInfoTopicName>
