Commit message: Working on the refactored simulator

File: urdf/lynxmotion_al5d.gazebo.xacro (robot description, xacro)
@@ -18,5 +18,5 @@
             <origin rpy="0 0 0" xyz="0 0 0" />
         </collision>
-        <xacro:inertial_matrix mass="0.133" ixx="3.6565e-7" ixy="-3.72e-9" ixz="1e-6" iyy="9.404e-8" iyz="4.375e-8" izz="4.1776e-7" xyz="0.000585 0.0602746 0.0170628" />
+        <xacro:inertial_matrix mass="1" ixx="3.6565e-7" ixy="-3.72e-9" ixz="1e-6" iyy="9.404e-8" iyz="4.375e-8" izz="4.1776e-7" xyz="0.000585 0.0602746 0.0170628" />
     </link>
     <gazebo reference="robot_support" />
@@ -34,5 +34,5 @@
             <origin rpy="0 0 0" xyz="0 -0.021165 0" />
         </collision>
-        <xacro:inertial_matrix_bis mass="0.042" />
+        <xacro:inertial_matrix_bis mass="0.01" />
     </link>
     <gazebo reference="robot_base_cylinder" />
@@ -42,5 +42,5 @@
                 <mesh filename="package://lynxmotion_al5d_description/meshes/robot_parts/top_box.dae" />
             </geometry>
-            <origin xyz="0.007 -0.024 0" rpy="0 0 0" />
+            <origin xyz="-0.007 0.024 0" rpy="0 0 ${PI}" />
         </visual>
         <collision>
@@ -48,7 +48,7 @@
                 <mesh filename="package://lynxmotion_al5d_description/meshes/robot_parts/top_box.dae" />
             </geometry>
-            <origin xyz="0.007 -0.024 0" rpy="0 0 0" />
-        </collision>
-        <xacro:inertial_matrix_bis mass="0.184" />
+            <origin xyz="-0.007 0.024 0" rpy="0 0 0" />
+        </collision>
+        <xacro:inertial_matrix_bis mass="0.6" />
     </link>
     <gazebo reference="robot_base_top_box" />
@@ -66,5 +66,5 @@
             <origin rpy="${-5*PI/8} 0 0" xyz="0 -0.0625 0.036" />
         </collision>
-        <xacro:inertial_matrix_bis mass="0.095" />
+        <xacro:inertial_matrix_bis mass="0.1" />
     </link>
     <gazebo reference="shoulder" />
@@ -74,5 +74,5 @@
                 <mesh filename="package://lynxmotion_al5d_description/meshes/robot_parts/arm.dae" />
             </geometry>
-            <origin rpy="-0.895 0 0" xyz="0 ${-tube_length + 2*hs_755eb_depth/5} ${-shoulder_to_elbow - 0.02}" />
+            <origin rpy="${-PI-0.895} 0 0" xyz="0 ${tube_length - 2*hs_755eb_depth/5} ${shoulder_to_elbow + 0.02}" />
         </visual>
         <collision>
@@ -80,7 +80,7 @@
                 <mesh filename="package://lynxmotion_al5d_description/meshes/robot_parts/arm.dae" />
             </geometry>
-            <origin rpy="-0.895 0 0" xyz="0 ${-tube_length + 2*hs_755eb_depth/5} ${-shoulder_to_elbow - 0.02}" />
-        </collision>
-        <xacro:inertial_matrix_bis mass="0.1" />
+            <origin rpy="${-PI-0.895} 0 0" xyz="0 ${-tube_length + 2*hs_755eb_depth/5} ${-shoulder_to_elbow - 0.02}" />
+        </collision>
+        <xacro:inertial_matrix_bis mass="0.05" />
     </link>
     <gazebo reference="arm" />
@@ -98,5 +98,5 @@
             <origin rpy="${PI} 0 0" xyz="0.005 -0.165 0.067" />
         </collision>
-        <xacro:inertial_matrix_bis mass="0.055" />
+        <xacro:inertial_matrix_bis mass="0" />
     </link>
     <gazebo reference="wrist" />
@@ -114,5 +114,5 @@
             <origin rpy="${PI/2} 0 ${-PI/2}" xyz="0 -0.021 -0.005" />
         </collision>
-        <xacro:inertial_matrix_bis mass="0.042" />
+        <xacro:inertial_matrix_bis mass="0" />
     </link>
     <gazebo reference="gripper" />
@@ -130,5 +130,5 @@
             <origin rpy="${PI/2} 0 ${-PI/2}" xyz="0.003 -0.012 0" />
         </collision>
-        <xacro:inertial_matrix_bis mass="0.0006" />
+        <xacro:inertial_matrix_bis mass="0" />
     </link>
     <gazebo reference="left_finger" />
@@ -146,5 +146,5 @@
             <origin rpy="${PI/2} 0 ${-PI/2}" xyz="-0.003 -0.012 0" />
         </collision>
-        <xacro:inertial_matrix_bis mass="0.0006" />
+        <xacro:inertial_matrix_bis mass="0" />
     </link>
     <gazebo reference="right_finger" />
@@ -186,14 +186,14 @@
         <dynamics damping="10" friction="0.7" />
     </joint>
-    <joint name="Joint1" type="revolute">
+     <joint name="Joint1" type="revolute">
         <parent link="robot_support" />
         <child link="robot_base_cylinder" />
-        <axis xyz="0 0 1" />
-        <origin xyz="0 0.021 0" />
+        <axis xyz="0 0 -1" />
+        <origin xyz="0 0.021 0" rpy="0 0 ${PI}" />
         <limit effort="10" velocity="1" lower="${-PI}" upper="${PI}" />
         <dynamics damping="0" friction="0" />
         <dynamics damping="10" friction="0.7" />
     </joint>
-    <joint name="robot_base_fixed" type="fixed">
+    <joint name="base_to_cylinder" type="fixed">
         <parent link="robot_base_cylinder" />
         <child link="robot_base_top_box" />
@@ -203,6 +203,6 @@
         <parent link="robot_base_top_box" />
         <child link="shoulder" />
-        <axis xyz="1 0 0" />
-        <origin xyz="0 -0.015 0.071" />
+        <axis xyz="1 0 0"/>
+        <origin xyz="0 0.015 0.071"  rpy="0 0 0" />
         <limit effort="10" velocity="1" lower="0" upper="${PI}" />
         <dynamics damping="10" friction="0.7" />
@@ -220,5 +220,5 @@
         <child link="wrist" />
         <axis xyz="1 0 0" />
-        <origin xyz="0 ${-tube_length - hs_645_depth + 0.003} 0" rpy="0 0 ${PI}"/>
+        <origin xyz="0 ${tube_length + hs_645_depth - 0.003} 0" rpy="0 0 0"/>
         <limit effort="10" velocity="1" lower="${-PI/2}" upper="${PI/2}" />
         <dynamics damping="10" friction="0.7" />

File: urdf/lynxmotion_al5d.xacro (robot description, xacro)
@@ -40,5 +40,5 @@
                 <mesh filename="package://lynxmotion_al5d_description/meshes/robot_parts/top_box.dae" />
             </geometry>
-            <origin xyz="0.007 -0.024 0" rpy="0 0 0" />
+            <origin xyz="-0.007 0.024 0" rpy="0 0 ${PI}" />
         </visual>
         <collision>
@@ -46,5 +46,5 @@
                 <mesh filename="package://lynxmotion_al5d_description/meshes/robot_parts/top_box.dae" />
             </geometry>
-            <origin xyz="0.007 -0.024 0" rpy="0 0 0" />
+            <origin xyz="-0.007 0.024 0" rpy="0 0 0" />
         </collision>
         <xacro:inertial_matrix_bis mass="0.184" />
@@ -72,5 +72,5 @@
                 <mesh filename="package://lynxmotion_al5d_description/meshes/robot_parts/arm.dae" />
             </geometry>
-            <origin rpy="-0.895 0 0" xyz="0 ${-tube_length + 2*hs_755eb_depth/5} ${-shoulder_to_elbow - 0.02}" />
+            <origin rpy="${-PI-0.895} 0 0" xyz="0 ${tube_length - 2*hs_755eb_depth/5} ${shoulder_to_elbow + 0.02}" />
         </visual>
         <collision>
@@ -78,5 +78,5 @@
                 <mesh filename="package://lynxmotion_al5d_description/meshes/robot_parts/arm.dae" />
             </geometry>
-            <origin rpy="-0.895 0 0" xyz="0 ${-tube_length + 2*hs_755eb_depth/5} ${-shoulder_to_elbow - 0.02}" />
+            <origin rpy="${-PI-0.895} 0 0" xyz="0 ${-tube_length + 2*hs_755eb_depth/5} ${-shoulder_to_elbow - 0.02}" />
         </collision>
         <xacro:inertial_matrix_bis mass="0.1" />
@@ -182,6 +182,6 @@
         <parent link="base_link" />
         <child link="robot_base_cylinder" />
-        <axis xyz="0 0 1" />
-        <origin xyz="0 0.021 0" />
+        <axis xyz="0 0 -1" />
+        <origin xyz="0 0.021 0" rpy="0 0 ${PI}" />
         <limit effort="10" velocity="1" lower="${-PI}" upper="${PI}" />
         <dynamics damping="0" friction="0" />
@@ -196,6 +196,6 @@
         <parent link="robot_base_top_box" />
         <child link="shoulder" />
-        <axis xyz="1 0 0" />
-        <origin xyz="0 -0.015 0.071" />
+        <axis xyz="1 0 0"/>
+        <origin xyz="0 0.015 0.071"  rpy="0 0 0" />
         <limit effort="10" velocity="1" lower="0" upper="${PI}" />
         <dynamics damping="10" friction="0.7" />
@@ -213,5 +213,5 @@
         <child link="wrist" />
         <axis xyz="1 0 0" />
-        <origin xyz="0 ${-tube_length - hs_645_depth + 0.003} 0" rpy="0 0 ${PI}"/>
+        <origin xyz="0 ${tube_length + hs_645_depth - 0.003} 0" rpy="0 0 0"/>
         <limit effort="10" velocity="1" lower="${-PI/2}" upper="${PI/2}" />
         <dynamics damping="10" friction="0.7" />

Commit message: Solved issues related to the model

File: urdf/lynxmotion_al5d.gazebo.xacro (robot description, xacro)
@@ -1,8 +1,8 @@
 <?xml version="1.0" ?>
 <robot name="lynxmotion_al5d" xmlns:xacro="http://www.ros.org/wiki/xacro" xmlns:sensor="http://playerstage.sourceforge.net/gazebo/xmlschema/#sensor" xmlns:controller="http://playerstage.sourceforge.net/gazebo/xmlschema/#controller" xmlns:interface="http://playerstage.sourceforge.net/gazebo/xmlschema/#interface">
-<!-- This file has been created specifically to run with Gazebo since this requires a specific link named world for the robot to stick to the map -->
     <xacro:include filename="$(find lynxmotion_al5d_description)/urdf/lynxmotion_al5d_properties.urdf.xacro" />
     <!-- Base link comprising the board behind the robot and the cylinder at its bottom -->
     <link name="world" />
+    <gazebo reference="world" />
     <link name="robot_support">
         <visual>
@@ -18,5 +18,5 @@
             <origin rpy="0 0 0" xyz="0 0 0" />
         </collision>
-        <xacro:inertial_matrix mass="1" ixx="3.6565e-7" ixy="-3.72e-9" ixz="1e-6" iyy="9.404e-8" iyz="4.375e-8" izz="4.1776e-7" xyz="0.000585 0.0602746 0.0170628" />
+        <xacro:inertial_matrix mass="0.133" ixx="3.6565e-7" ixy="-3.72e-9" ixz="1e-6" iyy="9.404e-8" iyz="4.375e-8" izz="4.1776e-7" xyz="0.000585 0.0602746 0.0170628" />
     </link>
     <gazebo reference="robot_support" />
@@ -34,5 +34,5 @@
             <origin rpy="0 0 0" xyz="0 -0.021165 0" />
         </collision>
-        <xacro:inertial_matrix_bis mass="0.01" />
+        <xacro:inertial_matrix_bis mass="0.042" />
     </link>
     <gazebo reference="robot_base_cylinder" />
@@ -42,5 +42,5 @@
                 <mesh filename="package://lynxmotion_al5d_description/meshes/robot_parts/top_box.dae" />
             </geometry>
-            <origin xyz="-0.007 0.024 0" rpy="0 0 ${PI}" />
+            <origin xyz="0.007 -0.024 0" rpy="0 0 0" />
         </visual>
         <collision>
@@ -48,7 +48,7 @@
                 <mesh filename="package://lynxmotion_al5d_description/meshes/robot_parts/top_box.dae" />
             </geometry>
-            <origin xyz="-0.007 0.024 0" rpy="0 0 0" />
-        </collision>
-        <xacro:inertial_matrix_bis mass="0.6" />
+            <origin xyz="0.007 -0.024 0" rpy="0 0 0" />
+        </collision>
+        <xacro:inertial_matrix_bis mass="0.184" />
     </link>
     <gazebo reference="robot_base_top_box" />
@@ -66,5 +66,5 @@
             <origin rpy="${-5*PI/8} 0 0" xyz="0 -0.0625 0.036" />
         </collision>
-        <xacro:inertial_matrix_bis mass="0.1" />
+        <xacro:inertial_matrix_bis mass="0.095" />
     </link>
     <gazebo reference="shoulder" />
@@ -80,7 +80,7 @@
                 <mesh filename="package://lynxmotion_al5d_description/meshes/robot_parts/arm.dae" />
             </geometry>
-            <origin rpy="${-PI-0.895} 0 0" xyz="0 ${-tube_length + 2*hs_755eb_depth/5} ${-shoulder_to_elbow - 0.02}" />
-        </collision>
-        <xacro:inertial_matrix_bis mass="0.05" />
+            <origin rpy="${-PI-0.895} 0 0" xyz="0 ${tube_length - 2*hs_755eb_depth/5} ${shoulder_to_elbow + 0.02}" />
+        </collision>
+        <xacro:inertial_matrix_bis mass="0.1" />
     </link>
     <gazebo reference="arm" />
@@ -98,5 +98,5 @@
             <origin rpy="${PI} 0 0" xyz="0.005 -0.165 0.067" />
         </collision>
-        <xacro:inertial_matrix_bis mass="0" />
+        <xacro:inertial_matrix_bis mass="0.055" />
     </link>
     <gazebo reference="wrist" />
@@ -114,5 +114,5 @@
             <origin rpy="${PI/2} 0 ${-PI/2}" xyz="0 -0.021 -0.005" />
         </collision>
-        <xacro:inertial_matrix_bis mass="0" />
+        <xacro:inertial_matrix_bis mass="0.042" />
     </link>
     <gazebo reference="gripper" />
@@ -130,5 +130,5 @@
             <origin rpy="${PI/2} 0 ${-PI/2}" xyz="0.003 -0.012 0" />
         </collision>
-        <xacro:inertial_matrix_bis mass="0" />
+        <xacro:inertial_matrix_bis mass="0.0006" />
     </link>
     <gazebo reference="left_finger" />
@@ -146,5 +146,5 @@
             <origin rpy="${PI/2} 0 ${-PI/2}" xyz="-0.003 -0.012 0" />
         </collision>
-        <xacro:inertial_matrix_bis mass="0" />
+        <xacro:inertial_matrix_bis mass="0.0006" />
     </link>
     <gazebo reference="right_finger" />
@@ -186,5 +186,5 @@
         <dynamics damping="10" friction="0.7" />
     </joint>
-     <joint name="Joint1" type="revolute">
+   <joint name="Joint1" type="revolute">
         <parent link="robot_support" />
         <child link="robot_base_cylinder" />
@@ -192,5 +192,4 @@
         <origin xyz="0 0.021 0" rpy="0 0 ${PI}" />
         <limit effort="10" velocity="1" lower="${-PI}" upper="${PI}" />
-        <dynamics damping="0" friction="0" />
         <dynamics damping="10" friction="0.7" />
     </joint>
@@ -243,5 +242,5 @@
         <child link="right_finger" />
         <origin xyz="0 -0.01 0" />
-        <limit effort="10" velocity="0.005" lower="0" upper="${gripper_base_width/2}" />
+        <limit effort="10" velocity="0.001" lower="0" upper="${gripper_base_width/2}" />
         <mimic joint="Gripper" multiplier="-1" />
         <dynamics damping="10" friction="0.7" />
@@ -281,5 +280,5 @@
                 <alwaysOn>true</alwaysOn>
                 <updateRate>1.0</updateRate>
-                <cameraName>camera</cameraName>
+                <cameraName>al5d_external_vision</cameraName>
                 <imageTopicName>image_raw</imageTopicName>
                 <cameraInfoTopicName>camera_info</cameraInfoTopicName>

File: urdf/lynxmotion_al5d.xacro (robot description, xacro)
@@ -46,5 +46,5 @@
                 <mesh filename="package://lynxmotion_al5d_description/meshes/robot_parts/top_box.dae" />
             </geometry>
-            <origin xyz="-0.007 0.024 0" rpy="0 0 0" />
+            <origin xyz="-0.007 0.024 0" rpy="0 0 ${PI}" />
         </collision>
         <xacro:inertial_matrix_bis mass="0.184" />
@@ -78,5 +78,5 @@
                 <mesh filename="package://lynxmotion_al5d_description/meshes/robot_parts/arm.dae" />
             </geometry>
-            <origin rpy="${-PI-0.895} 0 0" xyz="0 ${-tube_length + 2*hs_755eb_depth/5} ${-shoulder_to_elbow - 0.02}" />
+            <origin rpy="${-PI-0.895} 0 0" xyz="0 ${tube_length - 2*hs_755eb_depth/5} ${shoulder_to_elbow + 0.02}" />
         </collision>
         <xacro:inertial_matrix_bis mass="0.1" />
@@ -185,5 +185,4 @@
         <origin xyz="0 0.021 0" rpy="0 0 ${PI}" />
         <limit effort="10" velocity="1" lower="${-PI}" upper="${PI}" />
-        <dynamics damping="0" friction="0" />
         <dynamics damping="10" friction="0.7" />
     </joint>
