Commit message: Removed the necessity to have a 7th joint value passed for the topic

File: urdf/lynxmotion_al5d.gazebo.xacro (robot description, xacro)
@@ -231,16 +231,16 @@
         <dynamics damping="10" friction="0.7" />
     </joint>
-   <joint name="Gripper" type="prismatic">
+    <joint name="Gripper" type="prismatic">
+        <parent link="gripper" />
+        <child link="right_finger" />
+        <origin xyz="0 -0.01 0" />
+        <limit effort="10" velocity="0.01" lower="0" upper="${gripper_base_width/2}" />
+        <dynamics damping="10" friction="0.7" />
+    </joint>
+   <joint name="GripperBis" type="prismatic">
         <parent link="gripper" />
         <child link="left_finger" />
         <origin xyz="0 -0.01 0" />
-        <limit effort="10" velocity="0.005" upper="0" lower="${-gripper_base_width/2}" />
-        <dynamics damping="10" friction="0.7" />
-    </joint>
-   <joint name="GripperBis" type="prismatic">
-        <parent link="gripper" />
-        <child link="right_finger" />
-        <origin xyz="0 -0.01 0" />
-        <limit effort="10" velocity="0.001" lower="0" upper="${gripper_base_width/2}" />
+        <limit effort="10" velocity="0.01" upper="0" lower="${-gripper_base_width/2}" />
         <mimic joint="Gripper" multiplier="-1" />
         <dynamics damping="10" friction="0.7" />
@@ -252,7 +252,6 @@
     <xacro:transmission_block joint_name="Joint4"/>
     <xacro:transmission_block joint_name="Joint5"/>
-    <xacro:transmission_block_finger joint_name="Gripper"/>
-    <xacro:transmission_block_finger joint_name="GripperBis"/>
-      <!-- ros_control plugin -->
+    <xacro:transmission_block joint_name="Gripper"/>
+    <!-- ros_control plugin -->
     <gazebo>
         <plugin name="gazebo_ros_control" filename="libgazebo_ros_control.so">
@@ -261,4 +260,7 @@
         </plugin>
     </gazebo>
+    <xacro:mimic_joint_plugin_gazebo name_prefix="gripper_"
+    parent_joint="Gripper" mimic_joint="GripperBis"
+    has_pid="true" multiplier="-1.0" max_effort="10.0" />
     <gazebo reference="camera_link">
         <sensor name="external_camera" type="camera">

File: urdf/lynxmotion_al5d.xacro (robot description, xacro)
@@ -3,5 +3,7 @@
     <xacro:include filename="$(find lynxmotion_al5d_description)/urdf/lynxmotion_al5d_properties.urdf.xacro" />
     <!-- Base link comprising the board behind the robot and the cylinder at its bottom -->
-    <link name="base_link">
+    <link name="world" />
+    <gazebo reference="world" />
+    <link name="robot_support">
         <visual>
             <geometry>
@@ -18,5 +20,5 @@
         <xacro:inertial_matrix mass="0.133" ixx="3.6565e-7" ixy="-3.72e-9" ixz="1e-6" iyy="9.404e-8" iyz="4.375e-8" izz="4.1776e-7" xyz="0.000585 0.0602746 0.0170628" />
     </link>
-    <gazebo reference="base_link" />
+    <gazebo reference="robot_support" />
     <link name="robot_base_cylinder">
         <visual>
@@ -40,5 +42,5 @@
                 <mesh filename="package://lynxmotion_al5d_description/meshes/robot_parts/top_box.dae" />
             </geometry>
-            <origin xyz="-0.007 0.024 0" rpy="0 0 ${PI}" />
+            <origin xyz="0.007 -0.024 0" rpy="0 0 0" />
         </visual>
         <collision>
@@ -46,5 +48,5 @@
                 <mesh filename="package://lynxmotion_al5d_description/meshes/robot_parts/top_box.dae" />
             </geometry>
-            <origin xyz="-0.007 0.024 0" rpy="0 0 ${PI}" />
+            <origin xyz="0.007 -0.024 0" rpy="0 0 0" />
         </collision>
         <xacro:inertial_matrix_bis mass="0.184" />
@@ -120,5 +122,5 @@
                 <mesh filename="package://lynxmotion_al5d_description/meshes/robot_parts/finger_left.dae" />
             </geometry>
-            <origin rpy="${PI/2} 0 ${-PI/2}" xyz="0.003 -0.012 0" />
+            <origin rpy="${PI/2} 0 ${-PI/2}" xyz="0 -0.012 0" />
         </visual>
         <collision>
@@ -126,5 +128,5 @@
                 <mesh filename="package://lynxmotion_al5d_description/meshes/robot_parts/finger_left.dae" />
             </geometry>
-            <origin rpy="${PI/2} 0 ${-PI/2}" xyz="0.003 -0.012 0" />
+            <origin rpy="${PI/2} 0 ${-PI/2}" xyz="0 -0.012 0" />
         </collision>
         <xacro:inertial_matrix_bis mass="0.0006" />
@@ -136,5 +138,5 @@
                 <mesh filename="package://lynxmotion_al5d_description/meshes/robot_parts/finger_right.dae" />
             </geometry>
-            <origin rpy="${PI/2} 0 ${-PI/2}" xyz="-0.003 -0.012 0" />
+            <origin rpy="${PI/2} 0 ${-PI/2}" xyz="0 -0.012 0" />
         </visual>
         <collision>
@@ -173,17 +175,20 @@
     </sensor>
     <!-- Adding joints -->
+    <joint name="world_to_robot" type="fixed">
+        <parent link="world" />
+        <child link="robot_support" />
+    </joint>
     <joint name="camera_joint" type="fixed">
-        <parent link="base_link" />
+        <parent link="world" />
         <child link="camera_link" />
         <origin xyz="0 -0.35 0" />
-        <dynamics damping="10" friction="0.7" />
-    </joint>
-    <joint name="Joint1" type="revolute">
-        <parent link="base_link" />
+    </joint>
+   <joint name="Joint1" type="revolute">
+        <parent link="robot_support" />
         <child link="robot_base_cylinder" />
         <axis xyz="0 0 -1" />
         <origin xyz="0 0.021 0" rpy="0 0 ${PI}" />
         <limit effort="10" velocity="1" lower="${-PI}" upper="${PI}" />
-        <dynamics damping="10" friction="0.7" />
+        <dynamics damping="50" friction="1" />
     </joint>
     <joint name="base_to_cylinder" type="fixed">
@@ -198,5 +203,5 @@
         <origin xyz="0 0.015 0.071"  rpy="0 0 0" />
         <limit effort="10" velocity="1" lower="0" upper="${PI}" />
-        <dynamics damping="10" friction="0.7" />
+        <dynamics damping="50" friction="1" />
     </joint>
     <joint name="Joint3" type="revolute">
@@ -206,5 +211,5 @@
         <origin xyz="0 ${shoulder_to_elbow} 0" />
         <limit effort="10" velocity="1" lower="${-PI/2}" upper="${PI/2}" />
-        <dynamics damping="10" friction="0.7" />
+        <dynamics damping="50" friction="1" />
     </joint>
     <joint name="Joint4" type="revolute">
@@ -214,5 +219,5 @@
         <origin xyz="0 ${tube_length + hs_645_depth - 0.003} 0" rpy="0 0 0"/>
         <limit effort="10" velocity="1" lower="${-PI/2}" upper="${PI/2}" />
-        <dynamics damping="10" friction="0.7" />
+        <dynamics damping="50" friction="1" />
     </joint>
    <joint name="Joint5" type="revolute">
@@ -224,16 +229,16 @@
         <dynamics damping="10" friction="0.7" />
     </joint>
-   <joint name="Gripper" type="prismatic">
+    <joint name="Gripper" type="prismatic">
+        <parent link="gripper" />
+        <child link="right_finger" />
+        <origin xyz="0 -0.01 0" />
+        <limit effort="10" velocity="0.01" lower="0" upper="${gripper_base_width/2}" />
+        <dynamics damping="10" friction="0.7" />
+    </joint>
+   <joint name="GripperBis" type="prismatic">
         <parent link="gripper" />
         <child link="left_finger" />
         <origin xyz="0 -0.01 0" />
-        <limit effort="10" velocity="0.005" upper="0" lower="${-gripper_base_width/2}" />
-        <dynamics damping="10" friction="0.7" />
-    </joint>
-   <joint name="GripperBis" type="prismatic">
-        <parent link="gripper" />
-        <child link="right_finger" />
-        <origin xyz="0 -0.01 0" />
-        <limit effort="10" velocity="0.001" lower="0" upper="${gripper_base_width/2}" />
+        <limit effort="10" velocity="0.01" upper="0" lower="${-gripper_base_width/2}" />
         <mimic joint="Gripper" multiplier="-1" />
         <dynamics damping="10" friction="0.7" />
@@ -245,7 +250,6 @@
     <xacro:transmission_block joint_name="Joint4"/>
     <xacro:transmission_block joint_name="Joint5"/>
-    <xacro:transmission_block_finger joint_name="Gripper"/>
-    <xacro:transmission_block_finger joint_name="GripperBis"/>
-      <!-- ros_control plugin -->
+    <xacro:transmission_block joint_name="Gripper"/>
+    <!-- ros_control plugin -->
     <gazebo>
         <plugin name="gazebo_ros_control" filename="libgazebo_ros_control.so">
@@ -254,4 +258,7 @@
         </plugin>
     </gazebo>
+    <xacro:mimic_joint_plugin_gazebo name_prefix="gripper_"
+    parent_joint="Gripper" mimic_joint="GripperBis"
+    has_pid="true" multiplier="-1.0" max_effort="10.0" />
     <gazebo reference="camera_link">
         <sensor name="external_camera" type="camera">
@@ -273,5 +280,5 @@
                 <alwaysOn>true</alwaysOn>
                 <updateRate>1.0</updateRate>
-                <cameraName>camera</cameraName>
+                <cameraName>al5d_external_vision</cameraName>
                 <imageTopicName>image_raw</imageTopicName>
                 <cameraInfoTopicName>camera_info</cameraInfoTopicName>

File: urdf/lynxmotion_al5d_properties.urdf.xacro (robot description, xacro)
@@ -90,4 +90,23 @@
       </inertial>
    </xacro:macro>
+   <!-- Copied from https://github.com/mintar/mimic_joint_gazebo_tutorial/blob/kinetic/urdf/mimic_joint_gazebo_tutorial.urdf.xacro -->
+   <xacro:macro name="mimic_joint_plugin_gazebo" params="name_prefix parent_joint mimic_joint has_pid:=false multiplier:=1.0 offset:=0 sensitiveness:=0.0 max_effort:=1.0 robot_namespace:=''">
+    <gazebo>
+      <plugin name="${name_prefix}mimic_joint_plugin" filename="libroboticsgroup_gazebo_mimic_joint_plugin.so">
+        <joint>${parent_joint}</joint>
+        <mimicJoint>${mimic_joint}</mimicJoint>
+        <xacro:if value="${has_pid}">
+          <hasPID />
+        </xacro:if>
+        <multiplier>${multiplier}</multiplier>
+        <offset>${offset}</offset>
+        <sensitiveness>${sensitiveness}</sensitiveness>
+        <maxEffort>${max_effort}</maxEffort>
+        <xacro:unless value="${robot_namespace == ''}">
+          <robotNamespace>($robot_namespace)</robotNamespace>
+        </xacro:unless>
+      </plugin>
+    </gazebo>
+  </xacro:macro>
     <xacro:macro name="transmission_block" params="joint_name">
         <transmission name="tran1">
@@ -97,17 +116,4 @@
             </joint>
             <actuator name="motor1">
-                <hardwareInterface>hardware_interface/PositionJointInterface</hardwareInterface>
-                <mechanicalReduction>1</mechanicalReduction>
-            </actuator>
-        </transmission>
-   </xacro:macro>
-    <xacro:macro name="transmission_block_finger" params="joint_name">
-        <transmission name="tran2">
-            <type>transmission_interface/SimpleTransmission</type>
-            <joint name="${joint_name}">
-                <hardwareInterface>hardware_interface/PositionJointInterface</hardwareInterface>
-            </joint>
-            <actuator name="motor2">
-                <hardwareInterface>hardware_interface/PositionJointInterface</hardwareInterface>
                 <mechanicalReduction>1</mechanicalReduction>
             </actuator>
