Commit message: Added a camera model to the robot description

File: urdf/lynxmotion_al5d.xacro (robot description, xacro)
@@ -169,5 +169,45 @@
         <xacro:inertial_matrix_box width="${finger_width}" height="${finger_height}" depth="${finger_depth}" mass="${finger_mass}" />
     </link>
+<xacro:property name="camera_support_depth" value="0.25" />
+    <xacro:property name="camera_support_size" value="0.003" />
+    <xacro:property name="camera_support_big_size" value="0.5" />
+    <xacro:property name="camera_support_to_base" value="0.06" />
+    <link name="camera_link">
+        <visual name="stick">
+            <geometry>
+                <box size="${camera_support_size} ${camera_support_size} ${camera_support_depth}" />
+            </geometry>
+            <origin rpy="0 0 0" xyz="0 ${camera_support_to_base} ${camera_support_depth/2}" />
+            <material name="BlueGrey" />
+        </visual>
+        <visual name="support">
+            <geometry>
+                <box size="${camera_support_big_size} ${camera_support_big_size + camera_support_to_base} ${camera_support_size}" />
+            </geometry>
+            <origin rpy="0 0 0" xyz="0 ${-camera_support_big_size/2} ${camera_support_depth - camera_support_size/2}" />
+            <material name="BlueGrey" />
+        </visual>
+        <collision name="support">
+            <geometry>
+                <box size="${camera_support_big_size} ${camera_support_big_size + camera_support_to_base} ${camera_support_size}" />
+            </geometry>
+            <origin rpy="0 0 0" xyz="0 ${-camera_support_big_size/2} ${camera_support_depth - camera_support_size/2}" />
+            <material name="BlueGrey" />
+        </collision>
+        <xacro:inertial_matrix_box mass="${camera_support_mass}" width="${camera_support_big_size}" height="${camera_support_big_size + camera_support_to_base}" depth="${camera_support_size}" />
+    </link>
+    <!-- Adding a camera sensor to the model -->
+    <sensor name="robot_camera" update_rate="1">
+        <parent link="camera_link" />
+        <origin xyz="0 0 0" rpy="0 0 0" />
+        <camera>
+            <image width="640" height="480" hfov="${PI/2}" format="RGB8" near="${camera_support_depth}" far="${camera_support_depth}" />
+        </camera>
+    </sensor>
     <!-- Adding joints -->
+    <joint name="camera_support_joint" type="fixed">
+        <parent link="base_link" />
+        <child link="camera_link" />
+    </joint>
     <joint name="shoulder_elbow_roll" type="revolute">
         <parent link="base_link" />

File: urdf/lynxmotion_al5d_properties.urdf.xacro (robot description, xacro)
@@ -13,4 +13,7 @@
     <material name="Silver">
         <color rgba="0.8 0.8 0.8 1" />
+    </material>
+    <material name="BlueGrey">
+        <color rgba="1 87 155 1" />
     </material>
     <!-- Setting properties to be used in the program -->
@@ -53,4 +56,9 @@
     <xacro:property name="wrist_cylinder_length" value="0.005" />
     <xacro:property name="wrist_cylinder_radius" value="0.01" />
+    <xacro:property name="camera_support_depth" value="0.5" />
+    <xacro:property name="camera_support_size" value="0.01" />
+    <xacro:property name="camera_support_big_size" value="0.5" />
+    <xacro:property name="camera_support_to_base" value="0.1" />
+    <xacro:property name="camera_support_mass" value="0.2" />
     <!-- Adding macros for the inertial matrixes -->
     <xacro:macro name="inertial_matrix_cylinder" params="mass height radius">

Commit message: Added the 3D models to the URDF file

File: urdf/lynxmotion_al5d.xacro (robot description, xacro)
@@ -4,17 +4,9 @@
     <!-- Base link comprising the board behind the robot and the cylinder at its bottom -->
     <link name="base_link">
-        <visual name="board">
-            <geometry>
-                <box size="${board_size} ${board_size} ${board_height}" />
-            </geometry>
-            <origin rpy="0 0 0" xyz="0 ${base_radius + board_size/2} 0" />
-            <material name="Green" />
-        </visual>
-        <visual name="base">
-            <geometry>
-                <cylinder length="${base_height}" radius="${base_radius}" />
-            </geometry>
-            <origin rpy="0 0 0" xyz="0 0 ${base_height/2}" />
-            <material name="Black" />
+        <visual>
+            <geometry>
+                <mesh filename="package://lynxmotion_al5d_description/meshes/robot_parts/base_link.dae" />
+            </geometry>
+            <origin rpy="0 0 0" xyz="0 0 0" />
         </visual>
         <collision>
@@ -30,8 +22,7 @@
         <visual>
             <geometry>
-                <box size="${top_box_width} ${top_box_height} ${top_box_depth}" />
-            </geometry>
-            <origin rpy="0 0 0" xyz="0 ${-top_box_height + base_radius} ${top_box_depth/2}" />
-            <material name="Black" />
+                <mesh filename="package://lynxmotion_al5d_description/meshes/robot_parts/top_box.dae" />
+            </geometry>
+            <origin rpy="0 0 0" xyz="0.01 ${-top_box_height + base_radius} 0" />
         </visual>
         <collision>
@@ -47,8 +38,6 @@
         <visual>
             <geometry>
-                <box size="${shoulder_width} ${shoulder_height} ${shoulder_to_elbow}" />
-            </geometry>
-            <origin rpy="0 0 0" xyz="0 0 ${shoulder_to_elbow/2}" />
-            <material name="Silver" />
+                <mesh filename="package://lynxmotion_al5d_description/meshes/robot_parts/shoulder.dae" />
+            </geometry>
         </visual>
         <collision>
@@ -62,5 +51,11 @@
     <!-- Link representing the elbow of the robot which ends at the beginning of the wrist -->
     <link name="elbow">
-        <visual name="before_arm">
+        <visual>
+            <geometry>
+                <mesh filename="package://lynxmotion_al5d_description/meshes/robot_parts/arm.dae" />
+            </geometry>
+            <origin xyz="0 -0.2 0" rpy="0 0 0" />
+        </visual>
+        <!--<visual name="before_arm">
             <geometry>
                 <cylinder length="${tube_length}" radius="${tube_radius}" />
@@ -82,5 +77,5 @@
             <material name="Black" />
             <origin rpy="${PI/2} 0 0" xyz="0 ${-tube_length} 0" />
-        </visual>
+        </visual> -->
         <collision>
             <geometry>
@@ -95,4 +90,9 @@
         <visual>
             <geometry>
+                <mesh filename="package://lynxmotion_al5d_description/meshes/robot_parts/wrist.dae" />
+            </geometry>
+        </visual>
+        <!-- <visual>
+            <geometry>
                 <box size="${hs_225_width} ${hs_225_height} ${hs_225_depth}" />
             </geometry>
@@ -106,5 +106,5 @@
             <origin rpy="${PI/2} 0 0" xyz="0 ${-(hs_225_depth/2 + wrist_cylinder_length/2)} 0" />
             <material name="Silver" />
-        </visual>
+        </visual> -->
         <collision>
             <geometry>
@@ -119,9 +119,14 @@
         <visual>
             <geometry>
+                <mesh filename="package://lynxmotion_al5d_description/meshes/robot_parts/gripper_base.dae" />
+            </geometry>
+        </visual>
+        <!-- <visual>
+            <geometry>
                 <box size="${gripper_base_width} ${gripper_base_height} ${gripper_base_depth}" />
             </geometry>
             <material name="Black" />
             <origin rpy="${PI/2} 0 0" xyz="0 0 0" />
-        </visual>
+        </visual>-->
         <collision>
             <geometry>
@@ -135,4 +140,9 @@
     <link name="left_finger">
         <visual>
+            <geometry>
+                <mesh filename="package://lynxmotion_al5d_description/meshes/robot_parts/finger_left.dae" />
+            </geometry>
+        </visual>
+        <!-- <visual>
             <geometry>
                 <box size="${finger_width} ${finger_height} ${finger_depth}" />
@@ -142,5 +152,5 @@
                 <color rgba="0.8 0.8 0.8 1" />
             </material>
-        </visual>
+        </visual>-->
         <collision>
             <geometry>
@@ -153,4 +163,9 @@
     <link name="right_finger">
         <visual>
+            <geometry>
+                <mesh filename="package://lynxmotion_al5d_description/meshes/robot_parts/finger_right.dae" />
+            </geometry>
+        </visual>
+        <!--<visual>
             <geometry>
                 <box size="${finger_width} ${finger_height} ${finger_depth}" />
@@ -160,5 +175,5 @@
                 <color rgba="0.8 0.8 0.8 1" />
             </material>
-        </visual>
+        </visual> -->
         <collision>
             <geometry>
@@ -213,5 +228,5 @@
         <parent link="base_link" />
         <child link="top_box" />
-        <origin xyz="0 0 ${base_height}" />
+        <origin xyz="0 0 0" />
         <axis xyz="1 0 0" />
         <limit effort="10" velocity="1" lower="${-PI/2}" upper="${PI/2}" />
@@ -229,5 +244,4 @@
         <parent link="shoulder" />
         <child link="elbow" />
-        <origin xyz="0 0 ${base_height + shoulder_to_elbow - hs_755eb_height}" />
         <axis xyz="1 0 0" />
         <limit effort="10" velocity="1" lower="${-PI/2}" upper="${PI/2}" />

Commit message: Setting a branch for updated simulator

File: urdf/lynxmotion_al5d.xacro (robot description, xacro)
@@ -4,9 +4,17 @@
     <!-- Base link comprising the board behind the robot and the cylinder at its bottom -->
     <link name="base_link">
-        <visual>
-            <geometry>
-                <mesh filename="package://lynxmotion_al5d_description/meshes/robot_parts/base_link.dae" />
-            </geometry>
-            <origin rpy="0 0 0" xyz="0 0 0" />
+        <visual name="board">
+            <geometry>
+                <box size="${board_size} ${board_size} ${board_height}" />
+            </geometry>
+            <origin rpy="0 0 0" xyz="0 ${base_radius + board_size/2} 0" />
+            <material name="Green" />
+        </visual>
+        <visual name="base">
+            <geometry>
+                <cylinder length="${base_height}" radius="${base_radius}" />
+            </geometry>
+            <origin rpy="0 0 0" xyz="0 0 ${base_height/2}" />
+            <material name="Black" />
         </visual>
         <collision>
@@ -22,7 +30,8 @@
         <visual>
             <geometry>
-                <mesh filename="package://lynxmotion_al5d_description/meshes/robot_parts/top_box.dae" />
-            </geometry>
-            <origin rpy="0 0 0" xyz="0.01 ${-top_box_height + base_radius} 0" />
+                <box size="${top_box_width} ${top_box_height} ${top_box_depth}" />
+            </geometry>
+            <origin rpy="0 0 0" xyz="0 ${-top_box_height + base_radius} ${top_box_depth/2}" />
+            <material name="Black" />
         </visual>
         <collision>
@@ -38,6 +47,8 @@
         <visual>
             <geometry>
-                <mesh filename="package://lynxmotion_al5d_description/meshes/robot_parts/shoulder.dae" />
-            </geometry>
+                <box size="${shoulder_width} ${shoulder_height} ${shoulder_to_elbow}" />
+            </geometry>
+            <origin rpy="0 0 0" xyz="0 0 ${shoulder_to_elbow/2}" />
+            <material name="Silver" />
         </visual>
         <collision>
@@ -51,11 +62,5 @@
     <!-- Link representing the elbow of the robot which ends at the beginning of the wrist -->
     <link name="elbow">
-        <visual>
-            <geometry>
-                <mesh filename="package://lynxmotion_al5d_description/meshes/robot_parts/arm.dae" />
-            </geometry>
-            <origin xyz="0 -0.2 0" rpy="0 0 0" />
-        </visual>
-        <!--<visual name="before_arm">
+        <visual name="before_arm">
             <geometry>
                 <cylinder length="${tube_length}" radius="${tube_radius}" />
@@ -77,5 +82,5 @@
             <material name="Black" />
             <origin rpy="${PI/2} 0 0" xyz="0 ${-tube_length} 0" />
-        </visual> -->
+        </visual>
         <collision>
             <geometry>
@@ -90,9 +95,4 @@
         <visual>
             <geometry>
-                <mesh filename="package://lynxmotion_al5d_description/meshes/robot_parts/wrist.dae" />
-            </geometry>
-        </visual>
-        <!-- <visual>
-            <geometry>
                 <box size="${hs_225_width} ${hs_225_height} ${hs_225_depth}" />
             </geometry>
@@ -106,5 +106,5 @@
             <origin rpy="${PI/2} 0 0" xyz="0 ${-(hs_225_depth/2 + wrist_cylinder_length/2)} 0" />
             <material name="Silver" />
-        </visual> -->
+        </visual>
         <collision>
             <geometry>
@@ -119,14 +119,9 @@
         <visual>
             <geometry>
-                <mesh filename="package://lynxmotion_al5d_description/meshes/robot_parts/gripper_base.dae" />
-            </geometry>
-        </visual>
-        <!-- <visual>
-            <geometry>
                 <box size="${gripper_base_width} ${gripper_base_height} ${gripper_base_depth}" />
             </geometry>
             <material name="Black" />
             <origin rpy="${PI/2} 0 0" xyz="0 0 0" />
-        </visual>-->
+        </visual>
         <collision>
             <geometry>
@@ -140,9 +135,4 @@
     <link name="left_finger">
         <visual>
-            <geometry>
-                <mesh filename="package://lynxmotion_al5d_description/meshes/robot_parts/finger_left.dae" />
-            </geometry>
-        </visual>
-        <!-- <visual>
             <geometry>
                 <box size="${finger_width} ${finger_height} ${finger_depth}" />
@@ -152,5 +142,5 @@
                 <color rgba="0.8 0.8 0.8 1" />
             </material>
-        </visual>-->
+        </visual>
         <collision>
             <geometry>
@@ -163,9 +153,4 @@
     <link name="right_finger">
         <visual>
-            <geometry>
-                <mesh filename="package://lynxmotion_al5d_description/meshes/robot_parts/finger_right.dae" />
-            </geometry>
-        </visual>
-        <!--<visual>
             <geometry>
                 <box size="${finger_width} ${finger_height} ${finger_depth}" />
@@ -175,5 +160,5 @@
                 <color rgba="0.8 0.8 0.8 1" />
             </material>
-        </visual> -->
+        </visual>
         <collision>
             <geometry>
@@ -228,5 +213,5 @@
         <parent link="base_link" />
         <child link="top_box" />
-        <origin xyz="0 0 0" />
+        <origin xyz="0 0 ${base_height}" />
         <axis xyz="1 0 0" />
         <limit effort="10" velocity="1" lower="${-PI/2}" upper="${PI/2}" />
@@ -244,4 +229,5 @@
         <parent link="shoulder" />
         <child link="elbow" />
+        <origin xyz="0 0 ${base_height + shoulder_to_elbow - hs_755eb_height}" />
         <axis xyz="1 0 0" />
         <limit effort="10" velocity="1" lower="${-PI/2}" upper="${PI/2}" />
