Commit message: Fully integrated the 3D meshes to the robot model. Rotations movements fixed

File: urdf/lynxmotion_al5d.xacro (robot description, xacro)
@@ -3,202 +3,97 @@
     <xacro:include filename="$(find lynxmotion_al5d_description)/urdf/lynxmotion_al5d_properties.urdf.xacro" />
     <!-- Base link comprising the board behind the robot and the cylinder at its bottom -->
-    <link name="base_link">
-        <visual name="board">
-            <geometry>
-                <box size="${board_size} ${board_size} ${board_height}" />
-            </geometry>
-            <origin rpy="0 0 0" xyz="0 ${base_radius + board_size/2} 0" />
-            <material name="Green" />
-        </visual>
-        <visual name="base">
-            <geometry>
-                <cylinder length="${base_height}" radius="${base_radius}" />
-            </geometry>
-            <origin rpy="0 0 0" xyz="0 0 ${base_height/2}" />
-            <material name="Black" />
-        </visual>
-        <collision>
-            <geometry>
-                <cylinder length="${base_height}" radius="${base_radius}" />
-            </geometry>
-            <origin rpy="0 0 0" xyz="0 0 0" />
-        </collision>
-        <xacro:inertial_matrix_cylinder height="${base_height}" radius="${base_radius}" mass="${base_mass}" />
-    </link>
-    <!-- Link representing the black box on top of the cylinder that rotates around the z axis in the link's frame of reference -->
-    <link name="top_box">
-        <visual>
-            <geometry>
-                <box size="${top_box_width} ${top_box_height} ${top_box_depth}" />
-            </geometry>
-            <origin rpy="0 0 0" xyz="0 ${-top_box_height + base_radius} ${top_box_depth/2}" />
-            <material name="Black" />
-        </visual>
-        <collision>
-            <geometry>
-                <box size="${top_box_width} ${top_box_height} ${top_box_depth}" />
-            </geometry>
-            <origin rpy="0 0 0" xyz="0 ${-top_box_height + base_radius} ${top_box_depth/2}" />
-        </collision>
-        <xacro:inertial_matrix_box height="${top_box_height}" width="${top_box_width}" depth="${top_box_depth}" mass="${top_box_mass}" />
-    </link>
-    <!-- Link representing the second link of the robot (i.e the shoulder) -->
+    <link name="world" />
+    <link name="robot_support">
+        <visual>
+            <geometry>
+                <mesh filename="package://lynxmotion_al5d_description/meshes/robot_parts/support.dae" />
+            </geometry>
+        </visual>
+        <xacro:inertial_matrix_cylinder mass="0.4" height="0.04" radius="0.04" />
+    </link>
+    <link name="robot_base_cylinder">
+        <visual>
+            <geometry>
+                <mesh filename="package://lynxmotion_al5d_description/meshes/robot_parts/rotation_cylinder.dae" />
+            </geometry>
+            <origin rpy="0 0 0" xyz="0 -0.021165 0" />
+        </visual>
+        <xacro:inertial_matrix_cylinder mass="0.05" height="0.004" radius="0.04" />
+    </link>
+    <link name="robot_base_top_box">
+        <visual>
+            <geometry>
+                <mesh filename="package://lynxmotion_al5d_description/meshes/robot_parts/top_box.dae" />
+            </geometry>
+            <origin xyz="0.007 -0.024 0" rpy="0 0 0" />
+        </visual>
+        <xacro:inertial_matrix_box mass="0.5" depth="0.03" height="0.04" width="0.06" />
+    </link>
     <link name="shoulder">
         <visual>
             <geometry>
-                <box size="${shoulder_width} ${shoulder_height} ${shoulder_to_elbow}" />
-            </geometry>
-            <origin rpy="0 0 0" xyz="0 0 ${shoulder_to_elbow/2}" />
-            <material name="Silver" />
-        </visual>
-        <collision>
-            <geometry>
-                <box size="${shoulder_width} ${shoulder_height} ${shoulder_to_elbow}" />
-            </geometry>
-            <origin rpy="0 0 0" xyz="0 0 ${shoulder_to_elbow/2}" />
-        </collision>
-        <xacro:inertial_matrix_box height="${shoulder_height}" width="${shoulder_width}" depth="${shoulder_to_elbow}" mass="${shoulder_mass}" />
-    </link>
-    <!-- Link representing the elbow of the robot which ends at the beginning of the wrist -->
-    <link name="elbow">
-        <visual name="before_arm">
-            <geometry>
-                <cylinder length="${tube_length}" radius="${tube_radius}" />
-            </geometry>
-            <material name="Silver" />
-            <origin rpy="${PI/2} 0 0" xyz="0 ${-tube_length/2} 0" />
-        </visual>
-        <visual name="hs-755eb">
-            <geometry>
-                <box size="${hs_755eb_width} ${hs_755eb_height} ${hs_755eb_depth}" />
-            </geometry>
-            <material name="Black" />
-            <origin rpy="0 0 0" xyz="0 0 0" />
-        </visual>
-        <visual name="hs-645">
-            <geometry>
-                <box size="${hs_645_width} ${hs_645_height} ${hs_645_depth}" />
-            </geometry>
-            <material name="Black" />
-            <origin rpy="${PI/2} 0 0" xyz="0 ${-tube_length} 0" />
-        </visual>
-        <collision>
-            <geometry>
-                <box size="${hs_755eb_width} ${hs_755eb_height} ${hs_755eb_depth}" />
-            </geometry>
-            <origin rpy="${PI/2} 0 0" xyz="0 ${-tube_length} 0" />
-        </collision>
-        <xacro:inertial_matrix_box height="${hs_755eb_height}" width="${hs_755eb_width}" depth="${hs_755eb_depth}" mass="${hs_755eb_mass}" />
-    </link>
-    <!-- Wrist of the robot -->
+                <mesh filename="package://lynxmotion_al5d_description/meshes/robot_parts/shoulder.dae" />
+            </geometry>
+            <origin rpy="${-PI/8} 0 0" xyz="0 -0.035 -0.06" />
+        </visual>
+        <xacro:inertial_matrix_box mass="0.5" depth="0.17" height="0.02" width="0.11" />
+    </link>
+    <link name="arm">
+        <visual>
+            <geometry>
+                <mesh filename="package://lynxmotion_al5d_description/meshes/robot_parts/arm.dae" />
+            </geometry>
+            <origin rpy="-0.895 0 0" xyz="0 ${-tube_length + 2*hs_755eb_depth/5} ${-shoulder_to_elbow - 0.02}" />
+        </visual>
+        <xacro:inertial_matrix_box mass="0.2" depth="0.03" height="0.07" width="0.05" />
+    </link>
     <link name="wrist">
         <visual>
             <geometry>
-                <box size="${hs_225_width} ${hs_225_height} ${hs_225_depth}" />
-            </geometry>
-            <origin rpy="${PI/2} 0 0" xyz="0 0 0" />
-            <material name="Black" />
-        </visual>
-        <visual name="wrist_cylinder">
-            <geometry>
-                <cylinder length="${wrist_cylinder_length}" radius="${wrist_cylinder_radius}" />
-            </geometry>
-            <origin rpy="${PI/2} 0 0" xyz="0 ${-(hs_225_depth/2 + wrist_cylinder_length/2)} 0" />
-            <material name="Silver" />
-        </visual>
-        <collision>
-            <geometry>
-                <box size="${hs_225_width} ${hs_225_height} ${hs_225_depth}" />
-            </geometry>
-            <origin rpy="${PI/2} 0 0" xyz="0 0 0" />
-        </collision>
-        <xacro:inertial_matrix_box height="${hs_225_height}" width="${hs_225_width}" depth="${hs_225_depth}" mass="${hs_225_mass}" />
-    </link>
-    <!-- The solid structure below the gripper -->
-    <link name="gripper_base">
-        <visual>
-            <geometry>
-                <box size="${gripper_base_width} ${gripper_base_height} ${gripper_base_depth}" />
-            </geometry>
-            <material name="Black" />
-            <origin rpy="${PI/2} 0 0" xyz="0 0 0" />
-        </visual>
-        <collision>
-            <geometry>
-                <box size="${gripper_base_width} ${gripper_base_height} ${gripper_base_depth}" />
-            </geometry>
-            <origin rpy="${PI/2} 0 0" xyz="0 0 0" />
-        </collision>
-        <xacro:inertial_matrix_box height="${gripper_base_height}" width="${gripper_base_width}" depth="${gripper_base_depth}" mass="0.01" />
-    </link>
-    <!-- Left and right -->
+                <mesh filename="package://lynxmotion_al5d_description/meshes/robot_parts/wrist.dae" />
+            </geometry>
+            <origin rpy="0 0 0" xyz="0 0.165 -0.065" />
+        </visual>
+        <xacro:inertial_matrix_cylinder mass="0.05" height="0.01" radius="0.01" />
+    </link>
+    <link name="gripper">
+        <visual>
+            <geometry>
+                <mesh filename="package://lynxmotion_al5d_description/meshes/robot_parts/gripper.dae" />
+            </geometry>
+            <origin rpy="${PI/2} 0 ${-PI/2}" xyz="0 0 0" />
+        </visual>
+        <xacro:inertial_matrix_box mass="0.2" depth="0.012" height="0.02" width="0.06" />
+    </link>
     <link name="left_finger">
         <visual>
             <geometry>
-                <box size="${finger_width} ${finger_height} ${finger_depth}" />
-            </geometry>
-            <origin rpy="${PI/2} 0 0" xyz="${gripper_base_width/2} ${-(wrist_cylinder_length + gripper_base_depth)} 0" />
-            <material name="silver">
-                <color rgba="0.8 0.8 0.8 1" />
-            </material>
-        </visual>
-        <collision>
-            <geometry>
-                <box size="${finger_width} ${finger_height} ${finger_depth}" />
-            </geometry>
-            <origin rpy="${PI/2} 0 0" xyz="${gripper_base_width/2} ${-(wrist_cylinder_length + gripper_base_depth)} 0" />
-        </collision>
-        <xacro:inertial_matrix_box width="${finger_width}" height="${finger_height}" depth="${finger_depth}" mass="${finger_mass}" />
+                <mesh filename="package://lynxmotion_al5d_description/meshes/robot_parts/finger_left.dae" />
+            </geometry>
+            <origin rpy="${PI/2} 0 ${-PI/2}" xyz="0 0 0" />
+        </visual>
+        <xacro:inertial_matrix_box mass="0.2" depth="0.012" height="0.15" width="0.008" />
     </link>
     <link name="right_finger">
         <visual>
             <geometry>
-                <box size="${finger_width} ${finger_height} ${finger_depth}" />
-            </geometry>
-            <origin rpy="${PI/2} 0 0" xyz="${-gripper_base_width/2} ${-(wrist_cylinder_length + gripper_base_depth)} 0" />
-            <material name="silver">
-                <color rgba="0.8 0.8 0.8 1" />
-            </material>
-        </visual>
-        <collision>
-            <geometry>
-                <box size="${finger_width} ${finger_height} ${finger_depth}" />
-            </geometry>
-            <origin rpy="${PI/2} 0 0" xyz="${-gripper_base_width/2} ${-(wrist_cylinder_length + gripper_base_depth)} 0" />
-        </collision>
-        <xacro:inertial_matrix_box width="${finger_width}" height="${finger_height}" depth="${finger_depth}" mass="${finger_mass}" />
-    </link>
-<xacro:property name="camera_support_depth" value="0.25" />
-    <xacro:property name="camera_support_size" value="0.003" />
-    <xacro:property name="camera_support_big_size" value="0.5" />
-    <xacro:property name="camera_support_to_base" value="0.06" />
+                <mesh filename="package://lynxmotion_al5d_description/meshes/robot_parts/finger_right.dae" />
+            </geometry>
+            <origin rpy="${PI/2} 0 ${-PI/2}" xyz="0 0 0" />
+        </visual>
+        <xacro:inertial_matrix_box mass="0.2" depth="0.012" height="0.15" width="0.008" />
+    </link>
     <link name="camera_link">
-        <visual name="stick">
-            <geometry>
-                <box size="${camera_support_size} ${camera_support_size} ${camera_support_depth}" />
-            </geometry>
-            <origin rpy="0 0 0" xyz="0 ${camera_support_to_base} ${camera_support_depth/2}" />
-            <material name="BlueGrey" />
-        </visual>
-        <visual name="support">
-            <geometry>
-                <box size="${camera_support_big_size} ${camera_support_big_size + camera_support_to_base} ${camera_support_size}" />
-            </geometry>
-            <origin rpy="0 0 0" xyz="0 ${-camera_support_big_size/2} ${camera_support_depth - camera_support_size/2}" />
-            <material name="BlueGrey" />
-        </visual>
-        <collision name="support">
-            <geometry>
-                <box size="${camera_support_big_size} ${camera_support_big_size + camera_support_to_base} ${camera_support_size}" />
-            </geometry>
-            <origin rpy="0 0 0" xyz="0 ${-camera_support_big_size/2} ${camera_support_depth - camera_support_size/2}" />
-            <material name="BlueGrey" />
-        </collision>
-        <xacro:inertial_matrix_box mass="${camera_support_mass}" width="${camera_support_big_size}" height="${camera_support_big_size + camera_support_to_base}" depth="${camera_support_size}" />
-    </link>
-    <!-- Adding a camera sensor to the model -->
+        <visual>
+            <geometry>
+                <box size="0.01 0.01 0.01" />
+            </geometry>
+            <origin rpy="0 0 0" xyz="0 0 ${camera_support_depth}" />
+            <material name="Transparent" />
+        </visual>
+    </link>
     <sensor name="robot_camera" update_rate="1">
         <parent link="camera_link" />
-        <origin xyz="0 0 0" rpy="0 0 0" />
+        <origin xyz="0.005 0.005 0.005" rpy="0 0 0" />
         <camera>
             <image width="640" height="480" hfov="${PI/2}" format="RGB8" near="${camera_support_depth}" far="${camera_support_depth}" />
@@ -206,122 +101,139 @@
     </sensor>
     <!-- Adding joints -->
-    <joint name="camera_support_joint" type="fixed">
-        <parent link="base_link" />
+    <joint name="world_to_robot" type="fixed">
+        <parent link="world" />
+        <child link="robot_support" />
+    </joint>
+    <joint name="camera_joint" type="fixed">
+        <parent link="robot_support" />
         <child link="camera_link" />
-    </joint>
-    <joint name="shoulder_elbow_roll" type="revolute">
-        <parent link="base_link" />
-        <child link="top_box" />
-        <origin xyz="0 0 ${base_height}" />
+        <origin xyz="0 -0.35 0" />
+    </joint>
+    <joint name="link1_rotz" type="revolute">
+        <parent link="robot_support" />
+        <child link="robot_base_cylinder" />
+        <axis xyz="0 0 1" />
+        <origin xyz="0 0.021 0" />
+        <limit effort="10" velocity="1" lower="${-PI}" upper="${PI}" />
+        <dynamics damping="50" friction="1" />
+    </joint>
+    <joint name="robot_base_fixed" type="fixed">
+        <parent link="robot_base_cylinder" />
+        <child link="robot_base_top_box" />
+    </joint>
+    <joint name="link1_rotx" type="revolute">
+        <parent link="robot_base_top_box" />
+        <child link="shoulder" />
         <axis xyz="1 0 0" />
+        <origin xyz="0 -0.015 0.071" />
         <limit effort="10" velocity="1" lower="${-PI/2}" upper="${PI/2}" />
         <dynamics damping="50" friction="1" />
     </joint>
-    <joint name="shoulder_elbow_yall" type="revolute">
-        <parent link="top_box" />
-        <child link="shoulder" />
-        <origin xyz="0 0 0" />
-        <axis xyz="0 0 1" />
+    <joint name="link2_rotx" type="revolute">
+        <parent link="shoulder" />
+        <child link="arm" />
+        <axis xyz="1 0 0" />
+        <origin xyz="0 0 ${shoulder_to_elbow}" />
         <limit effort="10" velocity="1" lower="${-PI/2}" upper="${PI/2}" />
         <dynamics damping="50" friction="1" />
     </joint>
-    <joint name="elbow_roll" type="revolute">
-        <parent link="shoulder" />
-        <child link="elbow" />
-        <origin xyz="0 0 ${base_height + shoulder_to_elbow - hs_755eb_height}" />
+    <joint name="link3_rotx" type="revolute">
+        <parent link="arm" />
+        <child link="wrist" />
         <axis xyz="1 0 0" />
+        <origin xyz="0 ${-tube_length - hs_645_depth + 0.003} 0" />
         <limit effort="10" velocity="1" lower="${-PI/2}" upper="${PI/2}" />
         <dynamics damping="50" friction="1" />
     </joint>
-    <joint name="elbow_to_wrist_roll" type="revolute">
-        <parent link="elbow" />
-        <child link="wrist" />
-        <origin xyz="0 ${-(tube_length+hs_645_height)} 0" />
-        <axis xyz="1 0 0" />
-        <limit effort="10" velocity="1" lower="${-PI/2}" upper="${PI/2}" />
-        <dynamics damping="50" friction="1" />
-    </joint>
-    <joint name="gripper_base_pitch" type="revolute">
+    <joint name="link4_rotz" type="revolute">
         <parent link="wrist" />
-        <child link="gripper_base" />
-        <origin xyz="0 ${-(hs_225_depth/2 + hs_645_height + wrist_cylinder_length)} 0" />
+        <child link="gripper" />
         <axis xyz="0 1 0" />
-        <limit effort="10" velocity="1" lower="0" upper="${PI}" />
-        <dynamics damping="50" friction="1" />
-    </joint>
-    <joint name="left_finger_mov" type="prismatic">
-        <parent link="gripper_base" />
+        <origin xyz="0 -0.055 0" rpy="0 0 0" />
+        <limit effort="10" velocity="1" lower="${-PI}" upper="${PI}" />
+        <dynamics damping="50" friction="1" />
+    </joint>
+    <joint name="finger_left_mov" type="prismatic">
+        <parent link="gripper" />
         <child link="left_finger" />
-        <limit effort="10" velocity="1" lower="${-gripper_base_width/2}" upper="0" />
-        <origin xyz="0 0 0" />
-    </joint>
-    <joint name="right_finger_mov" type="prismatic">
-        <parent link="gripper_base" />
+        <limit effort="10" velocity="1" lower="0" upper="${-gripper_base_width/2}" />
+    </joint>
+    <joint name="finger_right_mov" type="prismatic">
+        <parent link="gripper" />
         <child link="right_finger" />
         <limit effort="10" velocity="1" lower="0" upper="${gripper_base_width/2}" />
-        <origin xyz="0 0 0" />
     </joint>
     <!-- Setting transmissions -->
-    <transmission name="link1_roll_transmission">
-        <type>transmission_interface/SimpleTransmission</type>
-        <joint name="shoulder_elbow_roll">
-            <hardwareInterface>EffortJointInterface</hardwareInterface>
-        </joint>
-        <actuator name="link1_motor">
-            <mechanicalReduction>10</mechanicalReduction>
-            <hardwareInterface>EfforJointInterface</hardwareInterface>
-        </actuator>
-    </transmission>
-    <transmission name="link1_yall_transmission">
-        <type>transmission_interface/SimpleTransmission</type>
-        <joint name="shoulder_elbow_yall">
-            <hardwareInterface>EffortJointInterface</hardwareInterface>
-        </joint>
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
File: urdf/lynxmotion_al5d_properties.urdf.xacro (robot description, xacro)
@@ -16,4 +16,7 @@
     <material name="BlueGrey">
         <color rgba="1 87 155 1" />
+    </material>
+    <material name="Transparent">
+        <color rgba="0.0 0.0 0.0 0.0" />
     </material>
     <!-- Setting properties to be used in the program -->
@@ -41,5 +44,5 @@
     <xacro:property name="hs_645_width" value="0.0406" />
     <xacro:property name="hs_645_height" value="0.0198" />
-    <xacro:property name="hs_645_depth" value="0.0373" />
+    <xacro:property name="hs_645_depth" value="0.037" />
     <xacro:property name="hs_645_mass" value="0.05" />
     <xacro:property name="hs_225_width" value="0.05226" />
@@ -56,5 +59,5 @@
     <xacro:property name="wrist_cylinder_length" value="0.005" />
     <xacro:property name="wrist_cylinder_radius" value="0.01" />
-    <xacro:property name="camera_support_depth" value="0.5" />
+    <xacro:property name="camera_support_depth" value="0.3" />
     <xacro:property name="camera_support_size" value="0.01" />
     <xacro:property name="camera_support_big_size" value="0.5" />
