Commit message: Integrating the robot to Gazebo

File: urdf/lynxmotion_al5d.xacro (robot description, xacro)
@@ -9,7 +9,15 @@
                 <mesh filename="package://lynxmotion_al5d_description/meshes/robot_parts/support.dae" />
             </geometry>
-        </visual>
-        <xacro:inertial_matrix_cylinder mass="0.4" height="0.04" radius="0.04" />
-    </link>
+            <origin rpy="0 0 0" xyz="0 0 0" />
+        </visual>
+        <collision>
+            <geometry>
+                <mesh filename="package://lynxmotion_al5d_description/meshes/robot_parts/support.dae" />
+            </geometry>
+            <origin rpy="0 0 0" xyz="0 0 0" />
+        </collision>
+        <xacro:inertial_matrix_cylinder mass="4" height="0.4" radius="0.4" />
+    </link>
+    <gazebo reference="robot_support" />
     <link name="robot_base_cylinder">
         <visual>
@@ -19,6 +27,13 @@
             <origin rpy="0 0 0" xyz="0 -0.021165 0" />
         </visual>
-        <xacro:inertial_matrix_cylinder mass="0.05" height="0.004" radius="0.04" />
-    </link>
+        <collision>
+            <geometry>
+                <mesh filename="package://lynxmotion_al5d_description/meshes/robot_parts/rotation_cylinder.dae" />
+            </geometry>
+            <origin rpy="0 0 0" xyz="0 -0.021165 0" />
+        </collision>
+        <xacro:inertial_matrix_cylinder mass="0.5" height="0.04" radius="0.4" />
+    </link>
+    <gazebo reference="robot_base_cylinder" />
     <link name="robot_base_top_box">
         <visual>
@@ -28,6 +43,13 @@
             <origin xyz="0.007 -0.024 0" rpy="0 0 0" />
         </visual>
-        <xacro:inertial_matrix_box mass="0.5" depth="0.03" height="0.04" width="0.06" />
-    </link>
+        <collision>
+            <geometry>
+                <mesh filename="package://lynxmotion_al5d_description/meshes/robot_parts/top_box.dae" />
+            </geometry>
+            <origin xyz="0.007 -0.024 0" rpy="0 0 0" />
+        </collision>
+        <xacro:inertial_matrix_box mass="1.5" depth="3" height="4" width="6" />
+    </link>
+    <gazebo reference="robot_base_top_box" />
     <link name="shoulder">
         <visual>
@@ -37,6 +59,13 @@
             <origin rpy="${-PI/8} 0 0" xyz="0 -0.035 -0.06" />
         </visual>
-        <xacro:inertial_matrix_box mass="0.5" depth="0.17" height="0.02" width="0.11" />
-    </link>
+        <collision>
+            <geometry>
+                <mesh filename="package://lynxmotion_al5d_description/meshes/robot_parts/shoulder.dae" />
+            </geometry>
+            <origin rpy="${-PI/8} 0 0" xyz="0 -0.035 -0.06" />
+        </collision>
+        <xacro:inertial_matrix_box mass="0.5" depth="17" height="2" width="11" />
+    </link>
+    <gazebo reference="shoulder" />
     <link name="arm">
         <visual>
@@ -46,6 +75,13 @@
             <origin rpy="-0.895 0 0" xyz="0 ${-tube_length + 2*hs_755eb_depth/5} ${-shoulder_to_elbow - 0.02}" />
         </visual>
-        <xacro:inertial_matrix_box mass="0.2" depth="0.03" height="0.07" width="0.05" />
-    </link>
+        <collision>
+            <geometry>
+                <mesh filename="package://lynxmotion_al5d_description/meshes/robot_parts/arm.dae" />
+            </geometry>
+            <origin rpy="-0.895 0 0" xyz="0 ${-tube_length + 2*hs_755eb_depth/5} ${-shoulder_to_elbow - 0.02}" />
+        </collision>
+        <xacro:inertial_matrix_box mass="0.1" depth="0.3" height="0.7" width="0.5" />
+    </link>
+    <gazebo reference="arm" />
     <link name="wrist">
         <visual>
@@ -55,6 +91,13 @@
             <origin rpy="0 0 0" xyz="0 0.165 -0.065" />
         </visual>
-        <xacro:inertial_matrix_cylinder mass="0.05" height="0.01" radius="0.01" />
-    </link>
+        <collision>
+            <geometry>
+                <mesh filename="package://lynxmotion_al5d_description/meshes/robot_parts/wrist.dae" />
+            </geometry>
+            <origin rpy="0 0 0" xyz="0 0.165 -0.065" />
+        </collision>
+        <xacro:inertial_matrix_cylinder mass="0.5" height="0.1" radius="0.1" />
+    </link>
+    <gazebo reference="wrist" />
     <link name="gripper">
         <visual>
@@ -64,6 +107,13 @@
             <origin rpy="${PI/2} 0 ${-PI/2}" xyz="0 0 0" />
         </visual>
-        <xacro:inertial_matrix_box mass="0.2" depth="0.012" height="0.02" width="0.06" />
-    </link>
+        <collision>
+            <geometry>
+                <mesh filename="package://lynxmotion_al5d_description/meshes/robot_parts/gripper.dae" />
+            </geometry>
+            <origin rpy="${PI/2} 0 ${-PI/2}" xyz="0 0 0" />
+        </collision>
+        <xacro:inertial_matrix_box mass="1" depth="1.2" height="2" width="6" />
+    </link>
+    <gazebo reference="gripper" />
     <link name="left_finger">
         <visual>
@@ -73,6 +123,13 @@
             <origin rpy="${PI/2} 0 ${-PI/2}" xyz="0 0 0" />
         </visual>
-        <xacro:inertial_matrix_box mass="0.2" depth="0.012" height="0.15" width="0.008" />
-    </link>
+        <collision>
+            <geometry>
+                <mesh filename="package://lynxmotion_al5d_description/meshes/robot_parts/finger_left.dae" />
+            </geometry>
+            <origin rpy="${PI/2} 0 ${-PI/2}" xyz="0 0 0" />
+        </collision>
+        <xacro:inertial_matrix_box mass="0.5" depth="1.2" height="15" width="0.8" />
+    </link>
+    <gazebo reference="left_finger" />
     <link name="right_finger">
         <visual>
@@ -82,6 +139,13 @@
             <origin rpy="${PI/2} 0 ${-PI/2}" xyz="0 0 0" />
         </visual>
-        <xacro:inertial_matrix_box mass="0.2" depth="0.012" height="0.15" width="0.008" />
-    </link>
+        <collision>
+            <geometry>
+                <mesh filename="package://lynxmotion_al5d_description/meshes/robot_parts/finger_right.dae" />
+            </geometry>
+            <origin rpy="${PI/2} 0 ${-PI/2}" xyz="0 0 0" />
+        </collision>
+        <xacro:inertial_matrix_box mass="0.5" depth="1.2" height="15" width="0.8" />
+    </link>
+    <gazebo reference="right_finger" />
     <link name="camera_link">
         <visual>
@@ -92,5 +156,13 @@
             <material name="Transparent" />
         </visual>
-    </link>
+        <collision>
+            <geometry>
+                <box size="0.01 0.01 0.01" />
+            </geometry>
+            <origin rpy="0 0 0" xyz="0 0 ${camera_support_depth}" />
+            <material name="Transparent" />
+        </collision>
+    </link>
+    <gazebo reference="camera_link" />
     <sensor name="robot_camera" update_rate="1">
         <parent link="camera_link" />
@@ -165,64 +237,9 @@
     </joint>
     <!-- Setting transmissions -->
-    <transmission name="link1_rotx_transmission">
-        <type>transmission_interface/SimpleTransmission</type>
-        <joint name="link1_rotx">
-            <hardwareInterface>EffortJointInterface</hardwareInterface>
-        </joint>
-        <actuator name="link1_rotx_motor">
-            <mechanicalReduction>10</mechanicalReduction>
-            <hardwareInterface>EffortJointInterface</hardwareInterface>
-        </actuator>
-    </transmission>
-    <transmission name="link1_rotx_transmission">
-        <type>transmission_interface/SimpleTransmission</type>
-        <joint name="link1_rotx">
-            <hardwareInterface>EffortJointInterface</hardwareInterface>
-        </joint>
-        <actuator name="link1_rotx_motor">
-            <mechanicalReduction>10</mechanicalReduction>
-            <hardwareInterface>EffortJointInterface</hardwareInterface>
-        </actuator>
-    </transmission>
-    <transmission name="link1_rotz_transmission">
-        <type>transmission_interface/SimpleTransmission</type>
-        <joint name="link1_rotz">
-            <hardwareInterface>EffortJointInterface</hardwareInterface>
-        </joint>
-        <actuator name="link1_rotz_motor">
-            <mechanicalReduction>10</mechanicalReduction>
-            <hardwareInterface>EffortJointInterface</hardwareInterface>
-        </actuator>
-    </transmission>
-    <transmission name="link2_rotx_transmission">
-        <type>transmission_interface/SimpleTransmission</type>
-        <joint name="link2_rotx">
-            <hardwareInterface>EffortJointInterface</hardwareInterface>
-        </joint>
-        <actuator name="link2_rotx_motor">
-            <mechanicalReduction>10</mechanicalReduction>
-            <hardwareInterface>EffortJointInterface</hardwareInterface>
-        </actuator>
-    </transmission>
-    <transmission name="link3_rotx_transmission">
-        <type>transmission_interface/SimpleTransmission</type>
-        <joint name="link3_rotx">
-            <hardwareInterface>EffortJointInterface</hardwareInterface>
-        </joint>
-        <actuator name="link3_rotx_motor">
-            <mechanicalReduction>10</mechanicalReduction>
-            <hardwareInterface>EffortJointInterface</hardwareInterface>
-        </actuator>
-    </transmission>
-    <transmission name="link4_rotz_transmission">
-        <type>transmission_interface/SimpleTransmission</type>
-        <joint name="link4_rotz">
-            <hardwareInterface>EffortJointInterface</hardwareInterface>
-        </joint>
-        <actuator name="link4_rotz_motor">
-            <mechanicalReduction>10</mechanicalReduction>
-            <hardwareInterface>EffortJointInterface</hardwareInterface>
-        </actuator>
-    </transmission>
+    <xacro:transmission_block joint_name="link1_rotx"/>
+    <xacro:transmission_block joint_name="link1_rotz"/>
+    <xacro:transmission_block joint_name="link2_rotx"/>
+    <xacro:transmission_block joint_name="link3_rotx"/>
+    <xacro:transmission_block joint_name="link4_rotz"/>
     <transmission name="fingers_transmission">
         <type>transmission_interface/SimpleTransmission</type>
@@ -238,3 +255,9 @@
         </actuator>
     </transmission>
+      <!-- ros_control plugin -->
+    <gazebo>
+        <plugin name="gazebo_ros_control" filename="libgazebo_ros_control.so">
+        <robotNamespace>/lynxmotion_al5d</robotNamespace>
+        </plugin>
+    </gazebo>
 </robot>

File: urdf/lynxmotion_al5d_properties.urdf.xacro (robot description, xacro)
@@ -68,5 +68,5 @@
         <inertial>
             <mass value="${mass}" />
-            <inertia ixx="${(3*radius*radius + height*height)*mass/12}" ixy="0.0" ixz="0.0" iyx="0.0" iyy="${(3*radius*radius + height*height)*mass/12}" iyz="0.0" izx="0.0" izy="0.0" izz="${(mass*radius*radius)/2}" />
+            <inertia ixx="${(3*radius*radius + height*height)*mass/12}" ixy="0.0" ixz="0.0" iyy="${(3*radius*radius + height*height)*mass/12}" iyz="0.0" izz="${(mass*radius*radius)/2}" />
         </inertial>
     </xacro:macro>
@@ -74,6 +74,18 @@
         <inertial>
             <mass value="${mass}" />
-            <inertia ixx="${(depth*depth + height*height)*mass/12}" ixy="0.0" ixz="0.0" iyx="0.0" iyy="${(width*width + depth*depth)*mass/12}" iyz="0.0" izx="0.0" izy="0.0" izz="${(width*width + height*height)*mass/12}" />
+            <inertia ixx="${(depth*depth + height*height)*mass/12}" ixy="0.0" ixz="0.0" iyy="${(width*width + depth*depth)*mass/12}" iyz="0.0" izz="${(width*width + height*height)*mass/12}" />
         </inertial>
     </xacro:macro>
+    <xacro:macro name="transmission_block" params="joint_name">
+        <transmission name="tran1">
+            <type>transmission_interface/SimpleTransmission</type>
+            <joint name="${joint_name}">
+                <hardwareInterface>PositionJointInterface</hardwareInterface>
+            </joint>
+            <actuator name="motor1">
+                <hardwareInterface>PositionJointInterface</hardwareInterface>
+                <mechanicalReduction>1</mechanicalReduction>
+            </actuator>
+        </transmission>
+   </xacro:macro>
 </robot>

Commit message: Updating the inertia values

File: urdf/lynxmotion_al5d.xacro (robot description, xacro)
@@ -17,5 +17,5 @@
             <origin rpy="0 0 0" xyz="0 0 0" />
         </collision>
-        <xacro:inertial_matrix_cylinder mass="4" height="0.4" radius="0.4" />
+        <xacro:inertial_matrix mass="0.6" ixx="0.000008" ixy="0" ixz="0" iyy="0.000002" iyz="0.000001" izz="0.000009" xyz="0.001689 0.073328 0.021330" />
     </link>
     <gazebo reference="robot_support" />
@@ -33,5 +33,5 @@
             <origin rpy="0 0 0" xyz="0 -0.021165 0" />
         </collision>
-        <xacro:inertial_matrix_cylinder mass="0.5" height="0.04" radius="0.4" />
+        <xacro:inertial_matrix mass="0.05" ixx="0" ixy="0" ixz="0" iyy="0" iyz="0" izz="0" xyz="0 0.020888 0.046075" />
     </link>
     <gazebo reference="robot_base_cylinder" />
@@ -49,5 +49,5 @@
             <origin xyz="0.007 -0.024 0" rpy="0 0 0" />
         </collision>
-        <xacro:inertial_matrix_box mass="1.5" depth="3" height="4" width="6" />
+        <xacro:inertial_matrix mass="0.05" ixx="0" ixy="0" ixz="0" iyy="0" iyz="0" izz="0" xyz="-0.007419 0.026465 0.069384" />
     </link>
     <gazebo reference="robot_base_top_box" />
@@ -65,5 +65,5 @@
             <origin rpy="${-PI/8} 0 0" xyz="0 -0.035 -0.06" />
         </collision>
-        <xacro:inertial_matrix_box mass="0.5" depth="17" height="2" width="11" />
+        <xacro:inertial_matrix mass="0.4" ixx="0" ixy="0" ixz="0" iyy="0" iyz="0" izz="0" xyz="0.0014 -0.009124 0.113692" />
     </link>
     <gazebo reference="shoulder" />
@@ -81,5 +81,5 @@
             <origin rpy="-0.895 0 0" xyz="0 ${-tube_length + 2*hs_755eb_depth/5} ${-shoulder_to_elbow - 0.02}" />
         </collision>
-        <xacro:inertial_matrix_box mass="2" depth="0.3" height="0.7" width="0.5" />
+        <xacro:inertial_matrix mass="0.18" ixx="0.000008" ixy="0" ixz="0" iyy="0.000002" iyz="0.000001" izz="0.000009" xyz="-0.002468 -0.119892 0.126276" />
     </link>
     <gazebo reference="arm" />
@@ -97,5 +97,5 @@
             <origin rpy="0 0 0" xyz="0 0.165 -0.065" />
         </collision>
-        <xacro:inertial_matrix_box mass="0.25" depth="0.25" height="0.35" width="0.5" />
+        <xacro:inertial_matrix mass="0.04" ixx="0" ixy="0" ixz="0" iyy="0" iyz="0" izz="0" xyz="-0.002314 -0.187551 0.067613" />
     </link>
     <gazebo reference="wrist" />
@@ -113,5 +113,5 @@
             <origin rpy="${PI/2} 0 ${-PI/2}" xyz="0 0 0" />
         </collision>
-        <xacro:inertial_matrix_box mass="1" depth="0.12" height="0.2" width="0.6" />
+        <xacro:inertial_matrix mass="0.031" ixx="0" ixy="0" ixz="0" iyy="0" iyz="0" izz="0" xyz="-0.007640 0.007645 0.002347" />
     </link>
     <gazebo reference="gripper" />
@@ -129,5 +129,5 @@
             <origin rpy="${PI/2} 0 ${-PI/2}" xyz="0 0 0" />
         </collision>
-        <xacro:inertial_matrix_box mass="0.05" depth="0.12" height="1.5" width="0.08" />
+        <xacro:inertial_matrix mass="0.02" ixx="0" ixy="0" ixz="0" iyy="0" iyz="0" izz="0" xyz="0.01688 0.003755 -0.016411"/>
     </link>
     <gazebo reference="left_finger" />
@@ -145,5 +145,5 @@
             <origin rpy="${PI/2} 0 ${-PI/2}" xyz="0 0 0" />
         </collision>
-        <xacro:inertial_matrix_box mass="0.05" depth="0.12" height="1.5" width="0.08" />
+        <xacro:inertial_matrix mass="0.02" ixx="0" ixy="0" ixz="0" iyy="0" iyz="0" izz="0" xyz="0.016859 0.003755 0.021112" />
     </link>
     <gazebo reference="right_finger" />
@@ -163,4 +163,5 @@
             <material name="Transparent" />
         </collision>
+        <xacro:inertial_matrix_box mass="0.05" depth="0.01" height="0.01" width="0.01" />
     </link>
     <gazebo reference="camera_link" />
@@ -229,10 +230,11 @@
         <parent link="gripper" />
         <child link="left_finger" />
-        <limit effort="10" velocity="1" lower="0" upper="${-gripper_base_width/2}" />
+        <limit effort="10" velocity="0.001" upper="0" lower="${-gripper_base_width/2}" />
     </joint>
     <joint name="finger_right_mov" type="prismatic">
         <parent link="gripper" />
         <child link="right_finger" />
-        <limit effort="10" velocity="1" lower="0" upper="${gripper_base_width/2}" />
+        <limit effort="10" velocity="0.001" lower="0" upper="${gripper_base_width/2}" />
+        <mimic joint="finger_left_mov" multiplier="-1" />
     </joint>
     <!-- Setting transmissions -->

File: urdf/lynxmotion_al5d_properties.urdf.xacro (robot description, xacro)
@@ -71,4 +71,11 @@
         </inertial>
     </xacro:macro>
+    <xacro:macro name="inertial_matrix" params="mass ixx ixy ixz iyy iyz izz xyz">
+        <inertial>
+            <origin rpy="0 0 0" xyz="${xyz}" />
+            <mass value="${mass}" />
+            <inertia ixx="${ixx}" ixy="${ixy}" ixz="${ixz}" iyy="${iyy}" iyz="${iyz}" izz="${izz}" />
+        </inertial>
+    </xacro:macro>
     <xacro:macro name="inertial_matrix_box" params="mass height width depth">
         <inertial>
