Commit message: Updated robot model to cater for the joints movements

File: urdf/lynxmotion_al5d.xacro (robot description, xacro)
@@ -9,7 +9,15 @@
                 <mesh filename="package://lynxmotion_al5d_description/meshes/robot_parts/support.dae" />
             </geometry>
-        </visual>
-        <xacro:inertial_matrix_cylinder mass="0.4" height="0.04" radius="0.04" />
-    </link>
+            <origin rpy="0 0 0" xyz="0 0 0" />
+        </visual>
+        <collision>
+            <geometry>
+                <mesh filename="package://lynxmotion_al5d_description/meshes/robot_parts/support.dae" />
+            </geometry>
+            <origin rpy="0 0 0" xyz="0 0 0" />
+        </collision>
+        <xacro:inertial_matrix mass="0.133" ixx="3.6565e-7" ixy="-3.72e-9" ixz="1e-6" iyy="9.404e-8" iyz="4.375e-8" izz="4.1776e-7" xyz="0.000585 0.0602746 0.0170628" />
+    </link>
+    <gazebo reference="robot_support" />
     <link name="robot_base_cylinder">
         <visual>
@@ -19,6 +27,14 @@
             <origin rpy="0 0 0" xyz="0 -0.021165 0" />
         </visual>
-        <xacro:inertial_matrix_cylinder mass="0.05" height="0.004" radius="0.04" />
-    </link>
+        <collision>
+            <geometry>
+                <mesh filename="package://lynxmotion_al5d_description/meshes/robot_parts/rotation_cylinder.dae" />
+            </geometry>
+            <origin rpy="0 0 0" xyz="0 -0.021165 0" />
+        </collision>
+        <!-- <xacro:inertial_matrix mass="0.042" ixx="1.584e-8" ixy="-0" ixz="0" iyy="1.584e-8" iyz="-4e-11" izz="3.156e-8" xyz="-0 0.002088 0.046075" /> -->
+        <xacro:inertial_matrix_bis mass="0.042" />
+    </link>
+    <gazebo reference="robot_base_cylinder" />
     <link name="robot_base_top_box">
         <visual>
@@ -28,6 +44,14 @@
             <origin xyz="0.007 -0.024 0" rpy="0 0 0" />
         </visual>
-        <xacro:inertial_matrix_box mass="0.5" depth="0.03" height="0.04" width="0.06" />
-    </link>
+        <collision>
+            <geometry>
+                <mesh filename="package://lynxmotion_al5d_description/meshes/robot_parts/top_box.dae" />
+            </geometry>
+            <origin xyz="0.007 -0.024 0" rpy="0 0 0" />
+        </collision>
+         <!-- <xacro:inertial_matrix mass="0.084" ixx="7.063e-8" ixy="2.68e-9" ixz="1.7e-10" iyy="5.396e-8" iyz="9.3e-10" izz="9.744e-8" xyz="-0.007418 0.026464 0.069384" /> -->
+        <xacro:inertial_matrix_bis mass="0.184" />
+    </link>
+    <gazebo reference="robot_base_top_box" />
     <link name="shoulder">
         <visual>
@@ -37,6 +61,14 @@
             <origin rpy="${-PI/8} 0 0" xyz="0 -0.035 -0.06" />
         </visual>
-        <xacro:inertial_matrix_box mass="0.5" depth="0.17" height="0.02" width="0.11" />
-    </link>
+        <collision>
+            <geometry>
+                <mesh filename="package://lynxmotion_al5d_description/meshes/robot_parts/shoulder.dae" />
+            </geometry>
+            <origin rpy="${-PI/8} 0 0" xyz="0 -0.035 -0.06" />
+        </collision>
+        <!-- <xacro:inertial_matrix mass="0.035" ixx="6.151e-8" ixy="-2.57e-9" ixz="6.03e-9" iyy="7.851e-8" iyz="2.106e-8" izz="3.803e-8" xyz="0.001399 -0.009123 0.113692" /> -->
+        <xacro:inertial_matrix_bis mass="0.095" />
+    </link>
+    <gazebo reference="shoulder" />
     <link name="arm">
         <visual>
@@ -46,6 +78,14 @@
             <origin rpy="-0.895 0 0" xyz="0 ${-tube_length + 2*hs_755eb_depth/5} ${-shoulder_to_elbow - 0.02}" />
         </visual>
-        <xacro:inertial_matrix_box mass="0.2" depth="0.03" height="0.07" width="0.05" />
-    </link>
+        <collision>
+            <geometry>
+                <mesh filename="package://lynxmotion_al5d_description/meshes/robot_parts/arm.dae" />
+            </geometry>
+            <origin rpy="-0.895 0 0" xyz="0 ${-tube_length + 2*hs_755eb_depth/5} ${-shoulder_to_elbow - 0.02}" />
+        </collision>
+        <!--<xacro:inertial_matrix mass="0.18" ixx="0.000008" ixy="0" ixz="0" iyy="0.000002" iyz="0.000001" izz="0.000009" xyz="-0.002468 -0.119892 0.126276" /> -->
+        <xacro:inertial_matrix_bis mass="0.1" />
+    </link>
+    <gazebo reference="arm" />
     <link name="wrist">
         <visual>
@@ -55,6 +95,14 @@
             <origin rpy="0 0 0" xyz="0 0.165 -0.065" />
         </visual>
-        <xacro:inertial_matrix_cylinder mass="0.05" height="0.01" radius="0.01" />
-    </link>
+        <collision>
+            <geometry>
+                <mesh filename="package://lynxmotion_al5d_description/meshes/robot_parts/wrist.dae" />
+            </geometry>
+            <origin rpy="0 0 0" xyz="0 0.165 -0.065" />
+        </collision>
+        <!-- <xacro:inertial_matrix mass="0.04" ixx="0" ixy="0" ixz="0" iyy="0" iyz="0" izz="0" xyz="-0.002314 -0.187551 0.067613" /> -->
+            <xacro:inertial_matrix_bis mass="0.055" />
+    </link>
+    <gazebo reference="wrist" />
     <link name="gripper">
         <visual>
@@ -64,6 +112,14 @@
             <origin rpy="${PI/2} 0 ${-PI/2}" xyz="0 0 0" />
         </visual>
-        <xacro:inertial_matrix_box mass="0.2" depth="0.012" height="0.02" width="0.06" />
-    </link>
+        <collision>
+            <geometry>
+                <mesh filename="package://lynxmotion_al5d_description/meshes/robot_parts/gripper.dae" />
+            </geometry>
+            <origin rpy="${PI/2} 0 ${-PI/2}" xyz="0 0 0" />
+        </collision>
+        <!--<xacro:inertial_matrix mass="0.031" ixx="0" ixy="0" ixz="0" iyy="0" iyz="0" izz="0" xyz="-0.007640 0.007645 0.002347" /> -->
+        <xacro:inertial_matrix_bis mass="0.042" />
+    </link>
+    <gazebo reference="gripper" />
     <link name="left_finger">
         <visual>
@@ -73,6 +129,14 @@
             <origin rpy="${PI/2} 0 ${-PI/2}" xyz="0 0 0" />
         </visual>
-        <xacro:inertial_matrix_box mass="0.2" depth="0.012" height="0.15" width="0.008" />
-    </link>
+        <collision>
+            <geometry>
+                <mesh filename="package://lynxmotion_al5d_description/meshes/robot_parts/finger_left.dae" />
+            </geometry>
+            <origin rpy="${PI/2} 0 ${-PI/2}" xyz="0 0 0" />
+        </collision>
+        <!-- <xacro:inertial_matrix mass="0.02" ixx="0" ixy="0" ixz="0" iyy="0" iyz="0" izz="0" xyz="0.01688 0.003755 -0.016411"/> -->
+        <xacro:inertial_matrix_bis mass="0.0006" />
+    </link>
+    <gazebo reference="left_finger" />
     <link name="right_finger">
         <visual>
@@ -82,6 +146,14 @@
             <origin rpy="${PI/2} 0 ${-PI/2}" xyz="0 0 0" />
         </visual>
-        <xacro:inertial_matrix_box mass="0.2" depth="0.012" height="0.15" width="0.008" />
-    </link>
+        <collision>
+            <geometry>
+                <mesh filename="package://lynxmotion_al5d_description/meshes/robot_parts/finger_right.dae" />
+            </geometry>
+            <origin rpy="${PI/2} 0 ${-PI/2}" xyz="0 0 0" />
+        </collision>
+         <!-- <xacro:inertial_matrix mass="0.02" ixx="0" ixy="0" ixz="0" iyy="0" iyz="0" izz="0" xyz="0.01688 0.003755 -0.016411"/> -->
+        <xacro:inertial_matrix_bis mass="0.0006" />
+    </link>
+    <gazebo reference="right_finger" />
     <link name="camera_link">
         <visual>
@@ -92,5 +164,14 @@
             <material name="Transparent" />
         </visual>
-    </link>
+        <collision>
+            <geometry>
+                <box size="0.01 0.01 0.01" />
+            </geometry>
+            <origin rpy="0 0 0" xyz="0 0 ${camera_support_depth}" />
+            <material name="Transparent" />
+        </collision>
+        <xacro:inertial_matrix_bis mass="0.05" />
+    </link>
+    <gazebo reference="camera_link" />
     <sensor name="robot_camera" update_rate="1">
         <parent link="camera_link" />
@@ -104,4 +185,5 @@
         <parent link="world" />
         <child link="robot_support" />
+        <dynamics damping="0" friction="0" />
     </joint>
     <joint name="camera_joint" type="fixed">
@@ -109,4 +191,5 @@
         <child link="camera_link" />
         <origin xyz="0 -0.35 0" />
+        <dynamics damping="10" friction="0.7" />
     </joint>
     <joint name="link1_rotz" type="revolute">
@@ -116,9 +199,11 @@
         <origin xyz="0 0.021 0" />
         <limit effort="10" velocity="1" lower="${-PI}" upper="${PI}" />
-        <dynamics damping="50" friction="1" />
+        <dynamics damping="0" friction="0" />
+        <dynamics damping="10" friction="0.7" />
     </joint>
     <joint name="robot_base_fixed" type="fixed">
         <parent link="robot_base_cylinder" />
         <child link="robot_base_top_box" />
+        <dynamics damping="10" friction="0.7" />
     </joint>
     <joint name="link1_rotx" type="revolute">
@@ -128,5 +213,5 @@
         <origin xyz="0 -0.015 0.071" />
         <limit effort="10" velocity="1" lower="${-PI/2}" upper="${PI/2}" />
-        <dynamics damping="50" friction="1" />
+        <dynamics damping="10" friction="0.7" />
     </joint>
     <joint name="link2_rotx" type="revolute">
@@ -136,5 +221,5 @@
         <origin xyz="0 0 ${shoulder_to_elbow}" />
         <limit effort="10" velocity="1" lower="${-PI/2}" upper="${PI/2}" />
-        <dynamics damping="50" friction="1" />
+        <dynamics damping="10" friction="0.7" />
     </joint>
     <joint name="link3_rotx" type="revolute">
@@ -144,7 +229,7 @@
         <origin xyz="0 ${-tube_length - hs_645_depth + 0.003} 0" />
         <limit effort="10" velocity="1" lower="${-PI/2}" upper="${PI/2}" />
-        <dynamics damping="50" friction="1" />
-    </joint>
-    <joint name="link4_rotz" type="revolute">
+        <dynamics damping="10" friction="0.7" />
+    </joint>
+   <joint name="link4_rotz" type="revolute">
         <parent link="wrist" />
         <child link="gripper" />
@@ -152,89 +237,65 @@
         <origin xyz="0 -0.055 0" rpy="0 0 0" />
         <limit effort="10" velocity="1" lower="${-PI}" upper="${PI}" />
-        <dynamics damping="50" friction="1" />
-    </joint>
-    <joint name="finger_left_mov" type="prismatic">
+        <dynamics damping="10" friction="0.7" />
+    </joint>
+   <joint name="finger_left_mov" type="prismatic">
         <parent link="gripper" />
         <child link="left_finger" />
-        <limit effort="10" velocity="1" lower="0" upper="${-gripper_base_width/2}" />
-    </joint>
-    <joint name="finger_right_mov" type="prismatic">
+        <limit effort="10" velocity="0.005" upper="0" lower="${-gripper_base_width/2}" />
+        <dynamics damping="10" friction="0.7" />
+    </joint>
+   <joint name="finger_right_mov" type="prismatic">
         <parent link="gripper" />
         <child link="right_finger" />
-        <limit effort="10" velocity="1" lower="0" upper="${gripper_base_width/2}" />
+        <limit effort="10" velocity="0.001" lower="0" upper="${gripper_base_width/2}" />
+        <mimic joint="finger_left_mov" multiplier="-1" />
+        <dynamics damping="10" friction="0.7" />
     </joint>
     <!-- Setting transmissions -->
-    <transmission name="link1_rotx_transmission">
-        <type>transmission_interface/SimpleTransmission</type>
-        <joint name="link1_rotx">
-            <hardwareInterface>EffortJointInterface</hardwareInterface>
-        </joint>
-        <actuator name="link1_rotx_motor">
-            <mechanicalReduction>10</mechanicalReduction>
-            <hardwareInterface>EffortJointInterface</hardwareInterface>
-        </actuator>
-    </transmission>
-    <transmission name="link1_rotx_transmission">
-        <type>transmission_interface/SimpleTransmission</type>
-        <joint name="link1_rotx">
-            <hardwareInterface>EffortJointInterface</hardwareInterface>
-        </joint>
-        <actuator name="link1_rotx_motor">
-            <mechanicalReduction>10</mechanicalReduction>
-            <hardwareInterface>EffortJointInterface</hardwareInterface>
-        </actuator>
-    </transmission>
-    <transmission name="link1_rotz_transmission">
-        <type>transmission_interface/SimpleTransmission</type>
-        <joint name="link1_rotz">
-            <hardwareInterface>EffortJointInterface</hardwareInterface>
-        </joint>
-        <actuator name="link1_rotz_motor">
-            <mechanicalReduction>10</mechanicalReduction>
-            <hardwareInterface>EffortJointInterface</hardwareInterface>
-        </actuator>
-    </transmission>
-    <transmission name="link2_rotx_transmission">
-        <type>transmission_interface/SimpleTransmission</type>
-        <joint name="link2_rotx">
-            <hardwareInterface>EffortJointInterface</hardwareInterface>
-        </joint>
-        <actuator name="link2_rotx_motor">
-            <mechanicalReduction>10</mechanicalReduction>
-            <hardwareInterface>EffortJointInterface</hardwareInterface>
-        </actuator>
-    </transmission>
-    <transmission name="link3_rotx_transmission">
-        <type>transmission_interface/SimpleTransmission</type>
-        <joint name="link3_rotx">
-            <hardwareInterface>EffortJointInterface</hardwareInterface>
-        </joint>
-        <actuator name="link3_rotx_motor">
-            <mechanicalReduction>10</mechanicalReduction>
-            <hardwareInterface>EffortJointInterface</hardwareInterface>
-        </actuator>
-    </transmission>
-    <transmission name="link4_rotz_transmission">
-        <type>transmission_interface/SimpleTransmission</type>
-        <joint name="link4_rotz">
-            <hardwareInterface>EffortJointInterface</hardwareInterface>
-        </joint>
-        <actuator name="link4_rotz_motor">
-            <mechanicalReduction>10</mechanicalReduction>
-            <hardwareInterface>EffortJointInterface</hardwareInterface>
-        </actuator>
-    </transmission>
-    <transmission name="fingers_transmission">
-        <type>transmission_interface/SimpleTransmission</type>
-        <joint name="finger_left_mov">
-            <hardwareInterface>EffortJointInterface</hardwareInterface>
-        </joint>
-        <joint name="finger_right_mov">
-            <hardwareInterface>EffortJointInterface</hardwareInterface>
-        </joint>
-        <actuator name="fingers_motor">
-            <mechanicalReduction>10</mechanicalReduction>
-            <hardwareInterface>EffortJointInterface</hardwareInterface>
-        </actuator>
-    </transmission>
+    <xacro:transmission_block joint_name="link1_rotx"/>
+    <xacro:transmission_block joint_name="link1_rotz"/>
+    <xacro:transmission_block joint_name="link2_rotx"/>
+    <xacro:transmission_block joint_name="link3_rotx"/>
+    <xacro:transmission_block joint_name="link4_rotz"/>
+    <xacro:transmission_block_finger joint_name="finger_right_mov"/>
+    <xacro:transmission_block_finger joint_name="finger_left_mov"/>
+      <!-- ros_control plugin -->
+    <gazebo>
+        <plugin name="gazebo_ros_control" filename="libgazebo_ros_control.so">
+            <robotNamespace>/lynxmotion_al5d</robotNamespace>
+            <legacyModeNS>true</legacyModeNS>
+        </plugin>
+    </gazebo>
+    <gazebo reference="camera_link">
+        <sensor name="external_camera" type="camera">
+            <update_rate>1.0</update_rate>
+            <camera name="camera_top">
+                <horizontal_fov>1.0</horizontal_fov>
+                <image>
+                    <width>640</width>
+                    <height>480</height>
+                    <format>R8G8B8</format>
+                </image>
+                <clip>
+                    <near>0.3</near>
+                    <far>500</far>
+                </clip>
+            </camera>
+            <plugin filename="libgazebo_ros_camera.so" name="camera_controller">
+                <robotNamespace>/lynxmotion_al5d</robotNamespace>
+                <alwaysOn>true</alwaysOn>
+                <updateRate>1.0</updateRate>
+                <cameraName>al5d_external_vision</cameraName>
+                <imageTopicName>image_raw</imageTopicName>
+                <cameraInfoTopicName>camera_info</cameraInfoTopicName>
+                <frameName>camera_link</frameName>
+                <hackBaseline>0.07</hackBaseline>
+                <distortionK1>-0.0545211</distortionK1>
+                <distortionK2>0.06919734</distortionK2>
+                <distortionK3>-0.0241095</distortionK3>
+                <distortionT1>-0.0112245</distortionT1>
+                <distortionT2>0.0</distortionT2>
+            </plugin>
+        </sensor>
+    </gazebo>
 </robot>

File: urdf/lynxmotion_al5d_properties.urdf.xacro (robot description, xacro)
@@ -68,5 +68,12 @@
         <inertial>
             <mass value="${mass}" />
-            <inertia ixx="${(3*radius*radius + height*height)*mass/12}" ixy="0.0" ixz="0.0" iyx="0.0" iyy="${(3*radius*radius + height*height)*mass/12}" iyz="0.0" izx="0.0" izy="0.0" izz="${(mass*radius*radius)/2}" />
+            <inertia ixx="${(3*radius*radius + height*height)*mass/12}" ixy="0.0" ixz="0.0" iyy="${(3*radius*radius + height*height)*mass/12}" iyz="0.0" izz="${(mass*radius*radius)/2}" />
+        </inertial>
+    </xacro:macro>
+    <xacro:macro name="inertial_matrix" params="mass ixx ixy ixz iyy iyz izz xyz">
+        <inertial>
+            <origin rpy="0 0 0" xyz="${xyz}" />
+            <mass value="${mass}" />
+            <inertia ixx="${ixx}" ixy="${ixy}" ixz="${ixz}" iyy="${iyy}" iyz="${iyz}" izz="${izz}" />
         </inertial>
     </xacro:macro>
@@ -74,6 +81,36 @@
         <inertial>
             <mass value="${mass}" />
-            <inertia ixx="${(depth*depth + height*height)*mass/12}" ixy="0.0" ixz="0.0" iyx="0.0" iyy="${(width*width + depth*depth)*mass/12}" iyz="0.0" izx="0.0" izy="0.0" izz="${(width*width + height*height)*mass/12}" />
+            <inertia ixx="${(depth*depth + height*height)*mass/12}" ixy="0.0" ixz="0.0" iyy="${(width*width + depth*depth)*mass/12}" iyz="0.0" izz="${(width*width + height*height)*mass/12}" />
         </inertial>
     </xacro:macro>
+   <xacro:macro name="inertial_matrix_bis" params="mass">
+      <inertial>
+        <mass value="${mass}" />
+        <inertia ixx="1.0" ixy="0.0" ixz="0.0" iyy="0.5" iyz="0.0" izz="1.0" />
+      </inertial>
+   </xacro:macro>
+    <xacro:macro name="transmission_block" params="joint_name">
+        <transmission name="tran1">
+            <type>transmission_interface/SimpleTransmission</type>
+            <joint name="${joint_name}">
+                <hardwareInterface>hardware_interface/PositionJointInterface</hardwareInterface>
+            </joint>
+            <actuator name="motor1">
+                <hardwareInterface>hardware_interface/PositionJointInterface</hardwareInterface>
+                <mechanicalReduction>1</mechanicalReduction>
+            </actuator>
+        </transmission>
+   </xacro:macro>
+    <xacro:macro name="transmission_block_finger" params="joint_name">
+        <transmission name="tran2">
+            <type>transmission_interface/SimpleTransmission</type>
+            <joint name="${joint_name}">
+                <hardwareInterface>hardware_interface/PositionJointInterface</hardwareInterface>
+            </joint>
+            <actuator name="motor2">
+                <hardwareInterface>hardware_interface/PositionJointInterface</hardwareInterface>
+                <mechanicalReduction>1</mechanicalReduction>
+            </actuator>
+        </transmission>
+   </xacro:macro>
 </robot>
