Commit message: Fixing Gazebo issues

File: urdf/lynxmotion_al5d.xacro (robot description, xacro)
@@ -3,5 +3,20 @@
     <xacro:include filename="$(find lynxmotion_al5d_description)/urdf/lynxmotion_al5d_properties.urdf.xacro" />
     <!-- Base link comprising the board behind the robot and the cylinder at its bottom -->
-    <!--<link name="world" /> -->
+    <!-- <link name="world">
+        <visual>
+            <geometry>
+                <box size="0.001 0.001 0.001" />
+            </geometry>
+            <origin rpy="0 0 0" xyz="0 0 0" />
+        </visual>
+        <collision>
+            <geometry>
+                <box size="0.001 0.001 0.001" />
+            </geometry>
+            <origin rpy="0 0 0" xyz="0 0 0" />
+        </collision>
+        <xacro:inertial_matrix_bis mass="1" />
+    </link>
+    <gazebo reference="world" /> -->
     <link name="robot_support">
         <visual>
@@ -49,5 +64,4 @@
             <origin xyz="0.007 -0.024 0" rpy="0 0 0" />
         </collision>
-         <!-- <xacro:inertial_matrix mass="0.084" ixx="7.063e-8" ixy="2.68e-9" ixz="1.7e-10" iyy="5.396e-8" iyz="9.3e-10" izz="9.744e-8" xyz="-0.007418 0.026464 0.069384" /> -->
         <xacro:inertial_matrix_bis mass="0.184" />
     </link>
@@ -58,5 +72,5 @@
                 <mesh filename="package://lynxmotion_al5d_description/meshes/robot_parts/shoulder.dae" />
             </geometry>
-            <origin rpy="${-PI/8} 0 0" xyz="0 -0.035 -0.06" />
+            <origin rpy="${-5*PI/8} 0 0" xyz="0 -0.0625 0.036" />
         </visual>
         <collision>
@@ -64,7 +78,6 @@
                 <mesh filename="package://lynxmotion_al5d_description/meshes/robot_parts/shoulder.dae" />
             </geometry>
-            <origin rpy="${-PI/8} 0 0" xyz="0 -0.035 -0.06" />
-        </collision>
-        <!-- <xacro:inertial_matrix mass="0.035" ixx="6.151e-8" ixy="-2.57e-9" ixz="6.03e-9" iyy="7.851e-8" iyz="2.106e-8" izz="3.803e-8" xyz="0.001399 -0.009123 0.113692" /> -->
+            <origin rpy="${-5*PI/8} 0 0" xyz="0 -0.0625 0.036" />
+        </collision>
         <xacro:inertial_matrix_bis mass="0.095" />
     </link>
@@ -83,5 +96,4 @@
             <origin rpy="-0.895 0 0" xyz="0 ${-tube_length + 2*hs_755eb_depth/5} ${-shoulder_to_elbow - 0.02}" />
         </collision>
-        <!--<xacro:inertial_matrix mass="0.18" ixx="0.000008" ixy="0" ixz="0" iyy="0.000002" iyz="0.000001" izz="0.000009" xyz="-0.002468 -0.119892 0.126276" /> -->
         <xacro:inertial_matrix_bis mass="0.1" />
     </link>
@@ -92,5 +104,5 @@
                 <mesh filename="package://lynxmotion_al5d_description/meshes/robot_parts/wrist.dae" />
             </geometry>
-            <origin rpy="0 0 0" xyz="0 0.165 -0.065" />
+            <origin rpy="${PI} 0 0" xyz="0.005 -0.165 0.067" />
         </visual>
         <collision>
@@ -98,8 +110,7 @@
                 <mesh filename="package://lynxmotion_al5d_description/meshes/robot_parts/wrist.dae" />
             </geometry>
-            <origin rpy="0 0 0" xyz="0 0.165 -0.065" />
-        </collision>
-        <!-- <xacro:inertial_matrix mass="0.04" ixx="0" ixy="0" ixz="0" iyy="0" iyz="0" izz="0" xyz="-0.002314 -0.187551 0.067613" /> -->
-            <xacro:inertial_matrix_bis mass="0.055" />
+            <origin rpy="${PI} 0 0" xyz="0.005 -0.165 0.067" />
+        </collision>
+        <xacro:inertial_matrix_bis mass="0.055" />
     </link>
     <gazebo reference="wrist" />
@@ -109,5 +120,5 @@
                 <mesh filename="package://lynxmotion_al5d_description/meshes/robot_parts/gripper.dae" />
             </geometry>
-            <origin rpy="${PI/2} 0 ${-PI/2}" xyz="0 0 0" />
+            <origin rpy="${PI/2} 0 ${-PI/2}" xyz="0 -0.021 -0.005" />
         </visual>
         <collision>
@@ -115,7 +126,6 @@
                 <mesh filename="package://lynxmotion_al5d_description/meshes/robot_parts/gripper.dae" />
             </geometry>
-            <origin rpy="${PI/2} 0 ${-PI/2}" xyz="0 0 0" />
-        </collision>
-        <!--<xacro:inertial_matrix mass="0.031" ixx="0" ixy="0" ixz="0" iyy="0" iyz="0" izz="0" xyz="-0.007640 0.007645 0.002347" /> -->
+            <origin rpy="${PI/2} 0 ${-PI/2}" xyz="0 -0.021 -0.005" />
+        </collision>
         <xacro:inertial_matrix_bis mass="0.042" />
     </link>
@@ -126,5 +136,5 @@
                 <mesh filename="package://lynxmotion_al5d_description/meshes/robot_parts/finger_left.dae" />
             </geometry>
-            <origin rpy="${PI/2} 0 ${-PI/2}" xyz="0 0 0" />
+            <origin rpy="${PI/2} 0 ${-PI/2}" xyz="0.003 -0.012 0" />
         </visual>
         <collision>
@@ -132,7 +142,6 @@
                 <mesh filename="package://lynxmotion_al5d_description/meshes/robot_parts/finger_left.dae" />
             </geometry>
-            <origin rpy="${PI/2} 0 ${-PI/2}" xyz="0 0 0" />
-        </collision>
-        <!-- <xacro:inertial_matrix mass="0.02" ixx="0" ixy="0" ixz="0" iyy="0" iyz="0" izz="0" xyz="0.01688 0.003755 -0.016411"/> -->
+            <origin rpy="${PI/2} 0 ${-PI/2}" xyz="0.003 -0.012 0" />
+        </collision>
         <xacro:inertial_matrix_bis mass="0.0006" />
     </link>
@@ -143,5 +152,5 @@
                 <mesh filename="package://lynxmotion_al5d_description/meshes/robot_parts/finger_right.dae" />
             </geometry>
-            <origin rpy="${PI/2} 0 ${-PI/2}" xyz="0 0 0" />
+            <origin rpy="${PI/2} 0 ${-PI/2}" xyz="-0.003 -0.012 0" />
         </visual>
         <collision>
@@ -149,7 +158,6 @@
                 <mesh filename="package://lynxmotion_al5d_description/meshes/robot_parts/finger_right.dae" />
             </geometry>
-            <origin rpy="${PI/2} 0 ${-PI/2}" xyz="0 0 0" />
-        </collision>
-         <!-- <xacro:inertial_matrix mass="0.02" ixx="0" ixy="0" ixz="0" iyy="0" iyz="0" izz="0" xyz="0.01688 0.003755 -0.016411"/> -->
+            <origin rpy="${PI/2} 0 ${-PI/2}" xyz="-0.003 -0.012 0" />
+        </collision>
         <xacro:inertial_matrix_bis mass="0.0006" />
     </link>
@@ -181,5 +189,5 @@
     </sensor>
     <!-- Adding joints -->
-    <!--<joint name="world_to_robot" type="fixed">
+    <!-- <joint name="world_to_robot" type="fixed">
         <parent link="world" />
         <child link="robot_support" />
@@ -192,5 +200,5 @@
         <dynamics damping="10" friction="0.7" />
     </joint>
-    <joint name="link1_rotz" type="revolute">
+    <joint name="Joint1" type="revolute">
         <parent link="robot_support" />
         <child link="robot_base_cylinder" />
@@ -201,62 +209,64 @@
         <dynamics damping="10" friction="0.7" />
     </joint>
-    <joint name="robot_base_fixed" type="fixed">
+    <joint name="base_to_cylinder" type="fixed">
         <parent link="robot_base_cylinder" />
         <child link="robot_base_top_box" />
         <dynamics damping="10" friction="0.7" />
     </joint>
-    <joint name="link1_rotx" type="revolute">
+    <joint name="Joint2" type="revolute">
         <parent link="robot_base_top_box" />
         <child link="shoulder" />
         <axis xyz="1 0 0" />
         <origin xyz="0 -0.015 0.071" />
-        <limit effort="10" velocity="1" lower="${-PI/2}" upper="${PI/2}" />
-        <dynamics damping="10" friction="0.7" />
-    </joint>
-    <joint name="link2_rotx" type="revolute">
+        <limit effort="10" velocity="1" lower="0" upper="${PI}" />
+        <dynamics damping="10" friction="0.7" />
+    </joint>
+    <joint name="Joint3" type="revolute">
         <parent link="shoulder" />
         <child link="arm" />
         <axis xyz="1 0 0" />
-        <origin xyz="0 0 ${shoulder_to_elbow}" />
+        <origin xyz="0 ${shoulder_to_elbow} 0" />
         <limit effort="10" velocity="1" lower="${-PI/2}" upper="${PI/2}" />
         <dynamics damping="10" friction="0.7" />
     </joint>
-    <joint name="link3_rotx" type="revolute">
+    <joint name="Joint4" type="revolute">
         <parent link="arm" />
         <child link="wrist" />
         <axis xyz="1 0 0" />
-        <origin xyz="0 ${-tube_length - hs_645_depth + 0.003} 0" />
+        <origin xyz="0 ${-tube_length - hs_645_depth + 0.003} 0" rpy="0 0 ${PI}"/>
         <limit effort="10" velocity="1" lower="${-PI/2}" upper="${PI/2}" />
         <dynamics damping="10" friction="0.7" />
     </joint>
-   <joint name="link4_rotz" type="revolute">
+   <joint name="Joint5" type="revolute">
         <parent link="wrist" />
         <child link="gripper" />
         <axis xyz="0 1 0" />
-        <origin xyz="0 -0.055 0" rpy="0 0 0" />
+        <origin xyz="0 0.04 -0.005" rpy="0 0 ${PI}" />
         <limit effort="10" velocity="1" lower="${-PI}" upper="${PI}" />
         <dynamics damping="10" friction="0.7" />
     </joint>
-   <joint name="finger_left_mov" type="prismatic">
+   <joint name="Gripper" type="prismatic">
         <parent link="gripper" />
         <child link="left_finger" />
+        <origin xyz="0 -0.01 0" />
         <limit effort="10" velocity="0.005" upper="0" lower="${-gripper_base_width/2}" />
         <dynamics damping="10" friction="0.7" />
     </joint>
-   <joint name="finger_right_mov" type="prismatic">
+   <joint name="GripperBis" type="prismatic">
         <parent link="gripper" />
         <child link="right_finger" />
+        <origin xyz="0 -0.01 0" />
         <limit effort="10" velocity="0.001" lower="0" upper="${gripper_base_width/2}" />
-        <mimic joint="finger_left_mov" multiplier="-1" />
+        <mimic joint="Gripper" multiplier="-1" />
         <dynamics damping="10" friction="0.7" />
     </joint>
     <!-- Setting transmissions -->
-    <xacro:transmission_block joint_name="link1_rotx"/>
-    <xacro:transmission_block joint_name="link1_rotz"/>
-    <xacro:transmission_block joint_name="link2_rotx"/>
-    <xacro:transmission_block joint_name="link3_rotx"/>
-    <xacro:transmission_block joint_name="link4_rotz"/>
-    <xacro:transmission_block_finger joint_name="finger_right_mov"/>
-    <xacro:transmission_block_finger joint_name="finger_left_mov"/>
+    <xacro:transmission_block joint_name="Joint1"/>
+    <xacro:transmission_block joint_name="Joint2"/>
+    <xacro:transmission_block joint_name="Joint3"/>
+    <xacro:transmission_block joint_name="Joint4"/>
+    <xacro:transmission_block joint_name="Joint5"/>
+    <xacro:transmission_block_finger joint_name="Gripper"/>
+    <xacro:transmission_block_finger joint_name="GripperBis"/>
       <!-- ros_control plugin -->
     <gazebo>

Commit message: Update package reference

File: urdf/lynxmotion_al5d.xacro (robot description, xacro)
@@ -1,10 +1,10 @@
 <?xml version="1.0" ?>
 <robot name="lynxmotion_al5d" xmlns:xacro="http://www.ros.org/wiki/xacro" xmlns:sensor="http://playerstage.sourceforge.net/gazebo/xmlschema/#sensor" xmlns:controller="http://playerstage.sourceforge.net/gazebo/xmlschema/#controller" xmlns:interface="http://playerstage.sourceforge.net/gazebo/xmlschema/#interface">
-    <xacro:include filename="$(find al5d_description)/urdf/lynxmotion_al5d_properties.urdf.xacro" />
+    <xacro:include filename="$(find lynxmotion_al5d_description)/urdf/lynxmotion_al5d_properties.urdf.xacro" />
     <!-- Base link comprising the board behind the robot and the cylinder at its bottom -->
     <link name="base_link">
         <visual>
             <geometry>
-                <mesh filename="package://al5d_description/meshes/robot_parts/support.dae" />
+                <mesh filename="package://lynxmotion_al5d_description/meshes/robot_parts/support.dae" />
             </geometry>
             <origin rpy="0 0 0" xyz="0 0 0" />
@@ -12,5 +12,5 @@
         <collision>
             <geometry>
-                <mesh filename="package://al5d_description/meshes/robot_parts/support.dae" />
+                <mesh filename="package://lynxmotion_al5d_description/meshes/robot_parts/support.dae" />
             </geometry>
             <origin rpy="0 0 0" xyz="0 0 0" />
@@ -22,5 +22,5 @@
         <visual>
             <geometry>
-                <mesh filename="package://al5d_description/meshes/robot_parts/rotation_cylinder.dae" />
+                <mesh filename="package://lynxmotion_al5d_description/meshes/robot_parts/rotation_cylinder.dae" />
             </geometry>
             <origin rpy="0 0 0" xyz="0 -0.021165 0" />
@@ -28,5 +28,5 @@
         <collision>
             <geometry>
-                <mesh filename="package://al5d_description/meshes/robot_parts/rotation_cylinder.dae" />
+                <mesh filename="package://lynxmotion_al5d_description/meshes/robot_parts/rotation_cylinder.dae" />
             </geometry>
             <origin rpy="0 0 0" xyz="0 -0.021165 0" />
@@ -38,5 +38,5 @@
         <visual>
             <geometry>
-                <mesh filename="package://al5d_description/meshes/robot_parts/top_box.dae" />
+                <mesh filename="package://lynxmotion_al5d_description/meshes/robot_parts/top_box.dae" />
             </geometry>
             <origin xyz="0.007 -0.024 0" rpy="0 0 0" />
@@ -44,5 +44,5 @@
         <collision>
             <geometry>
-                <mesh filename="package://al5d_description/meshes/robot_parts/top_box.dae" />
+                <mesh filename="package://lynxmotion_al5d_description/meshes/robot_parts/top_box.dae" />
             </geometry>
             <origin xyz="0.007 -0.024 0" rpy="0 0 0" />
@@ -54,5 +54,5 @@
         <visual>
             <geometry>
-                <mesh filename="package://al5d_description/meshes/robot_parts/shoulder.dae" />
+                <mesh filename="package://lynxmotion_al5d_description/meshes/robot_parts/shoulder.dae" />
             </geometry>
             <origin rpy="${-5*PI/8} 0 0" xyz="0 -0.0625 0.036" />
@@ -60,5 +60,5 @@
         <collision>
             <geometry>
-                <mesh filename="package://al5d_description/meshes/robot_parts/shoulder.dae" />
+                <mesh filename="package://lynxmotion_al5d_description/meshes/robot_parts/shoulder.dae" />
             </geometry>
             <origin rpy="${-5*PI/8} 0 0" xyz="0 -0.0625 0.036" />
@@ -70,5 +70,5 @@
         <visual>
             <geometry>
-                <mesh filename="package://al5d_description/meshes/robot_parts/arm.dae" />
+                <mesh filename="package://lynxmotion_al5d_description/meshes/robot_parts/arm.dae" />
             </geometry>
             <origin rpy="-0.895 0 0" xyz="0 ${-tube_length + 2*hs_755eb_depth/5} ${-shoulder_to_elbow - 0.02}" />
@@ -76,5 +76,5 @@
         <collision>
             <geometry>
-                <mesh filename="package://al5d_description/meshes/robot_parts/arm.dae" />
+                <mesh filename="package://lynxmotion_al5d_description/meshes/robot_parts/arm.dae" />
             </geometry>
             <origin rpy="-0.895 0 0" xyz="0 ${-tube_length + 2*hs_755eb_depth/5} ${-shoulder_to_elbow - 0.02}" />
@@ -86,5 +86,5 @@
         <visual>
             <geometry>
-                <mesh filename="package://al5d_description/meshes/robot_parts/wrist.dae" />
+                <mesh filename="package://lynxmotion_al5d_description/meshes/robot_parts/wrist.dae" />
             </geometry>
             <origin rpy="${PI} 0 0" xyz="0.005 -0.165 0.067" />
@@ -92,5 +92,5 @@
         <collision>
             <geometry>
-                <mesh filename="package://al5d_description/meshes/robot_parts/wrist.dae" />
+                <mesh filename="package://lynxmotion_al5d_description/meshes/robot_parts/wrist.dae" />
             </geometry>
             <origin rpy="${PI} 0 0" xyz="0.005 -0.165 0.067" />
@@ -102,5 +102,5 @@
         <visual>
             <geometry>
-                <mesh filename="package://al5d_description/meshes/robot_parts/gripper.dae" />
+                <mesh filename="package://lynxmotion_al5d_description/meshes/robot_parts/gripper.dae" />
             </geometry>
             <origin rpy="${PI/2} 0 ${-PI/2}" xyz="0 -0.021 -0.005" />
@@ -108,5 +108,5 @@
         <collision>
             <geometry>
-                <mesh filename="package://al5d_description/meshes/robot_parts/gripper.dae" />
+                <mesh filename="package://lynxmotion_al5d_description/meshes/robot_parts/gripper.dae" />
             </geometry>
             <origin rpy="${PI/2} 0 ${-PI/2}" xyz="0 -0.021 -0.005" />
@@ -118,5 +118,5 @@
         <visual>
             <geometry>
-                <mesh filename="package://al5d_description/meshes/robot_parts/finger_left.dae" />
+                <mesh filename="package://lynxmotion_al5d_description/meshes/robot_parts/finger_left.dae" />
             </geometry>
             <origin rpy="${PI/2} 0 ${-PI/2}" xyz="0.003 -0.012 0" />
@@ -124,5 +124,5 @@
         <collision>
             <geometry>
-                <mesh filename="package://al5d_description/meshes/robot_parts/finger_left.dae" />
+                <mesh filename="package://lynxmotion_al5d_description/meshes/robot_parts/finger_left.dae" />
             </geometry>
             <origin rpy="${PI/2} 0 ${-PI/2}" xyz="0.003 -0.012 0" />
@@ -134,5 +134,5 @@
         <visual>
             <geometry>
-                <mesh filename="package://al5d_description/meshes/robot_parts/finger_right.dae" />
+                <mesh filename="package://lynxmotion_al5d_description/meshes/robot_parts/finger_right.dae" />
             </geometry>
             <origin rpy="${PI/2} 0 ${-PI/2}" xyz="-0.003 -0.012 0" />
@@ -140,5 +140,5 @@
         <collision>
             <geometry>
-                <mesh filename="package://al5d_description/meshes/robot_parts/finger_right.dae" />
+                <mesh filename="package://lynxmotion_al5d_description/meshes/robot_parts/finger_right.dae" />
             </geometry>
             <origin rpy="${PI/2} 0 ${-PI/2}" xyz="-0.003 -0.012 0" />

Commit message: Making distance working

File: urdf/lynxmotion_al5d.xacro (robot description, xacro)
@@ -130,5 +130,5 @@
             <origin rpy="${PI/2} 0 ${-PI/2}" xyz="0 -0.012 0" />
         </collision>
-        <xacro:inertial_matrix_bis mass="0.0006" />
+        <xacro:inertial_matrix_bis mass="0.006" />
     </link>
     <gazebo reference="left_finger" />
@@ -146,5 +146,5 @@
             <origin rpy="${PI/2} 0 ${-PI/2}" xyz="-0.003 -0.012 0" />
         </collision>
-        <xacro:inertial_matrix_bis mass="0.0006" />
+        <xacro:inertial_matrix_bis mass="0.006" />
     </link>
     <gazebo reference="right_finger" />
@@ -229,18 +229,45 @@
         <dynamics damping="10" friction="0.7" />
     </joint>
-    <joint name="Gripper" type="prismatic">
+    <joint name="right_finger_joint" type="prismatic">
         <parent link="gripper" />
         <child link="right_finger" />
         <origin xyz="0 -0.01 0" />
         <limit effort="10" velocity="0.01" lower="0" upper="${gripper_base_width/2}" />
-        <dynamics damping="10" friction="0.7" />
-    </joint>
-   <joint name="GripperBis" type="prismatic">
+        <mimic joint="Gripper" multiplier="-0.5" offset="${gripper_base_width/2}" />
+        <dynamics damping="10" friction="1" />
+    </joint>
+   <joint name="left_finger_joint" type="prismatic">
         <parent link="gripper" />
         <child link="left_finger" />
         <origin xyz="0 -0.01 0" />
-        <limit effort="10" velocity="0.01" upper="0" lower="${-gripper_base_width/2}" />
-        <mimic joint="Gripper" multiplier="-1" />
-        <dynamics damping="10" friction="0.7" />
+        <axis xyz="-1 0 0" />
+        <limit effort="10" velocity="0.01" lower="0" upper="${gripper_base_width/2}" />
+        <mimic joint="right_finger_joint" />
+        <dynamics damping="10" friction="1" />
+    </joint>
+    <link name="gripper_mov">
+        <visual>
+            <origin xyz="0 0 0" rpy="0 0 0" />
+            <geometry>
+                <box size="0.01 0.01 0.01" />
+            </geometry>
+            <material name="Transparent" />
+        </visual>
+        <collision>
+            <origin xyz="0 0 0" rpy="0 0 0" />
+            <geometry>
+                <box size="0.01 0.01 0.01" />
+            </geometry>
+        </collision>
+        <xacro:inertial_matrix_box mass="0.01" width="0.01" height="0.01" depth="0.01" />
+    </link>
+    <gazebo reference="gripper_mov" /> -->
+    <joint name="Gripper" type="revolute">
+        <parent link="world" />
+        <child link="gripper_mov" />
+        <origin xyz="0 -0.2 0" />
+        <limit lower="0" upper="${gripper_base_width}" effort="10" velocity="0.01" />
+        <axis xyz="1 0 0" />
+        <dynamics damping="50" friction="1" />
     </joint>
     <!-- Setting transmissions -->
@@ -258,7 +285,10 @@
         </plugin>
     </gazebo>
-    <xacro:mimic_joint_plugin_gazebo name_prefix="gripper_"
-    parent_joint="Gripper" mimic_joint="GripperBis"
-    has_pid="true" multiplier="-1.0" max_effort="10.0" />
+    <xacro:mimic_joint_plugin_gazebo name_prefix="finger_right"
+    parent_joint="Gripper" mimic_joint="right_finger_joint"
+    has_pid="true" multiplier="-0.5" max_effort="10.0" offset="${gripper_base_width/2}" />
+    <xacro:mimic_joint_plugin_gazebo name_prefix="finger_left_"
+    parent_joint="right_finger_joint" mimic_joint="left_finger_joint"
+    has_pid="true" max_effort="10.0" />
     <gazebo reference="camera_link">
         <sensor name="external_camera" type="camera">
