Commit message: Fixed issues with the mimic plugin integration to the robot

File: urdf/lynxmotion_al5d.xacro (robot description, xacro)
@@ -122,5 +122,5 @@
                 <mesh filename="package://lynxmotion_al5d_description/meshes/robot_parts/finger_left.dae" />
             </geometry>
-            <origin rpy="${PI/2} 0 ${-PI/2}" xyz="0 -0.012 0" />
+            <origin rpy="${PI/2} 0 ${-PI/2}" xyz="0 -0.009 0" />
         </visual>
         <collision>
@@ -128,5 +128,5 @@
                 <mesh filename="package://lynxmotion_al5d_description/meshes/robot_parts/finger_left.dae" />
             </geometry>
-            <origin rpy="${PI/2} 0 ${-PI/2}" xyz="0 -0.012 0" />
+            <origin rpy="${PI/2} 0 ${-PI/2}" xyz="0 -0.009 0" />
         </collision>
         <xacro:inertial_matrix_bis mass="0.006" />
@@ -138,5 +138,5 @@
                 <mesh filename="package://lynxmotion_al5d_description/meshes/robot_parts/finger_right.dae" />
             </geometry>
-            <origin rpy="${PI/2} 0 ${-PI/2}" xyz="0 -0.012 0" />
+            <origin rpy="${PI/2} 0 ${-PI/2}" xyz="0 -0.009 0" />
         </visual>
         <collision>
@@ -144,9 +144,27 @@
                 <mesh filename="package://lynxmotion_al5d_description/meshes/robot_parts/finger_right.dae" />
             </geometry>
-            <origin rpy="${PI/2} 0 ${-PI/2}" xyz="-0.003 -0.012 0" />
+            <origin rpy="${PI/2} 0 ${-PI/2}" xyz="0 -0.009 0" />
         </collision>
         <xacro:inertial_matrix_bis mass="0.006" />
     </link>
     <gazebo reference="right_finger" />
+    <!-- Dummy link used for the gripper -->
+    <link name="gripper_mov">
+        <visual>
+            <origin xyz="0 0 0" rpy="0 0 0" />
+            <geometry>
+                <box size="0.001 0.001 0.001" />
+            </geometry>
+            <material name="Transparent" />
+        </visual>
+        <collision>
+            <origin xyz="0 0 0" rpy="0 0 0" />
+            <geometry>
+                <box size="0.001 0.001 0.001" />
+            </geometry>
+        </collision>
+        <xacro:inertial_matrix_box mass="0.0001" width="0.01" height="0.01" depth="0.01" />
+    </link>
+    <gazebo reference="gripper_mov" />
     <link name="camera_link">
         <visual>
@@ -190,5 +208,5 @@
         <origin xyz="0 0.021 0" rpy="0 0 ${PI}" />
         <limit effort="10" velocity="1" lower="${-PI}" upper="${PI}" />
-        <dynamics damping="50" friction="1" />
+        <dynamics damping="20" friction="1" />
     </joint>
     <joint name="base_to_cylinder" type="fixed">
@@ -203,5 +221,5 @@
         <origin xyz="0 0.015 0.071"  rpy="0 0 0" />
         <limit effort="10" velocity="1" lower="0" upper="${PI}" />
-        <dynamics damping="50" friction="1" />
+        <dynamics damping="20" friction="1" />
     </joint>
     <joint name="Joint3" type="revolute">
@@ -211,5 +229,5 @@
         <origin xyz="0 ${shoulder_to_elbow} 0" />
         <limit effort="10" velocity="1" lower="${-PI/2}" upper="${PI/2}" />
-        <dynamics damping="50" friction="1" />
+        <dynamics damping="20" friction="1" />
     </joint>
     <joint name="Joint4" type="revolute">
@@ -219,5 +237,5 @@
         <origin xyz="0 ${tube_length + hs_645_depth - 0.003} 0" rpy="0 0 0"/>
         <limit effort="10" velocity="1" lower="${-PI/2}" upper="${PI/2}" />
-        <dynamics damping="50" friction="1" />
+        <dynamics damping="20" friction="1" />
     </joint>
    <joint name="Joint5" type="revolute">
@@ -227,47 +245,28 @@
         <origin xyz="0 0.04 -0.005" rpy="0 0 ${PI}" />
         <limit effort="10" velocity="1" lower="${-PI}" upper="${PI}" />
-        <dynamics damping="10" friction="0.7" />
+        <dynamics damping="20" friction="0.7" />
     </joint>
     <joint name="right_finger_joint" type="prismatic">
         <parent link="gripper" />
         <child link="right_finger" />
-        <origin xyz="0 -0.01 0" />
+        <origin xyz="0 -0.015 0" />
         <limit effort="10" velocity="0.01" lower="0" upper="${gripper_base_width/2}" />
         <mimic joint="Gripper" multiplier="-0.5" offset="${gripper_base_width/2}" />
-        <dynamics damping="10" friction="1" />
     </joint>
    <joint name="left_finger_joint" type="prismatic">
         <parent link="gripper" />
         <child link="left_finger" />
-        <origin xyz="0 -0.01 0" />
+        <origin xyz="0 -0.015 0" />
         <axis xyz="-1 0 0" />
         <limit effort="10" velocity="0.01" lower="0" upper="${gripper_base_width/2}" />
         <mimic joint="right_finger_joint" />
-        <dynamics damping="10" friction="1" />
-    </joint>
-    <link name="gripper_mov">
-        <visual>
-            <origin xyz="0 0 0" rpy="0 0 0" />
-            <geometry>
-                <box size="0.01 0.01 0.01" />
-            </geometry>
-            <material name="Transparent" />
-        </visual>
-        <collision>
-            <origin xyz="0 0 0" rpy="0 0 0" />
-            <geometry>
-                <box size="0.01 0.01 0.01" />
-            </geometry>
-        </collision>
-        <xacro:inertial_matrix_box mass="0.01" width="0.01" height="0.01" depth="0.01" />
-    </link>
-    <gazebo reference="gripper_mov" /> -->
-    <joint name="Gripper" type="revolute">
-        <parent link="world" />
+    </joint>
+    <joint name="Gripper" type="prismatic">
+        <parent link="gripper" />
         <child link="gripper_mov" />
-        <origin xyz="0 -0.2 0" />
+        <origin xyz="${gripper_base_width/2} 0  0" />
         <limit lower="0" upper="${gripper_base_width}" effort="10" velocity="0.01" />
-        <axis xyz="1 0 0" />
-        <dynamics damping="50" friction="1" />
+        <axis xyz="-1 0 0" />
+        <dynamics damping="10" friction="0.7" />
     </joint>
     <!-- Setting transmissions -->
@@ -285,4 +284,5 @@
         </plugin>
     </gazebo>
+    <!-- Setting the mimic joints plugin -->
     <xacro:mimic_joint_plugin_gazebo name_prefix="finger_right"
     parent_joint="Gripper" mimic_joint="right_finger_joint"

Commit message: Right finger working properly

File: urdf/lynxmotion_al5d.xacro (robot description, xacro)
@@ -122,5 +122,5 @@
                 <mesh filename="package://lynxmotion_al5d_description/meshes/robot_parts/finger_left.dae" />
             </geometry>
-            <origin rpy="${PI/2} 0 ${-PI/2}" xyz="0 -0.009 0" />
+            <origin rpy="${PI/2} 0 ${-PI/2}" xyz="0.003 -0.009 0" />
         </visual>
         <collision>
@@ -138,5 +138,5 @@
                 <mesh filename="package://lynxmotion_al5d_description/meshes/robot_parts/finger_right.dae" />
             </geometry>
-            <origin rpy="${PI/2} 0 ${-PI/2}" xyz="0 -0.009 0" />
+            <origin rpy="${PI/2} 0 ${-PI/2}" xyz="-0.003 -0.009 0" />
         </visual>
         <collision>
@@ -154,15 +154,15 @@
             <origin xyz="0 0 0" rpy="0 0 0" />
             <geometry>
-                <box size="0.001 0.001 0.001" />
-            </geometry>
-            <material name="Transparent" />
+                <box size="0.01 0.01 0.01" />
+            </geometry>
+            <material name="Black" />
         </visual>
         <collision>
             <origin xyz="0 0 0" rpy="0 0 0" />
             <geometry>
-                <box size="0.001 0.001 0.001" />
-            </geometry>
-        </collision>
-        <xacro:inertial_matrix_box mass="0.0001" width="0.01" height="0.01" depth="0.01" />
+                <box size="0.01 0.01 0.01" />
+            </geometry>
+        </collision>
+        <xacro:inertial_matrix_box mass="0.01" width="0.01" height="0.01" depth="0.01" />
     </link>
     <gazebo reference="gripper_mov" />
@@ -196,4 +196,5 @@
         <parent link="world" />
         <child link="robot_support" />
+        <dynamics damping="20" friction="1" />
     </joint>
     <joint name="camera_joint" type="fixed">
@@ -201,4 +202,5 @@
         <child link="camera_link" />
         <origin xyz="0 -0.35 0" />
+        <dynamics damping="20" friction="1" />
     </joint>
    <joint name="Joint1" type="revolute">
@@ -245,5 +247,5 @@
         <origin xyz="0 0.04 -0.005" rpy="0 0 ${PI}" />
         <limit effort="10" velocity="1" lower="${-PI}" upper="${PI}" />
-        <dynamics damping="20" friction="0.7" />
+        <dynamics damping="20" friction="1" />
     </joint>
     <joint name="right_finger_joint" type="prismatic">
@@ -253,4 +255,5 @@
         <limit effort="10" velocity="0.01" lower="0" upper="${gripper_base_width/2}" />
         <mimic joint="Gripper" multiplier="-0.5" offset="${gripper_base_width/2}" />
+        <!-- <dynamics damping="10" friction="0.7" /> -->
     </joint>
    <joint name="left_finger_joint" type="prismatic">
@@ -261,9 +264,10 @@
         <limit effort="10" velocity="0.01" lower="0" upper="${gripper_base_width/2}" />
         <mimic joint="right_finger_joint" />
+        <dynamics damping="10" friction="0.7" />
     </joint>
     <joint name="Gripper" type="prismatic">
         <parent link="gripper" />
         <child link="gripper_mov" />
-        <origin xyz="${gripper_base_width/2} 0  0" />
+        <origin xyz="0.01 0  0" />
         <limit lower="0" upper="${gripper_base_width}" effort="10" velocity="0.01" />
         <axis xyz="-1 0 0" />
@@ -288,7 +292,7 @@
     parent_joint="Gripper" mimic_joint="right_finger_joint"
     has_pid="true" multiplier="-0.5" max_effort="10.0" offset="${gripper_base_width/2}" />
-    <xacro:mimic_joint_plugin_gazebo name_prefix="finger_left_"
+    <!-- <xacro:mimic_joint_plugin_gazebo name_prefix="finger_left_"
     parent_joint="right_finger_joint" mimic_joint="left_finger_joint"
-    has_pid="true" max_effort="10.0" />
+    has_pid="true" max_effort="10.0" sensitiveness="0.01" /> -->
     <gazebo reference="camera_link">
         <sensor name="external_camera" type="camera">

Commit message: Bug fixes and improvement

File: urdf/lynxmotion_al5d.xacro (robot description, xacro)
@@ -122,5 +122,5 @@
                 <mesh filename="package://lynxmotion_al5d_description/meshes/robot_parts/finger_left.dae" />
             </geometry>
-            <origin rpy="${PI/2} 0 ${-PI/2}" xyz="0.003 -0.009 0" />
+            <origin rpy="${PI/2} 0 ${-PI/2}" xyz="0.0028 -0.009 0" />
         </visual>
         <collision>
@@ -128,5 +128,5 @@
                 <mesh filename="package://lynxmotion_al5d_description/meshes/robot_parts/finger_left.dae" />
             </geometry>
-            <origin rpy="${PI/2} 0 ${-PI/2}" xyz="0 -0.009 0" />
+            <origin rpy="${PI/2} 0 ${-PI/2}" xyz="0.0028 -0.009 0" />
         </collision>
         <xacro:inertial_matrix_bis mass="0.006" />
@@ -138,5 +138,5 @@
                 <mesh filename="package://lynxmotion_al5d_description/meshes/robot_parts/finger_right.dae" />
             </geometry>
-            <origin rpy="${PI/2} 0 ${-PI/2}" xyz="-0.003 -0.009 0" />
+            <origin rpy="${PI/2} 0 ${-PI/2}" xyz="-0.0028 -0.009 0" />
         </visual>
         <collision>
@@ -144,5 +144,5 @@
                 <mesh filename="package://lynxmotion_al5d_description/meshes/robot_parts/finger_right.dae" />
             </geometry>
-            <origin rpy="${PI/2} 0 ${-PI/2}" xyz="0 -0.009 0" />
+            <origin rpy="${PI/2} 0 ${-PI/2}" xyz="-0.0028 -0.009 0" />
         </collision>
         <xacro:inertial_matrix_bis mass="0.006" />
@@ -209,5 +209,5 @@
         <axis xyz="0 0 -1" />
         <origin xyz="0 0.021 0" rpy="0 0 ${PI}" />
-        <limit effort="10" velocity="1" lower="${-PI}" upper="${PI}" />
+        <limit effort="100" velocity="5" lower="${-PI}" upper="${PI}" />
         <dynamics damping="20" friction="1" />
     </joint>
@@ -222,5 +222,5 @@
         <axis xyz="1 0 0"/>
         <origin xyz="0 0.015 0.071"  rpy="0 0 0" />
-        <limit effort="10" velocity="1" lower="0" upper="${PI}" />
+        <limit effort="100" velocity="5" lower="0" upper="${PI}" />
         <dynamics damping="20" friction="1" />
     </joint>
@@ -230,5 +230,5 @@
         <axis xyz="1 0 0" />
         <origin xyz="0 ${shoulder_to_elbow} 0" />
-        <limit effort="10" velocity="1" lower="${-PI/2}" upper="${PI/2}" />
+        <limit effort="100" velocity="5" lower="${-PI/2}" upper="${PI/2}" />
         <dynamics damping="20" friction="1" />
     </joint>
@@ -238,5 +238,5 @@
         <axis xyz="1 0 0" />
         <origin xyz="0 ${tube_length + hs_645_depth - 0.003} 0" rpy="0 0 0"/>
-        <limit effort="10" velocity="1" lower="${-PI/2}" upper="${PI/2}" />
+        <limit effort="40" velocity="5" lower="${-PI/2}" upper="${PI/2}" />
         <dynamics damping="20" friction="1" />
     </joint>
@@ -246,6 +246,6 @@
         <axis xyz="0 1 0" />
         <origin xyz="0 0.04 -0.005" rpy="0 0 ${PI}" />
-        <limit effort="10" velocity="1" lower="${-PI}" upper="${PI}" />
-        <dynamics damping="20" friction="1" />
+        <limit effort="100" velocity="5" lower="${-PI}" upper="${PI}" />
+        <dynamics damping="10" friction="0.7" />
     </joint>
     <joint name="right_finger_joint" type="prismatic">
@@ -253,7 +253,6 @@
         <child link="right_finger" />
         <origin xyz="0 -0.015 0" />
-        <limit effort="10" velocity="0.01" lower="0" upper="${gripper_base_width/2}" />
+        <limit effort="10" velocity="0.1" lower="0" upper="${gripper_base_width/2}" />
         <mimic joint="Gripper" multiplier="-0.5" offset="${gripper_base_width/2}" />
-        <!-- <dynamics damping="10" friction="0.7" /> -->
     </joint>
    <joint name="left_finger_joint" type="prismatic">
@@ -262,15 +261,14 @@
         <origin xyz="0 -0.015 0" />
         <axis xyz="-1 0 0" />
-        <limit effort="10" velocity="0.01" lower="0" upper="${gripper_base_width/2}" />
+        <limit effort="10" velocity="0.1" lower="0" upper="${gripper_base_width/2}" />
         <mimic joint="right_finger_joint" />
-        <dynamics damping="10" friction="0.7" />
-    </joint>
+    </joint>
+    <!-- Joint that accept the distance between the two fingers as parameter -->
     <joint name="Gripper" type="prismatic">
         <parent link="gripper" />
         <child link="gripper_mov" />
         <origin xyz="0.01 0  0" />
-        <limit lower="0" upper="${gripper_base_width}" effort="10" velocity="0.01" />
+        <limit lower="0" upper="${gripper_base_width}" effort="10" velocity="0.1" />
         <axis xyz="-1 0 0" />
-        <dynamics damping="10" friction="0.7" />
     </joint>
     <!-- Setting transmissions -->
@@ -292,7 +290,7 @@
     parent_joint="Gripper" mimic_joint="right_finger_joint"
     has_pid="true" multiplier="-0.5" max_effort="10.0" offset="${gripper_base_width/2}" />
-    <!-- <xacro:mimic_joint_plugin_gazebo name_prefix="finger_left_"
-    parent_joint="right_finger_joint" mimic_joint="left_finger_joint"
-    has_pid="true" max_effort="10.0" sensitiveness="0.01" /> -->
+    <xacro:mimic_joint_plugin_gazebo name_prefix="finger_left"
+    parent_joint="Gripper" mimic_joint="left_finger_joint"
+    has_pid="true" multiplier="-0.5" max_effort="10.0" offset="${gripper_base_width/2}" />
     <gazebo reference="camera_link">
         <sensor name="external_camera" type="camera">

Commit message: Updated documentation

File: urdf/lynxmotion_al5d.xacro (robot description, xacro)
@@ -156,5 +156,5 @@
                 <box size="0.01 0.01 0.01" />
             </geometry>
-            <material name="Black" />
+            <material name="Transparent" />
         </visual>
         <collision>

Commit message: Camera orientation corrected

File: urdf/lynxmotion_al5d.xacro (robot description, xacro)
@@ -172,5 +172,5 @@
                 <box size="0.01 0.01 0.01" />
             </geometry>
-            <origin rpy="0 0 0" xyz="0 0 ${camera_support_depth}" />
+            <origin rpy="0 0 0" xyz="0 0 0" />
             <material name="Transparent" />
         </visual>
@@ -179,5 +179,5 @@
                 <box size="0.01 0.01 0.01" />
             </geometry>
-            <origin rpy="0 0 0" xyz="0 0 ${camera_support_depth}" />
+            <origin rpy="0 0 0" xyz="0 0 0" />
             <material name="Transparent" />
         </collision>
@@ -201,6 +201,5 @@
         <parent link="world" />
         <child link="camera_link" />
-        <origin xyz="0 -0.35 0" />
-        <dynamics damping="20" friction="1" />
+        <origin xyz="0 ${-tube_length - hs_645_depth - gripper_base_height - 0.12} ${camera_support_depth}" />
     </joint>
    <joint name="Joint1" type="revolute">
@@ -293,9 +292,16 @@
     parent_joint="Gripper" mimic_joint="left_finger_joint"
     has_pid="true" multiplier="-0.5" max_effort="10.0" offset="${gripper_base_width/2}" />
+    <sensor name="camera">
+        <parent link="camera_link" />
+        <origin xyz="0 0 0" rpy="${PI/2} 0 0" />
+        <camera>
+            <image width="640" height="480" hfov="1.41" near="0.01" far="0.04" />
+        </camera>
+    </sensor>
     <gazebo reference="camera_link">
         <sensor name="external_camera" type="camera">
             <update_rate>1.0</update_rate>
             <camera name="camera_top">
-                <horizontal_fov>1.3962634</horizontal_fov>
+                <pose>0 0 0 3.1415 1.5708 1.5708</pose>
                 <image>
                     <width>640</width>
@@ -304,6 +310,6 @@
                 </image>
                 <clip>
-                    <near>0.3</near>
-                    <far>500</far>
+                    <near>0.1</near>
+                    <far>0.3</far>
                 </clip>
             </camera>
@@ -316,10 +322,4 @@
                 <cameraInfoTopicName>camera_info</cameraInfoTopicName>
                 <frameName>camera_link</frameName>
-                <hackBaseline>0.07</hackBaseline>
-                <distortionK1>-0.0545211</distortionK1>
-                <distortionK2>0.06919734</distortionK2>
-                <distortionK3>-0.0241095</distortionK3>
-                <distortionT1>-0.0112245</distortionT1>
-                <distortionT2>0.0</distortionT2>
             </plugin>
         </sensor>

File: urdf/lynxmotion_al5d_properties.urdf.xacro (robot description, xacro)
@@ -59,5 +59,5 @@
     <xacro:property name="wrist_cylinder_length" value="0.005" />
     <xacro:property name="wrist_cylinder_radius" value="0.01" />
-    <xacro:property name="camera_support_depth" value="0.3" />
+    <xacro:property name="camera_support_depth" value="0.25" />
     <xacro:property name="camera_support_size" value="0.01" />
     <xacro:property name="camera_support_big_size" value="0.5" />

Commit message: Changed materials for hidden links

File: urdf/lynxmotion_al5d.xacro (robot description, xacro)
@@ -156,5 +156,5 @@
                 <box size="0.01 0.01 0.01" />
             </geometry>
-            <material name="Transparent" />
+            <material name="transparent">Gazebo/GreyTransparent</material>
         </visual>
         <collision>
@@ -173,5 +173,5 @@
             </geometry>
             <origin rpy="0 0 0" xyz="0 0 0" />
-            <material name="Transparent" />
+            <material name="transparent">Gazebo/GreyTransparent</material>
         </visual>
         <collision>
@@ -180,5 +180,4 @@
             </geometry>
             <origin rpy="0 0 0" xyz="0 0 0" />
-            <material name="Transparent" />
         </collision>
         <xacro:inertial_matrix_bis mass="0.05" />

Commit message: Added lego block + Changed world state and camera position

File: urdf/lynxmotion_al5d.xacro (robot description, xacro)
@@ -170,5 +170,5 @@
         <visual>
             <geometry>
-                <box size="0.01 0.01 0.01" />
+                <box size="0.0001 0.0001 0.0001" />
             </geometry>
             <origin rpy="0 0 0" xyz="0 0 0" />
@@ -177,18 +177,10 @@
         <collision>
             <geometry>
-                <box size="0.01 0.01 0.01" />
+                <box size="0.0001 0.0001 0.0001" />
             </geometry>
             <origin rpy="0 0 0" xyz="0 0 0" />
         </collision>
-        <xacro:inertial_matrix_bis mass="0.05" />
-    </link>
-    <gazebo reference="camera_link" />
-    <sensor name="robot_camera" update_rate="1">
-        <parent link="camera_link" />
-        <origin xyz="0.005 0.005 0.005" rpy="0 0 0" />
-        <camera>
-            <image width="640" height="480" hfov="${PI/2}" format="RGB8" near="${camera_support_depth}" far="${camera_support_depth}" />
-        </camera>
-    </sensor>
+        <xacro:inertial_matrix_bis mass="0.0005" />
+    </link>
     <!-- Adding joints -->
     <joint name="world_to_robot" type="fixed">
@@ -200,5 +192,5 @@
         <parent link="world" />
         <child link="camera_link" />
-        <origin xyz="0 ${-tube_length - hs_645_depth - gripper_base_height - 0.12} ${camera_support_depth}" />
+        <origin xyz="0 -0.17 ${camera_support_depth}" />
     </joint>
    <joint name="Joint1" type="revolute">
@@ -302,4 +294,5 @@
             <update_rate>1.0</update_rate>
             <camera name="camera_top">
+                <horizontal_fov>1.6</horizontal_fov>
                 <pose>0 0 0 3.1415 1.5708 1.5708</pose>
                 <image>
