Commit message: Code fixes

File: urdf/lynxmotion_al5d.xacro (robot description, xacro)
@@ -9,5 +9,5 @@
             <geometry>
                 <mesh filename="package://lynxmotion_al5d_description/meshes/robot_parts/support.dae" />
-            </geometry>
+            </geometry>3
             <origin rpy="0 0 0" xyz="0 0 0" />
         </visual>
@@ -18,5 +18,5 @@
             <origin rpy="0 0 0" xyz="0 0 0" />
         </collision>
-        <xacro:inertial_matrix mass="0.133" ixx="3.6565e-7" ixy="-3.72e-9" ixz="1e-6" iyy="9.404e-8" iyz="4.375e-8" izz="4.1776e-7" xyz="0.000585 0.0602746 0.0170628" />
+        <xacro:inertial_matrix mass="${board_mass}" ixx="3.6565e-7" ixy="-3.72e-9" ixz="1e-6" iyy="9.404e-8" iyz="4.375e-8" izz="4.1776e-7" xyz="0.000585 0.0602746 0.0170628" />
     </link>
     <gazebo reference="robot_support" />
@@ -34,5 +34,5 @@
             <origin rpy="0 0 0" xyz="0 -0.021165 0" />
         </collision>
-        <xacro:inertial_matrix_bis mass="0.042" />
+        <xacro:inertial_matrix_bis mass="${base_mass}" />
     </link>
     <gazebo reference="robot_base_cylinder" />
@@ -50,5 +50,5 @@
             <origin xyz="0.007 -0.024 0" rpy="0 0 0" />
         </collision>
-        <xacro:inertial_matrix_bis mass="0.184" />
+        <xacro:inertial_matrix_bis mass="${top_box_mass}" />
     </link>
     <gazebo reference="robot_base_top_box" />
@@ -58,5 +58,5 @@
                 <mesh filename="package://lynxmotion_al5d_description/meshes/robot_parts/shoulder.dae" />
             </geometry>
-            <origin rpy="${-5*PI/8} 0 0" xyz="0 -0.0625 0.036" />
+            <origin rpy="${-5*PI/8} 0 0" xyz="0.005 -0.0625 0.036" />
         </visual>
         <collision>
@@ -64,7 +64,7 @@
                 <mesh filename="package://lynxmotion_al5d_description/meshes/robot_parts/shoulder.dae" />
             </geometry>
-            <origin rpy="${-5*PI/8} 0 0" xyz="0 -0.0625 0.036" />
-        </collision>
-        <xacro:inertial_matrix_bis mass="0.095" />
+            <origin rpy="${-5*PI/8} 0 0" xyz="0.005 -0.0625 0.036" />
+        </collision>
+        <xacro:inertial_matrix_bis mass="${shoulder_mass}" />
     </link>
     <gazebo reference="shoulder" />
@@ -74,5 +74,5 @@
                 <mesh filename="package://lynxmotion_al5d_description/meshes/robot_parts/arm.dae" />
             </geometry>
-            <origin rpy="${-PI-0.895} 0 0" xyz="0 ${tube_length - 2*hs_755eb_depth/5} ${shoulder_to_elbow + 0.02}" />
+            <origin rpy="${-PI-0.895} ${PI} 0" xyz="-0.005 ${tube_length - 2*hs_755eb_depth/5} ${-shoulder_to_elbow - 0.02} " />
         </visual>
         <collision>
@@ -80,7 +80,7 @@
                 <mesh filename="package://lynxmotion_al5d_description/meshes/robot_parts/arm.dae" />
             </geometry>
-            <origin rpy="${-PI-0.895} 0 0" xyz="0 ${tube_length - 2*hs_755eb_depth/5} ${shoulder_to_elbow + 0.02}" />
-        </collision>
-        <xacro:inertial_matrix_bis mass="0.1" />
+            <origin rpy="${-PI-0.895} ${PI} 0" xyz="-0.005 ${tube_length - 2*hs_755eb_depth/5} ${-shoulder_to_elbow - 0.02} " />
+        </collision>
+        <xacro:inertial_matrix_bis mass="${hs_755eb_mass+ hs_645_mass}" />
     </link>
     <gazebo reference="arm" />
@@ -98,5 +98,5 @@
             <origin rpy="${PI} 0 0" xyz="0.005 -0.165 0.067" />
         </collision>
-        <xacro:inertial_matrix_bis mass="0.055" />
+        <xacro:inertial_matrix_bis mass="${0.031}" />
     </link>
     <gazebo reference="wrist" />
@@ -130,5 +130,5 @@
             <origin rpy="${PI/2} 0 ${-PI/2}" xyz="0.0028 -0.009 0" />
         </collision>
-        <xacro:inertial_matrix_bis mass="0.006" />
+        <xacro:inertial_matrix_bis mass="${finger_mass}" />
     </link>
     <gazebo reference="left_finger" />
@@ -146,5 +146,5 @@
             <origin rpy="${PI/2} 0 ${-PI/2}" xyz="-0.0028 -0.009 0" />
         </collision>
-        <xacro:inertial_matrix_bis mass="0.006" />
+        <xacro:inertial_matrix_bis mass="${finger_mass}" />
     </link>
     <gazebo reference="right_finger" />
@@ -187,10 +187,11 @@
         <parent link="world" />
         <child link="robot_support" />
-        <dynamics damping="20" friction="1" />
+        <origin rpy="0 0 ${PI}" />
+        <dynamics damping="50" friction="1" />
     </joint>
     <joint name="camera_joint" type="fixed">
         <parent link="world" />
         <child link="camera_link" />
-        <origin xyz="0 -0.17 ${camera_support_depth}" />
+        <origin xyz="0 0.17 ${camera_support_depth}" />
     </joint>
    <joint name="Joint1" type="revolute">
@@ -199,11 +200,11 @@
         <axis xyz="0 0 -1" />
         <origin xyz="0 0.021 0" rpy="0 0 ${PI}" />
-        <limit effort="100" velocity="5" lower="${-PI}" upper="${PI}" />
-        <dynamics damping="20" friction="1" />
+        <limit effort="100" velocity="2" lower="${-PI}" upper="${PI}" />
+        <dynamics damping="50" friction="1" />
     </joint>
     <joint name="base_to_cylinder" type="fixed">
         <parent link="robot_base_cylinder" />
         <child link="robot_base_top_box" />
-        <dynamics damping="10" friction="0.7" />
+        <dynamics damping="50" friction="0.7" />
     </joint>
     <joint name="Joint2" type="revolute">
@@ -212,6 +213,6 @@
         <axis xyz="1 0 0"/>
         <origin xyz="0 0.015 0.071"  rpy="0 0 0" />
-        <limit effort="100" velocity="5" lower="0" upper="${PI}" />
-        <dynamics damping="20" friction="1" />
+        <limit effort="100" velocity="2" lower="0" upper="${PI}" />
+        <dynamics damping="50" friction="1" />
     </joint>
     <joint name="Joint3" type="revolute">
@@ -220,6 +221,6 @@
         <axis xyz="1 0 0" />
         <origin xyz="0 ${shoulder_to_elbow} 0" />
-        <limit effort="100" velocity="5" lower="${-PI/2}" upper="${PI/2}" />
-        <dynamics damping="20" friction="1" />
+        <limit effort="100" velocity="2" lower="${-PI/2}" upper="${PI/2}" />
+        <dynamics damping="50" friction="1" />
     </joint>
     <joint name="Joint4" type="revolute">
@@ -227,7 +228,7 @@
         <child link="wrist" />
         <axis xyz="1 0 0" />
-        <origin xyz="0 ${tube_length + hs_645_depth - 0.003} 0" rpy="0 0 0"/>
-        <limit effort="40" velocity="5" lower="${-PI/2}" upper="${PI/2}" />
-        <dynamics damping="20" friction="1" />
+        <origin xyz="0 ${tube_length + hs_645_depth - 0.003} 0.005" rpy="0 0 0"/>
+        <limit effort="40" velocity="2" lower="${-PI/2}" upper="${PI/2}" />
+        <dynamics damping="50" friction="1" />
     </joint>
    <joint name="Joint5" type="revolute">
@@ -235,7 +236,7 @@
         <child link="gripper" />
         <axis xyz="0 1 0" />
-        <origin xyz="0 0.04 -0.005" rpy="0 0 ${PI}" />
-        <limit effort="100" velocity="5" lower="${-PI}" upper="${PI}" />
-        <dynamics damping="10" friction="0.7" />
+        <origin xyz="0 0.04 0" rpy="0 0 ${PI}" />
+        <limit effort="100" velocity="2" lower="${-PI}" upper="${PI}" />
+        <dynamics damping="50" friction="0.7" />
     </joint>
     <joint name="right_finger_joint" type="prismatic">

Commit message: Updating code

File: urdf/lynxmotion_al5d.xacro (robot description, xacro)
@@ -222,5 +222,5 @@
         <origin xyz="0 ${shoulder_to_elbow} 0" />
         <limit effort="100" velocity="2" lower="${-PI/2}" upper="${PI/2}" />
-        <dynamics damping="50" friction="1" />
+        <dynamics damping="20" friction="1" />
     </joint>
     <joint name="Joint4" type="revolute">
@@ -229,6 +229,6 @@
         <axis xyz="1 0 0" />
         <origin xyz="0 ${tube_length + hs_645_depth - 0.003} 0.005" rpy="0 0 0"/>
-        <limit effort="40" velocity="2" lower="${-PI/2}" upper="${PI/2}" />
-        <dynamics damping="50" friction="1" />
+        <limit effort="40" velocity="5" lower="${-PI/2}" upper="${PI/2}" />
+        <dynamics damping="20" friction="1" />
     </joint>
    <joint name="Joint5" type="revolute">
@@ -279,9 +279,7 @@
     <!-- Setting the mimic joints plugin -->
     <xacro:mimic_joint_plugin_gazebo name_prefix="finger_right"
-    parent_joint="Gripper" mimic_joint="right_finger_joint"
-    has_pid="true" multiplier="-0.5" max_effort="10.0" offset="${gripper_base_width/2}" />
+    parent_joint="Gripper" mimic_joint="right_finger_joint" multiplier="-0.5" max_effort="10.0" offset="${gripper_base_width/2}" />
     <xacro:mimic_joint_plugin_gazebo name_prefix="finger_left"
-    parent_joint="Gripper" mimic_joint="left_finger_joint"
-    has_pid="true" multiplier="-0.5" max_effort="10.0" offset="${gripper_base_width/2}" />
+    parent_joint="Gripper" mimic_joint="left_finger_joint" multiplier="-0.5" max_effort="10.0" offset="${gripper_base_width/2}" />
     <sensor name="camera">
         <parent link="camera_link" />

Commit message: Updated blocks, dynamics and documentation

File: urdf/lynxmotion_al5d.xacro (robot description, xacro)
@@ -200,11 +200,11 @@
         <axis xyz="0 0 -1" />
         <origin xyz="0 0.021 0" rpy="0 0 ${PI}" />
-        <limit effort="100" velocity="2" lower="${-PI}" upper="${PI}" />
-        <dynamics damping="50" friction="1" />
+        <limit effort="100" velocity="5" lower="${-PI}" upper="${PI}" />
+        <dynamics damping="20" friction="1" />
     </joint>
     <joint name="base_to_cylinder" type="fixed">
         <parent link="robot_base_cylinder" />
         <child link="robot_base_top_box" />
-        <dynamics damping="50" friction="0.7" />
+        <dynamics damping="20" friction="0.7" />
     </joint>
     <joint name="Joint2" type="revolute">
@@ -213,6 +213,6 @@
         <axis xyz="1 0 0"/>
         <origin xyz="0 0.015 0.071"  rpy="0 0 0" />
-        <limit effort="100" velocity="2" lower="0" upper="${PI}" />
-        <dynamics damping="50" friction="1" />
+        <limit effort="100" velocity="5" lower="0" upper="${PI}" />
+        <dynamics damping="20" friction="1" />
     </joint>
     <joint name="Joint3" type="revolute">
@@ -221,5 +221,5 @@
         <axis xyz="1 0 0" />
         <origin xyz="0 ${shoulder_to_elbow} 0" />
-        <limit effort="100" velocity="2" lower="${-PI/2}" upper="${PI/2}" />
+        <limit effort="100" velocity="5" lower="${-PI/2}" upper="${PI/2}" />
         <dynamics damping="20" friction="1" />
     </joint>
@@ -237,6 +237,6 @@
         <axis xyz="0 1 0" />
         <origin xyz="0 0.04 0" rpy="0 0 ${PI}" />
-        <limit effort="100" velocity="2" lower="${-PI}" upper="${PI}" />
-        <dynamics damping="50" friction="0.7" />
+        <limit effort="100" velocity="5" lower="${-PI}" upper="${PI}" />
+        <dynamics damping="20" friction="1" />
     </joint>
     <joint name="right_finger_joint" type="prismatic">
@@ -279,14 +279,8 @@
     <!-- Setting the mimic joints plugin -->
     <xacro:mimic_joint_plugin_gazebo name_prefix="finger_right"
-    parent_joint="Gripper" mimic_joint="right_finger_joint" multiplier="-0.5" max_effort="10.0" offset="${gripper_base_width/2}" />
+    parent_joint="Gripper" mimic_joint="right_finger_joint" multiplier="-0.5"
+        has_pid="true" max_effort="10.0" offset="${gripper_base_width/2}" />
     <xacro:mimic_joint_plugin_gazebo name_prefix="finger_left"
-    parent_joint="Gripper" mimic_joint="left_finger_joint" multiplier="-0.5" max_effort="10.0" offset="${gripper_base_width/2}" />
-    <sensor name="camera">
-        <parent link="camera_link" />
-        <origin xyz="0 0 0" rpy="${PI/2} 0 0" />
-        <camera>
-            <image width="640" height="480" hfov="1.41" near="0.01" far="0.04" />
-        </camera>
-    </sensor>
+    parent_joint="Gripper" has_pid="true"  mimic_joint="left_finger_joint" multiplier="-0.5" max_effort="10.0" offset="${gripper_base_width/2}" />
     <gazebo reference="camera_link">
         <sensor name="external_camera" type="camera">
@@ -309,5 +303,5 @@
                 <alwaysOn>true</alwaysOn>
                 <updateRate>1.0</updateRate>
-                <cameraName>al5d_external_vision</cameraName>
+                <cameraName>external_vision</cameraName>
                 <imageTopicName>image_raw</imageTopicName>
                 <cameraInfoTopicName>camera_info</cameraInfoTopicName>

Commit message: Making minor changes

File: urdf/lynxmotion_al5d.xacro (robot description, xacro)
@@ -246,4 +246,5 @@
         <limit effort="10" velocity="0.1" lower="0" upper="${gripper_base_width/2}" />
         <mimic joint="Gripper" multiplier="-0.5" offset="${gripper_base_width/2}" />
+        <dynamics friction="0.7" />
     </joint>
    <joint name="left_finger_joint" type="prismatic">
@@ -254,4 +255,5 @@
         <limit effort="10" velocity="0.1" lower="0" upper="${gripper_base_width/2}" />
         <mimic joint="right_finger_joint" />
+        <dynamics friction="0" />
     </joint>
     <!-- Joint that accept the distance between the two fingers as parameter -->
@@ -262,4 +264,5 @@
         <limit lower="0" upper="${gripper_base_width}" effort="10" velocity="0.1" />
         <axis xyz="-1 0 0" />
+        <dynamics friction="0.7" />
     </joint>
     <!-- Setting transmissions -->
@@ -288,5 +291,5 @@
             <camera name="camera_top">
                 <horizontal_fov>1.2</horizontal_fov>
-                <pose>0 0 0 3.1415 1.5708 1.5708</pose>
+                <pose>0 0 0 3.1415 1.5708 -1.5708</pose>
                 <image>
                     <width>640</width>

Commit message: Work in progress

File: urdf/lynxmotion_al5d.xacro (robot description, xacro)
@@ -188,5 +188,5 @@
         <child link="robot_support" />
         <origin rpy="0 0 ${PI}" />
-        <dynamics damping="50" friction="1" />
+        <dynamics damping="50" friction="0.8" />
     </joint>
     <joint name="camera_joint" type="fixed">
@@ -201,5 +201,5 @@
         <origin xyz="0 0.021 0" rpy="0 0 ${PI}" />
         <limit effort="100" velocity="5" lower="${-PI}" upper="${PI}" />
-        <dynamics damping="20" friction="1" />
+        <dynamics damping="20" friction="0.8" />
     </joint>
     <joint name="base_to_cylinder" type="fixed">
@@ -214,5 +214,5 @@
         <origin xyz="0 0.015 0.071"  rpy="0 0 0" />
         <limit effort="100" velocity="5" lower="0" upper="${PI}" />
-        <dynamics damping="20" friction="1" />
+        <dynamics damping="20" friction="0.8" />
     </joint>
     <joint name="Joint3" type="revolute">
@@ -222,5 +222,5 @@
         <origin xyz="0 ${shoulder_to_elbow} 0" />
         <limit effort="100" velocity="5" lower="${-PI/2}" upper="${PI/2}" />
-        <dynamics damping="20" friction="1" />
+        <dynamics damping="20" friction="0.8" />
     </joint>
     <joint name="Joint4" type="revolute">
@@ -230,5 +230,5 @@
         <origin xyz="0 ${tube_length + hs_645_depth - 0.003} 0.005" rpy="0 0 0"/>
         <limit effort="40" velocity="5" lower="${-PI/2}" upper="${PI/2}" />
-        <dynamics damping="20" friction="1" />
+        <dynamics damping="20" friction="0.8" />
     </joint>
    <joint name="Joint5" type="revolute">
@@ -238,5 +238,5 @@
         <origin xyz="0 0.04 0" rpy="0 0 ${PI}" />
         <limit effort="100" velocity="5" lower="${-PI}" upper="${PI}" />
-        <dynamics damping="20" friction="1" />
+        <dynamics damping="20" friction="0.8" />
     </joint>
     <joint name="right_finger_joint" type="prismatic">
@@ -246,5 +246,5 @@
         <limit effort="10" velocity="0.1" lower="0" upper="${gripper_base_width/2}" />
         <mimic joint="Gripper" multiplier="-0.5" offset="${gripper_base_width/2}" />
-        <dynamics friction="0.7" />
+        <dynamics friction="0.058" />
     </joint>
    <joint name="left_finger_joint" type="prismatic">
@@ -255,5 +255,5 @@
         <limit effort="10" velocity="0.1" lower="0" upper="${gripper_base_width/2}" />
         <mimic joint="right_finger_joint" />
-        <dynamics friction="0" />
+        <dynamics friction="0.058" />
     </joint>
     <!-- Joint that accept the distance between the two fingers as parameter -->
@@ -264,5 +264,5 @@
         <limit lower="0" upper="${gripper_base_width}" effort="10" velocity="0.1" />
         <axis xyz="-1 0 0" />
-        <dynamics friction="0.7" />
+        <!-- <dynamics friction="0.42" /> -->
     </joint>
     <!-- Setting transmissions -->

Commit message: Updated robot base

File: urdf/lynxmotion_al5d.xacro (robot description, xacro)
@@ -42,5 +42,5 @@
                 <mesh filename="package://lynxmotion_al5d_description/meshes/robot_parts/top_box.dae" />
             </geometry>
-            <origin xyz="0.007 -0.024 0" rpy="0 0 0" />
+            <origin xyz="-0.01 0.01 0" rpy="0 0 ${PI}" />
         </visual>
         <collision>
@@ -212,5 +212,5 @@
         <child link="shoulder" />
         <axis xyz="1 0 0"/>
-        <origin xyz="0 0.015 0.071"  rpy="0 0 0" />
+        <origin xyz="0 0.005 0.071"  rpy="0 0 0" />
         <limit effort="100" velocity="5" lower="0" upper="${PI}" />
         <dynamics damping="20" friction="0.8" />

Commit message: Update to documentation

File: urdf/lynxmotion_al5d.xacro (robot description, xacro)
@@ -10,5 +10,5 @@
                 <mesh filename="package://lynxmotion_al5d_description/meshes/robot_parts/support.dae" />
             </geometry>3
-            <origin rpy="0 0 0" xyz="0 0 0" />
+            <origin rpy="0 0 0" xyz="0 -0.01 0" />
         </visual>
         <collision>
@@ -16,5 +16,5 @@
                 <mesh filename="package://lynxmotion_al5d_description/meshes/robot_parts/support.dae" />
             </geometry>
-            <origin rpy="0 0 0" xyz="0 0 0" />
+            <origin rpy="0 0 0" xyz="0 -0.01 0" />
         </collision>
         <xacro:inertial_matrix mass="${board_mass}" ixx="3.6565e-7" ixy="-3.72e-9" ixz="1e-6" iyy="9.404e-8" iyz="4.375e-8" izz="4.1776e-7" xyz="0.000585 0.0602746 0.0170628" />
@@ -26,5 +26,5 @@
                 <mesh filename="package://lynxmotion_al5d_description/meshes/robot_parts/rotation_cylinder.dae" />
             </geometry>
-            <origin rpy="0 0 0" xyz="0 -0.021165 0" />
+            <origin rpy="0 0 0" xyz="0 -0.011165 0" />
         </visual>
         <collision>
@@ -32,5 +32,5 @@
                 <mesh filename="package://lynxmotion_al5d_description/meshes/robot_parts/rotation_cylinder.dae" />
             </geometry>
-            <origin rpy="0 0 0" xyz="0 -0.021165 0" />
+            <origin rpy="0 0 0" xyz="0 -0.011165 0" />
         </collision>
         <xacro:inertial_matrix_bis mass="${base_mass}" />
@@ -42,5 +42,5 @@
                 <mesh filename="package://lynxmotion_al5d_description/meshes/robot_parts/top_box.dae" />
             </geometry>
-            <origin xyz="-0.01 0.01 0" rpy="0 0 ${PI}" />
+            <origin xyz="-0.01 0.03 0" rpy="0 0 ${PI}" />
         </visual>
         <collision>
@@ -48,5 +48,5 @@
                 <mesh filename="package://lynxmotion_al5d_description/meshes/robot_parts/top_box.dae" />
             </geometry>
-            <origin xyz="0.007 -0.024 0" rpy="0 0 0" />
+            <origin xyz="-0.01 0.03 0" rpy="0 0 ${PI}" />
         </collision>
         <xacro:inertial_matrix_bis mass="${top_box_mass}" />
@@ -212,5 +212,5 @@
         <child link="shoulder" />
         <axis xyz="1 0 0"/>
-        <origin xyz="0 0.005 0.071"  rpy="0 0 0" />
+        <origin xyz="0 0.020 0.071"  rpy="0 0 0" />
         <limit effort="100" velocity="5" lower="0" upper="${PI}" />
         <dynamics damping="20" friction="0.8" />

Commit message: Updated documentation

File: urdf/lynxmotion_al5d.xacro (robot description, xacro)
@@ -9,5 +9,5 @@
             <geometry>
                 <mesh filename="package://lynxmotion_al5d_description/meshes/robot_parts/support.dae" />
-            </geometry>3
+            </geometry>
             <origin rpy="0 0 0" xyz="0 -0.01 0" />
         </visual>

Commit message: Updated elbow angle range

File: urdf/lynxmotion_al5d.xacro (robot description, xacro)
@@ -221,5 +221,5 @@
         <axis xyz="1 0 0" />
         <origin xyz="0 ${shoulder_to_elbow} 0" />
-        <limit effort="100" velocity="5" lower="${-PI/2}" upper="${PI/2}" />
+        <limit effort="100" velocity="5" lower="${-PI}" upper="0" />
         <dynamics damping="20" friction="0.8" />
     </joint>

Commit message: Updated friction parameters

File: urdf/lynxmotion_al5d.xacro (robot description, xacro)
@@ -246,5 +246,5 @@
         <limit effort="10" velocity="0.1" lower="0" upper="${gripper_base_width/2}" />
         <mimic joint="Gripper" multiplier="-0.5" offset="${gripper_base_width/2}" />
-        <dynamics friction="0.058" />
+        <dynamics friction="0.16" />
     </joint>
    <joint name="left_finger_joint" type="prismatic">
@@ -255,5 +255,5 @@
         <limit effort="10" velocity="0.1" lower="0" upper="${gripper_base_width/2}" />
         <mimic joint="right_finger_joint" />
-        <dynamics friction="0.058" />
+        <dynamics friction="0.16" />
     </joint>
     <!-- Joint that accept the distance between the two fingers as parameter -->

Commit message: changed Joint5 axis

File: urdf/lynxmotion_al5d.xacro (robot description, xacro)
@@ -235,5 +235,5 @@
         <parent link="wrist" />
         <child link="gripper" />
-        <axis xyz="0 1 0" />
+        <axis xyz="0 -1 0" />
         <origin xyz="0 0.04 0" rpy="0 0 ${PI}" />
         <limit effort="100" velocity="5" lower="${-PI}" upper="${PI}" />
