Commit message: Changing dynamics parameter

File: urdf/lynxmotion_al5d.xacro (robot description, xacro)
@@ -188,5 +188,5 @@
         <child link="robot_support" />
         <origin rpy="0 0 ${PI}" />
-        <dynamics damping="50" friction="0.8" />
+        <dynamics damping="1.0" friction="0.16" />
     </joint>
     <joint name="camera_joint" type="fixed">
@@ -201,10 +201,10 @@
         <origin xyz="0 0.021 0" rpy="0 0 ${PI}" />
         <limit effort="100" velocity="5" lower="${-PI}" upper="${PI}" />
-        <dynamics damping="20" friction="0.8" />
+        <dynamics damping="1.0" friction="0.16" />
     </joint>
     <joint name="base_to_cylinder" type="fixed">
         <parent link="robot_base_cylinder" />
         <child link="robot_base_top_box" />
-        <dynamics damping="20" friction="0.7" />
+        <dynamics damping="1.0" friction="0.16" />
     </joint>
     <joint name="Joint2" type="revolute">
@@ -214,5 +214,5 @@
         <origin xyz="0 0.020 0.071"  rpy="0 0 0" />
         <limit effort="100" velocity="5" lower="0" upper="${PI}" />
-        <dynamics damping="20" friction="0.8" />
+        <dynamics damping="1.0" friction="0.16" />
     </joint>
     <joint name="Joint3" type="revolute">
@@ -222,5 +222,5 @@
         <origin xyz="0 ${shoulder_to_elbow} 0" />
         <limit effort="100" velocity="5" lower="${-PI}" upper="0" />
-        <dynamics damping="20" friction="0.8" />
+        <dynamics damping="1.0" friction="0.16" />
     </joint>
     <joint name="Joint4" type="revolute">
@@ -230,5 +230,5 @@
         <origin xyz="0 ${tube_length + hs_645_depth - 0.003} 0.005" rpy="0 0 0"/>
         <limit effort="40" velocity="5" lower="${-PI/2}" upper="${PI/2}" />
-        <dynamics damping="20" friction="0.8" />
+        <dynamics damping="1.0" friction="0.16" />
     </joint>
    <joint name="Joint5" type="revolute">
@@ -238,5 +238,5 @@
         <origin xyz="0 0.04 0" rpy="0 0 ${PI}" />
         <limit effort="100" velocity="5" lower="${-PI}" upper="${PI}" />
-        <dynamics damping="20" friction="0.8" />
+        <dynamics damping="1.0" friction="0.16" />
     </joint>
     <joint name="right_finger_joint" type="prismatic">

Commit message: Fixed message

File: urdf/lynxmotion_al5d.xacro (robot description, xacro)
@@ -82,5 +82,5 @@
             <origin rpy="${-PI-0.895} ${PI} 0" xyz="-0.005 ${tube_length - 2*hs_755eb_depth/5} ${-shoulder_to_elbow - 0.02} " />
         </collision>
-        <xacro:inertial_matrix_bis mass="${hs_755eb_mass+ hs_645_mass}" />
+        <xacro:inertial_matrix_bis mass="${hs_755eb_mass + hs_645_mass}" />
     </link>
     <gazebo reference="arm" />
@@ -98,5 +98,5 @@
             <origin rpy="${PI} 0 0" xyz="0.005 -0.165 0.067" />
         </collision>
-        <xacro:inertial_matrix_bis mass="${0.031}" />
+        <xacro:inertial_matrix_bis mass="0.031" />
     </link>
     <gazebo reference="wrist" />
@@ -188,5 +188,5 @@
         <child link="robot_support" />
         <origin rpy="0 0 ${PI}" />
-        <dynamics damping="1.0" friction="0.16" />
+        <dynamics damping="1.0" friction="0.8" />
     </joint>
     <joint name="camera_joint" type="fixed">
@@ -200,11 +200,11 @@
         <axis xyz="0 0 -1" />
         <origin xyz="0 0.021 0" rpy="0 0 ${PI}" />
-        <limit effort="100" velocity="5" lower="${-PI}" upper="${PI}" />
-        <dynamics damping="1.0" friction="0.16" />
+        <limit effort="100" velocity="3" lower="${-PI}" upper="${PI}" />
+        <dynamics damping="1.0" friction="0.8" />
     </joint>
     <joint name="base_to_cylinder" type="fixed">
         <parent link="robot_base_cylinder" />
         <child link="robot_base_top_box" />
-        <dynamics damping="1.0" friction="0.16" />
+        <dynamics damping="1.0" friction="0.8" />
     </joint>
     <joint name="Joint2" type="revolute">
@@ -213,6 +213,6 @@
         <axis xyz="1 0 0"/>
         <origin xyz="0 0.020 0.071"  rpy="0 0 0" />
-        <limit effort="100" velocity="5" lower="0" upper="${PI}" />
-        <dynamics damping="1.0" friction="0.16" />
+        <limit effort="100" velocity="3" lower="0" upper="${PI}" />
+        <dynamics damping="1.0" friction="0.8" />
     </joint>
     <joint name="Joint3" type="revolute">
@@ -221,6 +221,6 @@
         <axis xyz="1 0 0" />
         <origin xyz="0 ${shoulder_to_elbow} 0" />
-        <limit effort="100" velocity="5" lower="${-PI}" upper="0" />
-        <dynamics damping="1.0" friction="0.16" />
+        <limit effort="100" velocity="3" lower="${-PI}" upper="0" />
+        <dynamics damping="1.0" friction="0.8" />
     </joint>
     <joint name="Joint4" type="revolute">
@@ -229,14 +229,14 @@
         <axis xyz="1 0 0" />
         <origin xyz="0 ${tube_length + hs_645_depth - 0.003} 0.005" rpy="0 0 0"/>
-        <limit effort="40" velocity="5" lower="${-PI/2}" upper="${PI/2}" />
-        <dynamics damping="1.0" friction="0.16" />
+        <limit effort="40" velocity="3" lower="${-PI/2}" upper="${PI/2}" />
+        <dynamics damping="1.0" friction="0.8" />
     </joint>
    <joint name="Joint5" type="revolute">
         <parent link="wrist" />
         <child link="gripper" />
-        <axis xyz="0 -1 0" />
+        <axis xyz="0 1 0" />
         <origin xyz="0 0.04 0" rpy="0 0 ${PI}" />
-        <limit effort="100" velocity="5" lower="${-PI}" upper="${PI}" />
-        <dynamics damping="1.0" friction="0.16" />
+        <limit effort="100" velocity="3" lower="${-PI}" upper="${PI}" />
+        <dynamics damping="1.0" friction="0.8" />
     </joint>
     <joint name="right_finger_joint" type="prismatic">
@@ -246,14 +246,15 @@
         <limit effort="10" velocity="0.1" lower="0" upper="${gripper_base_width/2}" />
         <mimic joint="Gripper" multiplier="-0.5" offset="${gripper_base_width/2}" />
-        <dynamics friction="0.16" />
+        <dynamics damping="1.0" friction="0.16" />
     </joint>
    <joint name="left_finger_joint" type="prismatic">
         <parent link="gripper" />
         <child link="left_finger" />
-        <origin xyz="0 -0.015 0" />
+        <origin xyz="-0.0025 -0.015 0" />
         <axis xyz="-1 0 0" />
         <limit effort="10" velocity="0.1" lower="0" upper="${gripper_base_width/2}" />
-        <mimic joint="right_finger_joint" />
-        <dynamics friction="0.16" />
+        <!-- Added an offset to fix issues in Rviz -->
+        <mimic joint="right_finger_joint" offset="-0.0025" />
+        <dynamics damping="1.0" friction="0.16" />
     </joint>
     <!-- Joint that accept the distance between the two fingers as parameter -->
@@ -264,4 +265,5 @@
         <limit lower="0" upper="${gripper_base_width}" effort="10" velocity="0.1" />
         <axis xyz="-1 0 0" />
+        <dynamics damping="1.0" />
         <!-- <dynamics friction="0.42" /> -->
     </joint>

Commit message: Changed rotation axis

File: urdf/lynxmotion_al5d.xacro (robot description, xacro)
@@ -235,5 +235,5 @@
         <parent link="wrist" />
         <child link="gripper" />
-        <axis xyz="0 1 0" />
+        <axis xyz="0 -1 0" />
         <origin xyz="0 0.04 0" rpy="0 0 ${PI}" />
         <limit effort="100" velocity="3" lower="${-PI}" upper="${PI}" />

Commit message: Updated base movement

File: urdf/lynxmotion_al5d.xacro (robot description, xacro)
@@ -26,5 +26,5 @@
                 <mesh filename="package://lynxmotion_al5d_description/meshes/robot_parts/rotation_cylinder.dae" />
             </geometry>
-            <origin rpy="0 0 0" xyz="0 -0.011165 0" />
+            <origin rpy="0 0 0" xyz="0 -0.021 0" />
         </visual>
         <collision>
@@ -32,5 +32,5 @@
                 <mesh filename="package://lynxmotion_al5d_description/meshes/robot_parts/rotation_cylinder.dae" />
             </geometry>
-            <origin rpy="0 0 0" xyz="0 -0.011165 0" />
+            <origin rpy="0 0 0" xyz="0 -0.021 0" />
         </collision>
         <xacro:inertial_matrix_bis mass="${base_mass}" />
@@ -199,5 +199,5 @@
         <child link="robot_base_cylinder" />
         <axis xyz="0 0 -1" />
-        <origin xyz="0 0.021 0" rpy="0 0 ${PI}" />
+        <origin xyz="0 0.01 0" rpy="0 0 ${PI}" />
         <limit effort="100" velocity="3" lower="${-PI}" upper="${PI}" />
         <dynamics damping="1.0" friction="0.8" />

Commit message: Changed arm to elbow

File: urdf/lynxmotion_al5d.xacro (robot description, xacro)
@@ -69,8 +69,8 @@
     </link>
     <gazebo reference="shoulder" />
-    <link name="arm">
-        <visual>
-            <geometry>
-                <mesh filename="package://lynxmotion_al5d_description/meshes/robot_parts/arm.dae" />
+    <link name="elbow">
+        <visual>
+            <geometry>
+                <mesh filename="package://lynxmotion_al5d_description/meshes/robot_parts/elbow.dae" />
             </geometry>
             <origin rpy="${-PI-0.895} ${PI} 0" xyz="-0.005 ${tube_length - 2*hs_755eb_depth/5} ${-shoulder_to_elbow - 0.02} " />
@@ -78,11 +78,11 @@
         <collision>
             <geometry>
-                <mesh filename="package://lynxmotion_al5d_description/meshes/robot_parts/arm.dae" />
+                <mesh filename="package://lynxmotion_al5d_description/meshes/robot_parts/elbow.dae" />
             </geometry>
             <origin rpy="${-PI-0.895} ${PI} 0" xyz="-0.005 ${tube_length - 2*hs_755eb_depth/5} ${-shoulder_to_elbow - 0.02} " />
         </collision>
-        <xacro:inertial_matrix_bis mass="${hs_755eb_mass + hs_645_mass}" />
-    </link>
-    <gazebo reference="arm" />
+        <xacro:inertial_matrix_bis mass="0.01" />
+    </link>
+    <gazebo reference="elbow" />
     <link name="wrist">
         <visual>
@@ -218,5 +218,5 @@
     <joint name="Joint3" type="revolute">
         <parent link="shoulder" />
-        <child link="arm" />
+        <child link="elbow" />
         <axis xyz="1 0 0" />
         <origin xyz="0 ${shoulder_to_elbow} 0" />
@@ -225,5 +225,5 @@
     </joint>
     <joint name="Joint4" type="revolute">
-        <parent link="arm" />
+        <parent link="elbow" />
         <child link="wrist" />
         <axis xyz="1 0 0" />

Commit message: Updated PID values

File: urdf/lynxmotion_al5d.xacro (robot description, xacro)
@@ -82,5 +82,5 @@
             <origin rpy="${-PI-0.895} ${PI} 0" xyz="-0.005 ${tube_length - 2*hs_755eb_depth/5} ${-shoulder_to_elbow - 0.02} " />
         </collision>
-        <xacro:inertial_matrix_bis mass="0.01" />
+        <xacro:inertial_matrix_bis mass="${hs_755eb_mass + hs_645_mass}" />
     </link>
     <gazebo reference="elbow" />
@@ -230,5 +230,5 @@
         <origin xyz="0 ${tube_length + hs_645_depth - 0.003} 0.005" rpy="0 0 0"/>
         <limit effort="40" velocity="3" lower="${-PI/2}" upper="${PI/2}" />
-        <dynamics damping="1.0" friction="0.8" />
+        <dynamics damping="5.0" friction="0.08" />
     </joint>
    <joint name="Joint5" type="revolute">
@@ -244,7 +244,7 @@
         <child link="right_finger" />
         <origin xyz="0 -0.015 0" />
-        <limit effort="10" velocity="0.1" lower="0" upper="${gripper_base_width/2}" />
+        <limit effort="100" velocity="0.1" lower="0" upper="${gripper_base_width/2}" />
         <mimic joint="Gripper" multiplier="-0.5" offset="${gripper_base_width/2}" />
-        <dynamics damping="1.0" friction="0.16" />
+        <dynamics damping="1.0" friction="0.084" />
     </joint>
    <joint name="left_finger_joint" type="prismatic">
@@ -253,8 +253,8 @@
         <origin xyz="-0.0025 -0.015 0" />
         <axis xyz="-1 0 0" />
-        <limit effort="10" velocity="0.1" lower="0" upper="${gripper_base_width/2}" />
+        <limit effort="100" velocity="0.1" lower="0" upper="${gripper_base_width/2}" />
         <!-- Added an offset to fix issues in Rviz -->
         <mimic joint="right_finger_joint" offset="-0.0025" />
-        <dynamics damping="1.0" friction="0.16" />
+        <dynamics damping="1.0" friction="0.084" />
     </joint>
     <!-- Joint that accept the distance between the two fingers as parameter -->

Commit message: Fixing PID bad values

File: urdf/lynxmotion_al5d.xacro (robot description, xacro)
@@ -42,5 +42,5 @@
                 <mesh filename="package://lynxmotion_al5d_description/meshes/robot_parts/top_box.dae" />
             </geometry>
-            <origin xyz="-0.01 0.03 0" rpy="0 0 ${PI}" />
+            <origin xyz="-0.01 0.01 0" rpy="0 0 ${PI}" />
         </visual>
         <collision>
@@ -48,5 +48,5 @@
                 <mesh filename="package://lynxmotion_al5d_description/meshes/robot_parts/top_box.dae" />
             </geometry>
-            <origin xyz="-0.01 0.03 0" rpy="0 0 ${PI}" />
+            <origin xyz="-0.01 0.01 0" rpy="0 0 ${PI}" />
         </collision>
         <xacro:inertial_matrix_bis mass="${top_box_mass}" />
@@ -212,5 +212,5 @@
         <child link="shoulder" />
         <axis xyz="1 0 0"/>
-        <origin xyz="0 0.020 0.071"  rpy="0 0 0" />
+        <origin xyz="0 0.010 0.071"  rpy="0 0 0" />
         <limit effort="100" velocity="3" lower="0" upper="${PI}" />
         <dynamics damping="1.0" friction="0.8" />

Commit message: Fingers axis updated

File: urdf/lynxmotion_al5d.xacro (robot description, xacro)
@@ -122,5 +122,5 @@
                 <mesh filename="package://lynxmotion_al5d_description/meshes/robot_parts/finger_left.dae" />
             </geometry>
-            <origin rpy="${PI/2} 0 ${-PI/2}" xyz="0.0028 -0.009 0" />
+            <origin rpy="${PI/2} 0 ${-PI/2}" xyz="0.0015 -0.009 0" />
         </visual>
         <collision>
@@ -128,5 +128,5 @@
                 <mesh filename="package://lynxmotion_al5d_description/meshes/robot_parts/finger_left.dae" />
             </geometry>
-            <origin rpy="${PI/2} 0 ${-PI/2}" xyz="0.0028 -0.009 0" />
+            <origin rpy="${PI/2} 0 ${-PI/2}" xyz="0.0015 -0.009 0" />
         </collision>
         <xacro:inertial_matrix_bis mass="${finger_mass}" />
@@ -138,5 +138,5 @@
                 <mesh filename="package://lynxmotion_al5d_description/meshes/robot_parts/finger_right.dae" />
             </geometry>
-            <origin rpy="${PI/2} 0 ${-PI/2}" xyz="-0.0028 -0.009 0" />
+            <origin rpy="${PI/2} 0 ${-PI/2}" xyz="0.0025 -0.009 0" />
         </visual>
         <collision>
@@ -144,5 +144,5 @@
                 <mesh filename="package://lynxmotion_al5d_description/meshes/robot_parts/finger_right.dae" />
             </geometry>
-            <origin rpy="${PI/2} 0 ${-PI/2}" xyz="-0.0028 -0.009 0" />
+            <origin rpy="${PI/2} 0 ${-PI/2}" xyz="0.0025 -0.009 0" />
         </collision>
         <xacro:inertial_matrix_bis mass="${finger_mass}" />
@@ -243,5 +243,5 @@
         <parent link="gripper" />
         <child link="right_finger" />
-        <origin xyz="0 -0.015 0" />
+        <origin xyz="-0.006 -0.015 0" />
         <limit effort="100" velocity="0.1" lower="0" upper="${gripper_base_width/2}" />
         <mimic joint="Gripper" multiplier="-0.5" offset="${gripper_base_width/2}" />
@@ -251,5 +251,5 @@
         <parent link="gripper" />
         <child link="left_finger" />
-        <origin xyz="-0.0025 -0.015 0" />
+        <origin xyz="-0.0017 -0.015 0" />
         <axis xyz="-1 0 0" />
         <limit effort="100" velocity="0.1" lower="0" upper="${gripper_base_width/2}" />

Commit message: Fingers distance updated

File: urdf/lynxmotion_al5d.xacro (robot description, xacro)
@@ -122,5 +122,5 @@
                 <mesh filename="package://lynxmotion_al5d_description/meshes/robot_parts/finger_left.dae" />
             </geometry>
-            <origin rpy="${PI/2} 0 ${-PI/2}" xyz="0.0015 -0.009 0" />
+            <origin rpy="${PI/2} 0 ${-PI/2}" xyz="0.0045 -0.009 0" />
         </visual>
         <collision>
@@ -128,5 +128,5 @@
                 <mesh filename="package://lynxmotion_al5d_description/meshes/robot_parts/finger_left.dae" />
             </geometry>
-            <origin rpy="${PI/2} 0 ${-PI/2}" xyz="0.0015 -0.009 0" />
+            <origin rpy="${PI/2} 0 ${-PI/2}" xyz="0.0045 -0.009 0" />
         </collision>
         <xacro:inertial_matrix_bis mass="${finger_mass}" />
@@ -138,5 +138,5 @@
                 <mesh filename="package://lynxmotion_al5d_description/meshes/robot_parts/finger_right.dae" />
             </geometry>
-            <origin rpy="${PI/2} 0 ${-PI/2}" xyz="0.0025 -0.009 0" />
+            <origin rpy="${PI/2} 0 ${-PI/2}" xyz="-0.0005 -0.009 0" />
         </visual>
         <collision>
@@ -144,5 +144,5 @@
                 <mesh filename="package://lynxmotion_al5d_description/meshes/robot_parts/finger_right.dae" />
             </geometry>
-            <origin rpy="${PI/2} 0 ${-PI/2}" xyz="0.0025 -0.009 0" />
+            <origin rpy="${PI/2} 0 ${-PI/2}" xyz="-0.0005 -0.009 0" />
         </collision>
         <xacro:inertial_matrix_bis mass="${finger_mass}" />
@@ -265,5 +265,5 @@
         <limit lower="0" upper="${gripper_base_width}" effort="10" velocity="0.1" />
         <axis xyz="-1 0 0" />
-        <dynamics damping="1.0" />
+        <dynamics damping="5.0" />
         <!-- <dynamics friction="0.42" /> -->
     </joint>

Commit message: Checking PID

File: urdf/lynxmotion_al5d.xacro (robot description, xacro)
@@ -246,5 +246,5 @@
         <limit effort="100" velocity="0.1" lower="0" upper="${gripper_base_width/2}" />
         <mimic joint="Gripper" multiplier="-0.5" offset="${gripper_base_width/2}" />
-        <dynamics damping="1.0" friction="0.084" />
+        <dynamics friction="0.084" />
     </joint>
    <joint name="left_finger_joint" type="prismatic">
@@ -256,5 +256,5 @@
         <!-- Added an offset to fix issues in Rviz -->
         <mimic joint="right_finger_joint" offset="-0.0025" />
-        <dynamics damping="1.0" friction="0.084" />
+        <dynamics friction="0.084" />
     </joint>
     <!-- Joint that accept the distance between the two fingers as parameter -->

Commit message: Trying new PID values

File: urdf/lynxmotion_al5d.xacro (robot description, xacro)
@@ -130,5 +130,5 @@
             <origin rpy="${PI/2} 0 ${-PI/2}" xyz="0.0045 -0.009 0" />
         </collision>
-        <xacro:inertial_matrix_bis mass="${finger_mass}" />
+        <xacro:inertial_matrix_bis mass="0.002" />
     </link>
     <gazebo reference="left_finger" />
@@ -138,5 +138,5 @@
                 <mesh filename="package://lynxmotion_al5d_description/meshes/robot_parts/finger_right.dae" />
             </geometry>
-            <origin rpy="${PI/2} 0 ${-PI/2}" xyz="-0.0005 -0.009 0" />
+            <origin rpy="${PI/2} 0 ${-PI/2}" xyz="0.0045 -0.009 0" />
         </visual>
         <collision>
@@ -144,7 +144,7 @@
                 <mesh filename="package://lynxmotion_al5d_description/meshes/robot_parts/finger_right.dae" />
             </geometry>
-            <origin rpy="${PI/2} 0 ${-PI/2}" xyz="-0.0005 -0.009 0" />
-        </collision>
-        <xacro:inertial_matrix_bis mass="${finger_mass}" />
+            <origin rpy="${PI/2} 0 ${-PI/2}" xyz="0.0045 -0.009 0" />
+        </collision>
+        <xacro:inertial_matrix_bis mass="0.002" />
     </link>
     <gazebo reference="right_finger" />
@@ -246,5 +246,5 @@
         <limit effort="100" velocity="0.1" lower="0" upper="${gripper_base_width/2}" />
         <mimic joint="Gripper" multiplier="-0.5" offset="${gripper_base_width/2}" />
-        <dynamics friction="0.084" />
+        <dynamics damping="1.0" friction="0.16" />
     </joint>
    <joint name="left_finger_joint" type="prismatic">
@@ -256,5 +256,5 @@
         <!-- Added an offset to fix issues in Rviz -->
         <mimic joint="right_finger_joint" offset="-0.0025" />
-        <dynamics friction="0.084" />
+        <dynamics damping="1.0" friction="0.16" />
     </joint>
     <!-- Joint that accept the distance between the two fingers as parameter -->
