Commit message: Updated robot model

File: urdf/lynxmotion_al5d.xacro (robot description, xacro)
@@ -1,4 +1,4 @@
 <?xml version="1.0" ?>
-<robot name="lynxmotion_al5d" xmlns:xacro="http://www.ros.org/wiki/xacro" xmlns:sensor="http://playerstage.sourceforge.net/gazebo/xmlschema/#sensor" xmlns:controller="http://playerstage.sourceforge.net/gazebo/xmlschema/#controller" xmlns:interface="http://playerstage.sourceforge.net/gazebo/xmlschema/#interface">
+<robot name="lynxmotion_al5d" xmlns:xacro="http://www.ros.org/wiki/xacro">
     <xacro:include filename="$(find lynxmotion_al5d_description)/urdf/lynxmotion_al5d_properties.urdf.xacro" />
     <!-- Base link comprising the board behind the robot and the cylinder at its bottom -->
@@ -10,5 +10,5 @@
                 <mesh filename="package://lynxmotion_al5d_description/meshes/robot_parts/support.dae" />
             </geometry>
-            <origin rpy="0 0 0" xyz="0 -0.01 0" />
+            <origin rpy="0 0 0" xyz="0 0 0" />
         </visual>
         <collision>
@@ -16,7 +16,7 @@
                 <mesh filename="package://lynxmotion_al5d_description/meshes/robot_parts/support.dae" />
             </geometry>
-            <origin rpy="0 0 0" xyz="0 -0.01 0" />
-        </collision>
-        <xacro:inertial_matrix mass="${board_mass}" ixx="3.6565e-7" ixy="-3.72e-9" ixz="1e-6" iyy="9.404e-8" iyz="4.375e-8" izz="4.1776e-7" xyz="0.000585 0.0602746 0.0170628" />
+            <origin rpy="0 0 0" xyz="0 0 0" />
+        </collision>
+        <xacro:inertial_matrix mass="${base_mass + board_mass}" ixx="3.6565e-7" ixy="-3.72e-9" ixz="1e-6" iyy="9.404e-8" iyz="4.375e-8" izz="4.1776e-7" xyz="0.000585 0.0602746 0.0170628" />
     </link>
     <gazebo reference="robot_support" />
@@ -34,5 +34,5 @@
             <origin rpy="0 0 0" xyz="0 -0.021 0" />
         </collision>
-        <xacro:inertial_matrix_bis mass="${base_mass}" />
+        <xacro:inertial_matrix_bis mass="0.01" />
     </link>
     <gazebo reference="robot_base_cylinder" />
@@ -42,5 +42,5 @@
                 <mesh filename="package://lynxmotion_al5d_description/meshes/robot_parts/top_box.dae" />
             </geometry>
-            <origin xyz="-0.01 0.01 0" rpy="0 0 ${PI}" />
+            <origin xyz="-0.01 0.02 0" rpy="0 0 ${PI}" />
         </visual>
         <collision>
@@ -48,5 +48,5 @@
                 <mesh filename="package://lynxmotion_al5d_description/meshes/robot_parts/top_box.dae" />
             </geometry>
-            <origin xyz="-0.01 0.01 0" rpy="0 0 ${PI}" />
+            <origin xyz="-0.01 0.02 0" rpy="0 0 ${PI}" />
         </collision>
         <xacro:inertial_matrix_bis mass="${top_box_mass}" />
@@ -74,5 +74,5 @@
                 <mesh filename="package://lynxmotion_al5d_description/meshes/robot_parts/elbow.dae" />
             </geometry>
-            <origin rpy="${-PI-0.895} ${PI} 0" xyz="-0.005 ${tube_length - 2*hs_755eb_depth/5} ${-shoulder_to_elbow - 0.02} " />
+            <origin rpy="${-PI-0.895} ${PI} 0" xyz="-0.005 ${tube_length - 2*hs_755eb_depth/5} ${-shoulder_to_elbow - 0.026}" />
         </visual>
         <collision>
@@ -80,5 +80,5 @@
                 <mesh filename="package://lynxmotion_al5d_description/meshes/robot_parts/elbow.dae" />
             </geometry>
-            <origin rpy="${-PI-0.895} ${PI} 0" xyz="-0.005 ${tube_length - 2*hs_755eb_depth/5} ${-shoulder_to_elbow - 0.02} " />
+            <origin rpy="${-PI-0.895} ${PI} 0" xyz="-0.005 ${tube_length - 2*hs_755eb_depth/5} ${-shoulder_to_elbow - 0.026} " />
         </collision>
         <xacro:inertial_matrix_bis mass="${hs_755eb_mass + hs_645_mass}" />
@@ -90,5 +90,5 @@
                 <mesh filename="package://lynxmotion_al5d_description/meshes/robot_parts/wrist.dae" />
             </geometry>
-            <origin rpy="${PI} 0 0" xyz="0.005 -0.165 0.067" />
+            <origin rpy="${PI} 0 0" xyz="0 -0.165 0.067" />
         </visual>
         <collision>
@@ -96,5 +96,5 @@
                 <mesh filename="package://lynxmotion_al5d_description/meshes/robot_parts/wrist.dae" />
             </geometry>
-            <origin rpy="${PI} 0 0" xyz="0.005 -0.165 0.067" />
+            <origin rpy="${PI} 0 0" xyz="0 -0.165 0.067" />
         </collision>
         <xacro:inertial_matrix_bis mass="0.031" />
@@ -106,5 +106,5 @@
                 <mesh filename="package://lynxmotion_al5d_description/meshes/robot_parts/gripper.dae" />
             </geometry>
-            <origin rpy="${PI/2} 0 ${-PI/2}" xyz="0 -0.021 -0.005" />
+            <origin rpy="${PI/2} 0 ${-PI/2}" xyz="0 -0.02 0.0" />
         </visual>
         <collision>
@@ -112,5 +112,5 @@
                 <mesh filename="package://lynxmotion_al5d_description/meshes/robot_parts/gripper.dae" />
             </geometry>
-            <origin rpy="${PI/2} 0 ${-PI/2}" xyz="0 -0.021 -0.005" />
+            <origin rpy="${PI/2} 0 ${-PI/2}" xyz="0 -0.02 0" /> <!---0.021 -0.005" /> -->
         </collision>
         <xacro:inertial_matrix_bis mass="0.042" />
@@ -122,5 +122,5 @@
                 <mesh filename="package://lynxmotion_al5d_description/meshes/robot_parts/finger_left.dae" />
             </geometry>
-            <origin rpy="${PI/2} 0 ${-PI/2}" xyz="0.0045 -0.009 0" />
+            <origin rpy="${PI/2} 0 ${-PI/2}" xyz="0.001 -0.005 0" />
         </visual>
         <collision>
@@ -128,5 +128,5 @@
                 <mesh filename="package://lynxmotion_al5d_description/meshes/robot_parts/finger_left.dae" />
             </geometry>
-            <origin rpy="${PI/2} 0 ${-PI/2}" xyz="0.0045 -0.009 0" />
+            <origin rpy="${PI/2} 0 ${-PI/2}" xyz="0.001 -0.005 0" />
         </collision>
         <xacro:inertial_matrix_bis mass="0.002" />
@@ -138,5 +138,5 @@
                 <mesh filename="package://lynxmotion_al5d_description/meshes/robot_parts/finger_right.dae" />
             </geometry>
-            <origin rpy="${PI/2} 0 ${-PI/2}" xyz="0.0045 -0.009 0" />
+            <origin rpy="${PI/2} 0 ${-PI/2}" xyz="-0.003 -0.005 0" />
         </visual>
         <collision>
@@ -144,5 +144,5 @@
                 <mesh filename="package://lynxmotion_al5d_description/meshes/robot_parts/finger_right.dae" />
             </geometry>
-            <origin rpy="${PI/2} 0 ${-PI/2}" xyz="0.0045 -0.009 0" />
+            <origin rpy="${PI/2} 0 ${-PI/2}" xyz="-0.003 -0.005 0" />
         </collision>
         <xacro:inertial_matrix_bis mass="0.002" />
@@ -199,7 +199,7 @@
         <child link="robot_base_cylinder" />
         <axis xyz="0 0 -1" />
-        <origin xyz="0 0.01 0" rpy="0 0 ${PI}" />
+        <origin xyz="0 0.02 0" rpy="0 0 ${PI}" />
         <limit effort="100" velocity="3" lower="${-PI}" upper="${PI}" />
-        <dynamics damping="1.0" friction="0.8" />
+        <dynamics damping="50.0" friction="1" />
     </joint>
     <joint name="base_to_cylinder" type="fixed">
@@ -212,5 +212,5 @@
         <child link="shoulder" />
         <axis xyz="1 0 0"/>
-        <origin xyz="0 0.010 0.071"  rpy="0 0 0" />
+        <origin xyz="0 0.02 0.07" />
         <limit effort="100" velocity="3" lower="0" upper="${PI}" />
         <dynamics damping="1.0" friction="0.8" />
@@ -228,5 +228,5 @@
         <child link="wrist" />
         <axis xyz="1 0 0" />
-        <origin xyz="0 ${tube_length + hs_645_depth - 0.003} 0.005" rpy="0 0 0"/>
+        <origin xyz="0 0.187 0" rpy="0 0 0"/>
         <limit effort="40" velocity="3" lower="${-PI/2}" upper="${PI/2}" />
         <dynamics damping="5.0" friction="0.08" />
@@ -236,5 +236,5 @@
         <child link="gripper" />
         <axis xyz="0 -1 0" />
-        <origin xyz="0 0.04 0" rpy="0 0 ${PI}" />
+        <origin xyz="-0.005 0.04 0" rpy="0 0 ${PI}" />
         <limit effort="100" velocity="3" lower="${-PI}" upper="${PI}" />
         <dynamics damping="1.0" friction="0.8" />
@@ -243,5 +243,5 @@
         <parent link="gripper" />
         <child link="right_finger" />
-        <origin xyz="-0.006 -0.015 0" />
+        <origin xyz="-0.005 -0.015 0" />
         <limit effort="100" velocity="0.1" lower="0" upper="${gripper_base_width/2}" />
         <mimic joint="Gripper" multiplier="-0.5" offset="${gripper_base_width/2}" />
@@ -251,5 +251,5 @@
         <parent link="gripper" />
         <child link="left_finger" />
-        <origin xyz="-0.0017 -0.015 0" />
+        <origin xyz="0.005 -0.015 0" />
         <axis xyz="-1 0 0" />
         <limit effort="100" velocity="0.1" lower="0" upper="${gripper_base_width/2}" />
@@ -309,6 +309,6 @@
                 <updateRate>1.0</updateRate>
                 <cameraName>external_vision</cameraName>
-                <imageTopicName>image_raw</imageTopicName>
-                <cameraInfoTopicName>camera_info</cameraInfoTopicName>
+                <imageToPIcName>image_raw</imageToPIcName>
+                <cameraInfoToPIcName>camera_info</cameraInfoToPIcName>
                 <frameName>camera_link</frameName>
             </plugin>

Commit message: Updated robot model

File: urdf/lynxmotion_al5d.xacro (robot description, xacro)
@@ -74,5 +74,5 @@
                 <mesh filename="package://lynxmotion_al5d_description/meshes/robot_parts/elbow.dae" />
             </geometry>
-            <origin rpy="${-PI-0.895} ${PI} 0" xyz="-0.005 ${tube_length - 2*hs_755eb_depth/5} ${-shoulder_to_elbow - 0.026}" />
+            <origin rpy="${-PI-0.895} ${PI} 0" xyz="-0.005 ${tube_length - 2*hs_755eb_depth/5} ${-shoulder_to_elbow - 0.02}" />
         </visual>
         <collision>
@@ -80,5 +80,5 @@
                 <mesh filename="package://lynxmotion_al5d_description/meshes/robot_parts/elbow.dae" />
             </geometry>
-            <origin rpy="${-PI-0.895} ${PI} 0" xyz="-0.005 ${tube_length - 2*hs_755eb_depth/5} ${-shoulder_to_elbow - 0.026} " />
+            <origin rpy="${-PI-0.895} ${PI} 0" xyz="-0.005 ${tube_length - 2*hs_755eb_depth/5} ${-shoulder_to_elbow - 0.02} " />
         </collision>
         <xacro:inertial_matrix_bis mass="${hs_755eb_mass + hs_645_mass}" />
@@ -228,5 +228,5 @@
         <child link="wrist" />
         <axis xyz="1 0 0" />
-        <origin xyz="0 0.187 0" rpy="0 0 0"/>
+        <origin xyz="0 0.187 0.005" rpy="0 0 0"/>
         <limit effort="40" velocity="3" lower="${-PI/2}" upper="${PI/2}" />
         <dynamics damping="5.0" friction="0.08" />

Commit message: Updated model

File: urdf/lynxmotion_al5d.xacro (robot description, xacro)
@@ -74,5 +74,5 @@
                 <mesh filename="package://lynxmotion_al5d_description/meshes/robot_parts/elbow.dae" />
             </geometry>
-            <origin rpy="${-PI-0.895} ${PI} 0" xyz="-0.005 ${tube_length - 2*hs_755eb_depth/5} ${-shoulder_to_elbow - 0.02}" />
+            <origin rpy="${-PI-0.895} ${PI} 0" xyz="-0.005 ${tube_length - 2*hs_755eb_depth/5 + 0.005} ${-shoulder_to_elbow - 0.02}" />
         </visual>
         <collision>
@@ -80,5 +80,5 @@
                 <mesh filename="package://lynxmotion_al5d_description/meshes/robot_parts/elbow.dae" />
             </geometry>
-            <origin rpy="${-PI-0.895} ${PI} 0" xyz="-0.005 ${tube_length - 2*hs_755eb_depth/5} ${-shoulder_to_elbow - 0.02} " />
+            <origin rpy="${-PI-0.895} ${PI} 0" xyz="-0.005 ${tube_length - 2*hs_755eb_depth/5 + 0.005} ${-shoulder_to_elbow - 0.02} " />
         </collision>
         <xacro:inertial_matrix_bis mass="${hs_755eb_mass + hs_645_mass}" />
@@ -90,5 +90,5 @@
                 <mesh filename="package://lynxmotion_al5d_description/meshes/robot_parts/wrist.dae" />
             </geometry>
-            <origin rpy="${PI} 0 0" xyz="0 -0.165 0.067" />
+            <origin rpy="${PI} 0 0" xyz="0.005 -0.165 0.067" />
         </visual>
         <collision>
@@ -236,5 +236,5 @@
         <child link="gripper" />
         <axis xyz="0 -1 0" />
-        <origin xyz="-0.005 0.04 0" rpy="0 0 ${PI}" />
+        <origin xyz="0 0.04 0" rpy="0 0 ${PI}" />
         <limit effort="100" velocity="3" lower="${-PI}" upper="${PI}" />
         <dynamics damping="1.0" friction="0.8" />

Commit message: Repositioned joints

File: urdf/lynxmotion_al5d.xacro (robot description, xacro)
@@ -42,5 +42,5 @@
                 <mesh filename="package://lynxmotion_al5d_description/meshes/robot_parts/top_box.dae" />
             </geometry>
-            <origin xyz="-0.01 0.02 0" rpy="0 0 ${PI}" />
+            <origin xyz="-0.01 0.03 0" rpy="0 0 ${PI}" />
         </visual>
         <collision>
@@ -48,5 +48,5 @@
                 <mesh filename="package://lynxmotion_al5d_description/meshes/robot_parts/top_box.dae" />
             </geometry>
-            <origin xyz="-0.01 0.02 0" rpy="0 0 ${PI}" />
+            <origin xyz="-0.01 0.03 0" rpy="0 0 ${PI}" />
         </collision>
         <xacro:inertial_matrix_bis mass="${top_box_mass}" />
@@ -74,5 +74,5 @@
                 <mesh filename="package://lynxmotion_al5d_description/meshes/robot_parts/elbow.dae" />
             </geometry>
-            <origin rpy="${-PI-0.895} ${PI} 0" xyz="-0.005 ${tube_length - 2*hs_755eb_depth/5 + 0.005} ${-shoulder_to_elbow - 0.02}" />
+            <origin rpy="${-PI-0.895} ${PI} 0" xyz="-0.006 ${tube_length - 2*hs_755eb_depth/5} ${-shoulder_to_elbow - 0.018}" />
         </visual>
         <collision>
@@ -90,5 +90,5 @@
                 <mesh filename="package://lynxmotion_al5d_description/meshes/robot_parts/wrist.dae" />
             </geometry>
-            <origin rpy="${PI} 0 0" xyz="0.005 -0.165 0.067" />
+            <origin rpy="${PI} 0 0" xyz="0.005 -0.165 0.0695" />
         </visual>
         <collision>
@@ -228,5 +228,5 @@
         <child link="wrist" />
         <axis xyz="1 0 0" />
-        <origin xyz="0 0.187 0.005" rpy="0 0 0"/>
+        <origin xyz="0 0.181 0.005" rpy="0 0 0"/>
         <limit effort="40" velocity="3" lower="${-PI/2}" upper="${PI/2}" />
         <dynamics damping="5.0" friction="0.08" />
